Commit message: added files for obelix urdf model

File: hector_tracked_vehicles_description/urdf/obelix_ugv_base.urdf.xacro (robot description, xacro)
@@ -21,5 +21,5 @@
     <property name="top_size_y" value="0.3556" />
     <property name="top_size_z" value="0.0020" />
-    <macro name="jasmine_ugv_macro">
+    <macro name="obelix_ugv_macro">
         <!-- base_footprint is a fictitious link(frame) that is on the ground right below base_link origin,
              navigation stack depends on this frame -->
@@ -60,5 +60,5 @@
                 <geometry>
                     <!--<box size="${base_size_x} ${base_size_y} ${base_size_z}" />-->
-                    <mesh filename="package://hector_tracked_vehicles_description/meshes/jasmine_ugv/jasmine_ugv_simple_colored_v001.dae"/>
+                    <mesh filename="package://hector_tracked_vehicles_description/meshes/jasmine_ugv/obelix_ugv_simple_colored_v001.dae"/>
                 </geometry>
                 <material name="Grey" >
@@ -73,5 +73,5 @@
             </collision>
         </link>
-       <!--	Add wheels using the hlugv_wheel macro -->
+        <!--	Add wheels using the hlugv_wheel macro -->
         <tracked_wheel parent="base_link" prefix="left_0" offset_x= "0.21100" offset_y = "${wheel_offset_y}" offset_z = "${wheel_offset_z_from_base_link}" reflect="1" wheel_radius="${wheel_radius_big}"/>
         <tracked_wheel parent="base_link" prefix="left_1" offset_x= "0.0" offset_y = "${wheel_offset_y}" offset_z = "${wheel_offset_z_from_base_link-0.01}" reflect="1" wheel_radius="${wheel_radius_big}"/>

File: hector_tracked_vehicles_description/urdf/tracked_wheel.urdf.xacro (robot description, xacro)
@@ -12,5 +12,5 @@
     <xacro:property name="wheel_offset_z" value="-0.112" />
      <!-- wheel_radius - socket height -->
-    <xacro:macro name="tracked_wheel" params="parent prefix offset_x offset_y offset_z reflect">
+    <xacro:macro name="tracked_wheel" params="parent prefix offset_x offset_y offset_z reflect wheel_radius">
         <joint name="${prefix}_wheel_joint" type="continuous">
             <origin xyz="${offset_x } ${offset_y * reflect} ${offset_z}" rpy="0 0 0" />
