Commit message: -Remove obsolete xacro file

File: hector_tracked_vehicles_description/urdf/obelix_ugv_standalone.urdf.xacro (robot description, xacro)
@@ -1,9 +1,30 @@
 <?xml version="1.0"?>
-<robot name="obelix_ugv"
+<robot name="obelix_ugv "
     xmlns:sensor="http://playerstage.sourceforge.net/gazebo/xmlschema/#sensor"
     xmlns:controller="http://playerstage.sourceforge.net/gazebo/xmlschema/#controller"
     xmlns:interface="http://playerstage.sourceforge.net/gazebo/xmlschema/#interface">
     <!-- Included URDF Files -->
+    <include filename="$(find hector_tracked_vehicles_description)/urdf/obelix_2flipper_wheel.urdf.xacro" />
     <include filename="$(find hector_tracked_vehicles_description)/urdf/obelix_ugv_base.urdf.xacro" />
-    <obelix_ugv_macro />
+<obelix_ugv_macro />
+  <!-- use for 4 flippers
+  <obelix_flipper_macro parent="base_link" name="left_front" front="1">
+    <origin xyz="${base_size_x*0.5} ${base_size_y*0.5+wheel_offset_y+0.5*wheel_size_y}  0 " rpy="0 0 0"/>
+  </obelix_flipper_macro >
+  <obelix_flipper_macro parent="base_link" name="right_front" front="1">
+    <origin xyz="${base_size_x*0.5} ${-(base_size_y*0.5+wheel_offset_y+0.5*wheel_size_y)}  0  " rpy="0 0 0"/>
+  </obelix_flipper_macro >
+  <obelix_flipper_macro parent="base_link" name="right_back" front="-1">
+    <origin xyz="${-base_size_x*0.5} ${-(base_size_y*0.5+wheel_offset_y+0.5*wheel_size_y)}  0  " rpy="0 0 0"/>
+  </obelix_flipper_macro >
+<obelix_flipper_macro parent="base_link" name="left_back" front="-1">
+    <origin xyz="${-base_size_x*0.5} ${(base_size_y*0.5+wheel_offset_y+0.5*wheel_size_y)}  0  " rpy="0 0 0"/>
+  </obelix_flipper_macro > -->
+  <!-- use for 2*2 flippers -->
+  <obelix_flipper_macro parent="base_link" name="front" front="1">
+    <origin xyz="${base_size_x*0.5} ${base_size_y*0.5+wheel_offset_y+0.5*wheel_size_y}  0 " rpy="0 0 0"/>
+  </obelix_flipper_macro >
+  <obelix_flipper_macro parent="base_link" name="back" front="-1">
+    <origin xyz="${-base_size_x*0.5} ${(base_size_y*0.5+wheel_offset_y+0.5*wheel_size_y)}  0  " rpy="0 0 0"/>
+  </obelix_flipper_macro >
 </robot>

Commit message: -Separate real robot and gazebo versions for obelix ugv

File: hector_tracked_vehicles_description/urdf/obelix_ugv_standalone.urdf.xacro (robot description, xacro)
@@ -7,4 +7,11 @@
     <include filename="$(find hector_tracked_vehicles_description)/urdf/obelix_ugv_base.urdf.xacro" />
     <obelix_ugv_macro />
-    <include filename="$(find hector_tracked_vehicles_description)/urdf/obelix_ugv_base.gazebo.xacro" />
+    <include filename="$(find hector_tracked_vehicles_description)/urdf/obelix_2flipper_box.urdf.xacro" />
+      <!-- use for 2*2 flippers -->
+   <obelix_flipper_macro parent="base_link" name="front" front="1">
+     <origin xyz="${base_size_x*0.5} ${base_size_y*0.5+wheel_offset_y+0.5*wheel_size_y}  0 " rpy="0 0 0"/>
+   </obelix_flipper_macro >
+  <obelix_flipper_macro parent="base_link" name="back" front="-1">
+    <origin xyz="${-base_size_x*0.5} ${(base_size_y*0.5+wheel_offset_y+0.5*wheel_size_y)}  0  " rpy="0 0 0"/>
+  </obelix_flipper_macro >
 </robot>
