Commit message: -Change joint name for flippers

File: hector_tracked_vehicles_description/urdf/obelix_flipper_box.urdf.xacro (robot description, xacro)
@@ -10,5 +10,5 @@
     <macro name="obelix_flipper_macro" params="parent name front *origin">
  <!-- front is either 1 (for front flipper) or -1 (for back flipper) -->
-<joint name="${parent}_${name}_flipper_joint" type="revolute">
+<joint name="${name}_flipper_joint" type="revolute">
 <insert_block name="origin"/>
       <axis xyz="0 1 0"/>
