Commit message: Use common base xacro file for gazebo and real robot

File: hector_tracked_vehicles_description/urdf/bertl_ugv_vision_box.gazebo.xacro (robot description, xacro)
@@ -4,26 +4,8 @@
     xmlns:controller="http://playerstage.sourceforge.net/gazebo/xmlschema/#controller"
     xmlns:interface="http://playerstage.sourceforge.net/gazebo/xmlschema/#interface">
-    <include filename="$(find taurob_tracker_description)/urdf/tracker_chassis.urdf.xacro.xml" />
+    <!--Include complete standard bertl setup-->
+    <include filename="$(find hector_tracked_vehicles_description)/urdf/bertl_ugv_vision_box.urdf.xacro"/>
+    <!-- Add gazebo specific additions -->
     <include filename="$(find taurob_tracker_description)/urdf/tracker_chassis.gazebo.xacro.xml" />
-    <include filename="$(find hector_components_description)/urdf/vision_box_common.urdf.xacro"/>
-    <include filename="$(find hector_components_description)/urdf/vision_box_dimensions_hector2.urdf.xacro" />
-    <tracker_chassis_macro />
-    <vision_box parent="chassis_link" box_type="hector2">
-      <origin xyz="-0.155 0 0.105" rpy="0 0 0"/>
-    </vision_box>
     <tracker_chassis_gazebo_macro />
-    <gazebo>
-      <plugin name="imu_controller" filename="libhector_gazebo_ros_imu.so">
-        <alwaysOn>true</alwaysOn>
-        <updateRate>50.0</updateRate>
-        <bodyName>base_link</bodyName>
-        <topicName>imu_quat</topicName>
-        <accelDrift>0.0 0.0 0.0</accelDrift>
-        <accelGaussianNoise>0.1 0.1 0.1</accelGaussianNoise>
-        <rateDrift>0.0 0.0 0.0</rateDrift>
-        <rateGaussianNoise>0.05 0.05 0.05</rateGaussianNoise>
-        <headingDrift>0.0</headingDrift>
-        <headingGaussianNoise>0.05</headingGaussianNoise>
-      </plugin>
-    </gazebo>
   </robot>

Commit message: Update xacro files

File: hector_tracked_vehicles_description/urdf/bertl_ugv_vision_box.gazebo.xacro (robot description, xacro)
@@ -3,9 +3,10 @@
     xmlns:sensor="http://playerstage.sourceforge.net/gazebo/xmlschema/#sensor"
     xmlns:controller="http://playerstage.sourceforge.net/gazebo/xmlschema/#controller"
-    xmlns:interface="http://playerstage.sourceforge.net/gazebo/xmlschema/#interface">
+    xmlns:interface="http://playerstage.sourceforge.net/gazebo/xmlschema/#interface"
+    xmlns:xacro="http://playerstage.sourceforge.net/gazebo/xmlschema/#interface">
     <!--Include complete standard bertl setup-->
-    <include filename="$(find hector_tracked_vehicles_description)/urdf/bertl_ugv_vision_box.urdf.xacro"/>
+    <xacro:include filename="$(find hector_tracked_vehicles_description)/urdf/bertl_ugv_vision_box.urdf.xacro"/>
     <!-- Add gazebo specific additions -->
-    <include filename="$(find taurob_tracker_description)/urdf/tracker_chassis.gazebo.xacro.xml" />
-    <tracker_chassis_gazebo_macro />
+    <xacro:include filename="$(find taurob_tracker_description)/urdf/tracker_chassis.gazebo.xacro.xml" />
+    <xacro:tracker_chassis_gazebo_macro />
   </robot>

File: hector_tracked_vehicles_description/urdf/bertl_ugv_vision_box.urdf.xacro (robot description, xacro)
@@ -3,16 +3,14 @@
     xmlns:sensor="http://playerstage.sourceforge.net/gazebo/xmlschema/#sensor"
     xmlns:controller="http://playerstage.sourceforge.net/gazebo/xmlschema/#controller"
-    xmlns:interface="http://playerstage.sourceforge.net/gazebo/xmlschema/#interface">
-    <property name="flipper_offset_x" value="0.205" />
-    <property name="flipper_offset_y" value="0.15" />
-    <property name="flipper_offset_z" value="0.099" />
-    <property name="M_PI" value="3.14159" />
-    <property name="angle_deg" value="45" />
-    <include filename="$(find taurob_tracker_description)/urdf/tracker_chassis.urdf.xacro.xml" />
-    <include filename="$(find hector_components_description)/urdf/vision_box_common.urdf.xacro"/>
-    <include filename="$(find hector_components_description)/urdf/vision_box_dimensions_hector2.urdf.xacro" />
-    <tracker_chassis_macro />
-    <vision_box parent="chassis_link" box_type="hector2">
+    xmlns:interface="http://playerstage.sourceforge.net/gazebo/xmlschema/#interface"
+    xmlns:xacro="http://playerstage.sourceforge.net/gazebo/xmlschema/#interface">
+    <xacro:property name="M_PI" value="3.14159" />
+    <xacro:include filename="$(find taurob_tracker_description)/urdf/tracker_chassis.urdf.xacro.xml" />
+    <xacro:include filename="$(find hector_components_description)/urdf/vision_box_common.urdf.xacro"/>
+    <xacro:include filename="$(find hector_components_description)/urdf/vision_box_dimensions_hector2.urdf.xacro" />
+    <xacro:tracker_chassis_macro />
+    <xacro:vision_box parent="chassis_link" box_type="hector2">
       <origin xyz="-0.155 0 0.105" rpy="0 0 0"/>
-    </vision_box>
+    </xacro:vision_box>
+    <xacro:include filename="$(find hector_components_description)/urdf/vision_box_hector2_addons.urdf.xacro" />
 </robot>

File: hector_tracked_vehicles_description/urdf/tracked_wheel.urdf.xacro (robot description, xacro)
@@ -1,67 +1,58 @@
 <?xml version="1.0"?>
 <robot
-    xmlns:sensor="http://playerstage.sourceforge.net/gazebo/xmlschema/#sensor"
-    xmlns:controller="http://playerstage.sourceforge.net/gazebo/xmlschema/#controller"
-    xmlns:interface="http://playerstage.sourceforge.net/gazebo/xmlschema/#interface"
-          xmlns:xacro="http://playerstage.sourceforge.net/gazebo/xmlschema/#interface">
-    <!-- Properties (Constants) -->
-    <xacro:property name="M_PI" value="3.14159" />
-    <!--<xacro:property name="wheel_radius" value="0.185" />-->
-    <!--<xacro:property name="wheel_size_y" value="0.0824" />-->
-     <!-- half of wheel width + half of socket width + gap -->
-    <xacro:property name="wheel_offset_z" value="-0.112" />
-     <!-- wheel_radius - socket height -->
-    <xacro:macro name="tracked_wheel" params="parent prefix offset_x offset_y offset_z reflect wheel_radius">
-        <joint name="${prefix}_wheel_joint" type="continuous">
-            <origin xyz="${offset_x } ${offset_y * reflect} ${offset_z}" rpy="0 0 0" />
-            <parent link="${parent}" />
-            <child link="${prefix}_wheel_link" />
-            <axis xyz="0 1 0" />
-            <limit effort="100" velocity="100" />
-            <joint_properties damping="0.0" friction="0.0" />
-            <anchor xyz="0 0 0" />
-        </joint>
-        <link name="${prefix}_wheel_link">
-            <inertial>
-                <mass value="0.01" />
-                <origin xyz=" 0 0 0 " />
-                <inertia  ixx="0.00012411765597" ixy="0.0" ixz="0.0"
-                          iyy="0.00015218160428" iyz="0.0"
-                          izz="0.00011763977943" />
-            </inertial>
-<!--            <visual>
-                <origin xyz="0 0 0" rpy="${-M_PI/2} 0 0" />
-                <geometry>
-                    <cylinder radius="${wheel_radius}" length="${wheel_size_y}"/>
-                </geometry>
-                <material name="DarkGrey" >
-                    <color rgba="0.3 0.3 0.3 1"/>
-                </material>
-            </visual>-->
-            <collision>
-                <origin xyz="0 0 0" rpy="${-M_PI/2} 0 0" />
-                <geometry>
-                    <cylinder radius="${wheel_radius}" length="${wheel_size_y}" />
-                    <!--<box size="1.0 0.5 0.1" />-->
-                </geometry>
-                <!--<material name="MTWheelColMat"/>-->
-            </collision>
-        </link>
-        <gazebo reference="${prefix}_wheel_link" >
-            <mu1>1.0</mu1>
-            <mu2>1.0</mu2>
-            <kp>1000000.0</kp>
-            <kd>100.0</kd>
-            <minDepth>0.001</minDepth>
-            <maxVel>1.0</maxVel>
-            <!--<fdir1>1 0 0</fdir1>-->
-            <!--<maxVel>1.0</maxVel>-->
-        </gazebo>
-        <transmission type="pr2_mechanism_model/SimpleTransmission" name="${prefix}_wheel_trans">
-            <actuator name="${prefix}_motor_link" />
-            <joint name="${prefix}_wheel_joint" />
-            <mechanicalReduction>1.0</mechanicalReduction>
-            <motorTorqueConstant>1</motorTorqueConstant>
-        </transmission>
+  xmlns:sensor="http://playerstage.sourceforge.net/gazebo/xmlschema/#sensor"
+  xmlns:controller="http://playerstage.sourceforge.net/gazebo/xmlschema/#controller"
+  xmlns:interface="http://playerstage.sourceforge.net/gazebo/xmlschema/#interface"
+  xmlns:xacro="http://playerstage.sourceforge.net/gazebo/xmlschema/#interface">
+  <!-- Properties (Constants) -->
+  <xacro:property name="M_PI" value="3.14159" />
+  <!--<xacro:property name="wheel_radius" value="0.185" />-->
+  <!--<xacro:property name="wheel_size_y" value="0.0824" />-->
+  <!-- half of wheel width + half of socket width + gap -->
+  <xacro:property name="wheel_offset_z" value="-0.112" />
+  <!-- wheel_radius - socket height -->
+  <xacro:macro name="tracked_wheel" params="parent prefix offset_x offset_y offset_z reflect wheel_radius">
+    <joint name="${prefix}_wheel_joint" type="continuous">
+      <origin xyz="${offset_x } ${offset_y * reflect} ${offset_z}" rpy="0 0 0" />
+      <parent link="${parent}" />
+      <child link="${prefix}_wheel_link" />
+      <axis xyz="0 1 0" />
+      <limit effort="100" velocity="100" />
+      <joint_properties damping="0.0" friction="0.0" />
+      <anchor xyz="0 0 0" />
+    </joint>
+    <link name="${prefix}_wheel_link">
+      <inertial>
+        <mass value="0.01" />
+        <origin xyz=" 0 0 0 " />
+        <inertia  ixx="0.00012411765597" ixy="0.0" ixz="0.0"
+                 iyy="0.00015218160428" iyz="0.0"
+                 izz="0.00011763977943" />
+        </inertial>
+        <collision>
+          <origin xyz="0 0 0" rpy="${-M_PI/2} 0 0" />
+          <geometry>
+            <cylinder radius="${wheel_radius}" length="${wheel_size_y}" />
+            <!--<box size="1.0 0.5 0.1" />-->
+          </geometry>
+          <!--<material name="MTWheelColMat"/>-->
+        </collision>
+      </link>
+      <gazebo reference="${prefix}_wheel_link" >
+        <mu1>1.0</mu1>
+        <mu2>1.0</mu2>
+        <kp>1000000.0</kp>
+        <kd>100.0</kd>
+        <minDepth>0.001</minDepth>
+        <maxVel>1.0</maxVel>
+        <!--<fdir1>1 0 0</fdir1>-->
+        <!--<maxVel>1.0</maxVel>-->
+      </gazebo>
+      <transmission type="pr2_mechanism_model/SimpleTransmission" name="${prefix}_wheel_trans">
+        <actuator name="${prefix}_motor_link" />
+        <joint name="${prefix}_wheel_joint" />
+        <mechanicalReduction>1.0</mechanicalReduction>
+        <motorTorqueConstant>1</motorTorqueConstant>
+      </transmission>
     </xacro:macro>
-</robot>
+  </robot>
