Commit message: Make things work properly in gazebo

File: hector_tracked_vehicles_description/urdf/obelix_2flipper_box.urdf.xacro (robot description, xacro)
@@ -78,7 +78,4 @@
       <flipper_geom_macro_collision front="${front}" />
     </link>
-    <gazebo reference="left_${name}_flipper_link">
-      <material>Gazebo/Grey</material>
-    </gazebo>
     <joint name="right_${name}_flipper_joint" type="fixed">
       <origin xyz="0 ${-2*flipper_offset_y} 0" rpy="0 0 0" />
@@ -94,6 +91,34 @@
       <flipper_geom_macro_collision front="${front}" />
     </link>
-    <gazebo reference="right_${name}_flipper_link">
+    <!--Needed for gazebo-->
+    <transmission name="${name}_flipper_joint_transmission">
+      <type>transmission_interface/SimpleTransmission</type>
+      <joint name="${name}_flipper_joint">
+        <hardwareInterface>EffortJointInterface</hardwareInterface>
+      </joint>
+      <actuator name="${name}_flipper_joint_motor">
+        <hardwareInterface>EffortJointInterface</hardwareInterface>
+        <mechanicalReduction>1</mechanicalReduction>
+      </actuator>
+    </transmission>
+    <gazebo reference="${name}_left_flipper_base_link">
       <material>Gazebo/Grey</material>
+      <mu1>0</mu1>
+      <mu2>0</mu2>
+      <kp>1000000.0</kp>
+      <kd>100.0</kd>
+      <minDepth>0.001</minDepth>
+      <maxVel>1.0</maxVel>
+      <maxContacts>1</maxContacts>
+    </gazebo>
+    <gazebo reference="${name}_right_flipper_base_link">
+      <material>Gazebo/Grey</material>
+      <mu1>0</mu1>
+      <mu2>0</mu2>
+      <kp>1000000.0</kp>
+      <kd>100.0</kd>
+      <minDepth>0.001</minDepth>
+      <maxVel>1.0</maxVel>
+      <maxContacts>1</maxContacts>
     </gazebo>
   </macro>

File: hector_tracked_vehicles_description/urdf/obelix_ugv_base.urdf.xacro (robot description, xacro)
@@ -8,10 +8,10 @@
   <!-- Properties (Constants) -->
   <property name="M_PI" value="3.14159"/>
-  <property name="base_size_x" value="0.52" />
-  <property name="base_size_y" value="0.18" />
-  <property name="base_size_z" value="0.118" />
+  <property name="base_link_size_x" value="0.52" />
+  <property name="base_link_size_y" value="0.18" />
+  <property name="base_link_size_z" value="0.118" />
   <property name="wheel_radius_big" value="0.085" />
-  <property name="wheel_offset_x" value="${base_size_x*0.5 - 0.042}" />
-  <property name="wheel_offset_z" value="${base_size_z*0.5 - 0.065}" />
+  <property name="wheel_offset_x" value="${base_link_size_x*0.5 - 0.042}" />
+  <property name="wheel_offset_z" value="${base_link_size_z*0.5 - 0.065}" />
   <property name="wheel_radius"   value="0.09" />
   <property name="track_width"    value="0.1" />
@@ -50,5 +50,5 @@
       <origin xyz="0.0 ${offset_y} ${wheel_offset_z}" rpy="0 0 0" />
       <geometry>
-        <box size="${base_size_x - wheel_radius} ${track_width} ${wheel_radius*2}" />
+        <box size="${base_link_size_x - wheel_radius} ${track_width} ${wheel_radius*2}" />
       </geometry>
     </visual>
@@ -70,5 +70,5 @@
       <origin xyz="0.0 ${offset_y} ${wheel_offset_z}" rpy="0 0 0" />
       <geometry>
-        <box size="${base_size_x - wheel_radius} ${track_width} ${wheel_radius*2}" />
+        <box size="${base_link_size_x - wheel_radius} ${track_width} ${wheel_radius*2}" />
       </geometry>
     </collision>
@@ -77,5 +77,5 @@
     <!-- Links and Joints (i.e., the robot) -->
     <link name="base_link">
-      <inertial_cuboid_with_pose mass="40" x_length="${base_size_x}" y_length="${base_size_y}" z_length="${base_size_z}" >
+      <inertial_cuboid_with_pose mass="40" x_length="${base_link_size_x}" y_length="${base_link_size_y}" z_length="${base_link_size_z}" >
         <origin xyz="0 0.0 0.0" rpy="0 0 0" />
       </inertial_cuboid_with_pose>
@@ -83,8 +83,8 @@
         <origin xyz="0.0 0.0 0.0" rpy="0 0 0" />
         <geometry>
-          <box size="${base_size_x} ${base_size_y} ${base_size_z}" />
+          <box size="${base_link_size_x} ${base_link_size_y} ${base_link_size_z}" />
         </geometry>
         <geometry>
-          <box size="${base_size_x} ${base_size_y} ${base_size_z}" />
+          <box size="${base_link_size_x} ${base_link_size_y} ${base_link_size_z}" />
         </geometry>
         <material name="Grey" >
@@ -97,8 +97,8 @@
         <origin xyz="0.0 0.0 0.0" rpy="0 0 0" />
         <geometry>
-          <box size="${base_size_x} ${base_size_y} ${base_size_z}" />
+          <box size="${base_link_size_x} ${base_link_size_y} ${base_link_size_z}" />
         </geometry>
         <geometry>
-          <box size="${base_size_x} ${base_size_y} ${base_size_z}" />
+          <box size="${base_link_size_x} ${base_link_size_y} ${base_link_size_z}" />
         </geometry>
       </collision>

File: hector_tracked_vehicles_description/urdf/obelix_ugv_standalone.urdf.xacro (robot description, xacro)
@@ -1,17 +1,61 @@
 <?xml version="1.0"?>
 <robot name="obelix_ugv "
-    xmlns:sensor="http://playerstage.sourceforge.net/gazebo/xmlschema/#sensor"
-    xmlns:controller="http://playerstage.sourceforge.net/gazebo/xmlschema/#controller"
-    xmlns:interface="http://playerstage.sourceforge.net/gazebo/xmlschema/#interface">
-    <!-- Included URDF Files -->
-    <include filename="$(find hector_tracked_vehicles_description)/urdf/obelix_ugv_base.urdf.xacro" />
-    <obelix_ugv_macro />
-    <include filename="$(find hector_tracked_vehicles_description)/urdf/obelix_2flipper_box.urdf.xacro" />
-      <!-- use for 2*2 flippers -->
-   <obelix_flipper_macro parent="base_link" name="front" front="1">
-     <origin xyz="${wheel_offset_x}  ${flipper_offset_y}  0 " rpy="0 0 0"/>
-   </obelix_flipper_macro >
+       xmlns:sensor="http://playerstage.sourceforge.net/gazebo/xmlschema/#sensor"
+       xmlns:controller="http://playerstage.sourceforge.net/gazebo/xmlschema/#controller"
+       xmlns:interface="http://playerstage.sourceforge.net/gazebo/xmlschema/#interface">
+  <!-- Included URDF Files -->
+  <include filename="$(find hector_tracked_vehicles_description)/urdf/obelix_ugv_base.urdf.xacro" />
+  <obelix_ugv_macro />
+  <include filename="$(find hector_tracked_vehicles_description)/urdf/obelix_2flipper_box.urdf.xacro" />
+  <!-- use for 2*2 flippers -->
+  <obelix_flipper_macro parent="base_link" name="front" front="1">
+    <origin xyz="${wheel_offset_x}  ${flipper_offset_y}  0 " rpy="0 0 0"/>
+  </obelix_flipper_macro >
   <obelix_flipper_macro parent="base_link" name="rear" front="-1">
     <origin xyz="${-wheel_offset_x}  ${flipper_offset_y}  0  " rpy="0 0 0"/>
   </obelix_flipper_macro >
+  <gazebo reference="base_link">
+    <mu1>0.0</mu1>
+    <mu2>0.0</mu2>
+    <kp>1000000.0</kp>
+    <kd>100.0</kd>
+    <minDepth>0.001</minDepth>
+    <maxVel>1.0</maxVel>
+  </gazebo>
+  <gazebo>
+    <plugin name="force_based_move_controller" filename="libgazebo_ros_force_based_move.so">
+      <commandTopic>/cmd_vel_raw</commandTopic>
+      <odometryTopic>odom</odometryTopic>
+      <odometryFrame>odom</odometryFrame>
+      <odometryRate>20.0</odometryRate>
+      <robotBaseFrame>base_link</robotBaseFrame>
+      <publishOdometryTf>0</publishOdometryTf>
+    </plugin>
+    <!-- ros_control plugin -->
+    <plugin name="gazebo_ros_control" filename="libgazebo_ros_control.so">
+      <robotNamespace>obelix_robot</robotNamespace>
+    </plugin>
+    <plugin name="p3d_base_controller" filename="libgazebo_ros_p3d.so">
+      <alwaysOn>true</alwaysOn>
+      <updateRate>50.0</updateRate>
+      <bodyName>base_link</bodyName>
+      <topicName>ground_truth/state</topicName>
+      <gaussianNoise>0.01</gaussianNoise>
+      <frameName>world</frameName>
+      <xyzOffsets>0 0 0</xyzOffsets>
+      <rpyOffsets>0 0 0</rpyOffsets>
+    </plugin>
+    <plugin name="imu_controller" filename="libhector_gazebo_ros_imu.so">
+      <alwaysOn>true</alwaysOn>
+      <updateRate>50.0</updateRate>
+      <bodyName>base_link</bodyName>
+      <topicName>imu_quat</topicName>
+      <accelDrift>0.0 0.0 0.0</accelDrift>
+      <accelGaussianNoise>0.1 0.1 0.1</accelGaussianNoise>
+      <rateDrift>0.0 0.0 0.0</rateDrift>
+      <rateGaussianNoise>0.05 0.05 0.05</rateGaussianNoise>
+      <headingDrift>0.0</headingDrift>
+      <headingGaussianNoise>0.05</headingGaussianNoise>
+    </plugin>
+  </gazebo>
 </robot>

Commit message: Remove gazebo material tags for the moment

File: hector_tracked_vehicles_description/urdf/obelix_2flipper_box.urdf.xacro (robot description, xacro)
@@ -99,5 +99,5 @@
     </transmission>
     <gazebo reference="${name}_left_flipper_base_link">
-      <material>Gazebo/Grey</material>
+      <!--<material>Gazebo/Grey</material>-->
       <mu1>0</mu1>
       <mu2>0</mu2>
@@ -109,5 +109,5 @@
     </gazebo>
     <gazebo reference="${name}_right_flipper_base_link">
-      <material>Gazebo/Grey</material>
+      <!--<material>Gazebo/Grey</material>-->
       <mu1>0</mu1>
       <mu2>0</mu2>

File: hector_tracked_vehicles_description/urdf/obelix_ugv_standalone.urdf.xacro (robot description, xacro)
@@ -16,4 +16,5 @@
   </obelix_flipper_macro >
   <gazebo reference="base_link">
+    <!--<material>Gazebo/White</material>-->
     <mu1>0.0</mu1>
     <mu2>0.0</mu2>
