Commit message: improve the link&joint naming scheme

File: hector_tracked_vehicles_description/urdf/jasmine_2018_ugv_arm.gazebo.xacro (robot description, xacro)
@@ -9,4 +9,14 @@
     </joint>
     <actuator name="arm_yaw_joint_motor">
+      <hardwareInterface>hardware_interface/EffortJointInterface</hardwareInterface>
+      <mechanicalReduction>1</mechanicalReduction>
+    </actuator>
+  </transmission>
+  <transmission name="arm_pitch_joint_0_transmission">
+    <type>transmission_interface/SimpleTransmission</type>
+    <joint name="arm_pitch_joint_0">
+      <hardwareInterface>hardware_interface/EffortJointInterface</hardwareInterface>
+    </joint>
+    <actuator name="arm_pitch_joint_0_motor">
       <hardwareInterface>hardware_interface/EffortJointInterface</hardwareInterface>
       <mechanicalReduction>1</mechanicalReduction>
@@ -29,14 +39,4 @@
     </joint>
     <actuator name="arm_pitch_joint_2_motor">
-      <hardwareInterface>hardware_interface/EffortJointInterface</hardwareInterface>
-      <mechanicalReduction>1</mechanicalReduction>
-    </actuator>
-  </transmission>
-  <transmission name="arm_pitch_joint_3_transmission">
-    <type>transmission_interface/SimpleTransmission</type>
-    <joint name="arm_pitch_joint_3">
-      <hardwareInterface>hardware_interface/EffortJointInterface</hardwareInterface>
-    </joint>
-    <actuator name="arm_pitch_joint_3_motor">
       <hardwareInterface>hardware_interface/EffortJointInterface</hardwareInterface>
       <mechanicalReduction>1</mechanicalReduction>
@@ -66,5 +66,5 @@
     <plugin name="gazebo_ros_control_select_joints" filename="libgazebo_ros_control_select_joints.so">
       <robotNamespace>manipulator_arm_control</robotNamespace>
-      <joints>arm_yaw_joint arm_pitch_joint_1 arm_pitch_joint_2 arm_pitch_joint_3 arm_roll_joint</joints>
+      <joints>arm_yaw_joint arm_pitch_joint_0 arm_pitch_joint_1 arm_pitch_joint_2 arm_roll_joint</joints>
     </plugin>
   </gazebo>
@@ -76,7 +76,7 @@
   </gazebo>
   <gazebo>
-    <plugin name="mimic_gripper_finger_joint_1" filename="libroboticsgroup_gazebo_mimic_joint_plugin.so">
+    <plugin name="mimic_gripper_finger_joint_0" filename="libroboticsgroup_gazebo_mimic_joint_plugin.so">
       <joint>gripper_servo_joint</joint>
-      <mimicJoint>gripper_finger_joint_1</mimicJoint>
+      <mimicJoint>gripper_finger_joint_0</mimicJoint>
       <multiplier>${8/23}</multiplier>
       <offset>0</offset>
@@ -86,7 +86,7 @@
   </gazebo>
   <gazebo>
-    <plugin name="mimic_gripper_finger_joint_2" filename="libroboticsgroup_gazebo_mimic_joint_plugin.so">
+    <plugin name="mimic_gripper_finger_joint_1" filename="libroboticsgroup_gazebo_mimic_joint_plugin.so">
       <joint>gripper_servo_joint</joint>
-      <mimicJoint>gripper_finger_joint_2</mimicJoint>
+      <mimicJoint>gripper_finger_joint_1</mimicJoint>
       <multiplier>${8/23}</multiplier>
       <offset>0</offset>
@@ -112,20 +112,20 @@
     </plugin>
   </gazebo>-->
-  <gazebo reference="arm_link_0">
+  <gazebo reference="arm_base_link">
     <material>Gazebo/DarkGrey</material>
   </gazebo>
-  <gazebo reference="arm_link_1">
+  <gazebo reference="arm_yaw_link">
     <material>Gazebo/DarkGrey</material>
   </gazebo>
-  <gazebo reference="arm_link_2">
+  <gazebo reference="arm_pitch_link_0">
     <material>Gazebo/DarkGrey</material>
   </gazebo>
-  <gazebo reference="arm_link_3">
+  <gazebo reference="arm_pitch_link_1">
     <material>Gazebo/DarkGrey</material>
   </gazebo>
-  <gazebo reference="arm_link_4">
+  <gazebo reference="arm_pitch_link_2">
     <material>Gazebo/DarkGrey</material>
   </gazebo>
-  <gazebo reference="arm_link_5">
+  <gazebo reference="arm_roll_link">
     <material>Gazebo/DarkGrey</material>
   </gazebo>
@@ -133,8 +133,8 @@
     <material>Gazebo/DarkGrey</material>
   </gazebo>
-  <gazebo reference="gripper_finger_link_1">
+  <gazebo reference="gripper_finger_link_0">
     <material>Gazebo/DarkGrey</material>
   </gazebo>
-  <gazebo reference="gripper_finger_link_2">
+  <gazebo reference="gripper_finger_link_1">
     <material>Gazebo/DarkGrey</material>
   </gazebo>

File: hector_tracked_vehicles_description/urdf/jasmine_2018_ugv_arm.urdf.xacro (robot description, xacro)
@@ -13,10 +13,10 @@
   <xacro:property name="joint_friction" value="0.5" />
   <xacro:macro name="manipulator_arm_macro" params="parent *origin">
-    <joint name="arm_base" type="fixed">
+    <joint name="arm_base_joint" type="fixed">
       <xacro:insert_block name="origin" />
       <parent link="${parent}" />
-      <child link="arm_link_0" />
-    </joint>
-    <link name="arm_link_0">
+      <child link="arm_base_link" />
+    </joint>
+    <link name="arm_base_link">
       <visual>
         <origin xyz="0 0.0 0.0" rpy="0.0 0.0 0.0" />
@@ -46,9 +46,9 @@
       <axis xyz="0 0 1" />
       <limit lower="${-pi+0.001}" upper="${pi-0.001}" effort="${XM430_W350_max_effort}" velocity="${XM430_W350_max_velocity}" />
-      <parent link="arm_link_0" />
-      <child link="arm_link_1" />
-      <dynamics friction="${joint_friction}" damping="${joint_damping}" />
-    </joint>
-    <link name="arm_link_1">
+      <parent link="arm_base_link" />
+      <child link="arm_yaw_link" />
+      <dynamics friction="${joint_friction}" damping="${joint_damping}" />
+    </joint>
+    <link name="arm_yaw_link">
       <visual>
         <origin xyz="0 0.0 0.0" rpy="0.0 0.0 0.0" />
@@ -74,13 +74,13 @@
       </inertial>
     </link>
-    <joint name="arm_pitch_joint_1" type="revolute">
+    <joint name="arm_pitch_joint_0" type="revolute">
       <origin xyz="0.0 0.0 0.0515" rpy=" ${pi/2} 0.0 0.0" />
       <axis xyz="0 0 1" />
       <limit lower="${-100 * pi / 180}" upper="${100 * pi / 180}" effort="${XM540_W270_max_effort}" velocity="${XM540_W270_max_velocity}" />
-      <parent link="arm_link_1" />
-      <child link="arm_link_2" />
-      <dynamics friction="${joint_friction}" damping="${joint_damping}" />
-    </joint>
-    <link name="arm_link_2">
+      <parent link="arm_yaw_link" />
+      <child link="arm_pitch_link_0" />
+      <dynamics friction="${joint_friction}" damping="${joint_damping}" />
+    </joint>
+    <link name="arm_pitch_link_0">
       <visual>
         <origin xyz="0.0 0.0 0.0" rpy="0.0 0.0 0.0" />
@@ -124,13 +124,13 @@
       </inertial>
     </link>
-    <joint name="arm_pitch_joint_2" type="revolute">
+    <joint name="arm_pitch_joint_1" type="revolute">
       <origin xyz="0.026 0.2517 0.0" rpy="0.0 0.0 ${-pi/2}" />
       <axis xyz="0 0 1" />
       <limit lower="${-180 * pi / 180}" upper="${25 * pi / 180}" effort="${XM430_W350_max_effort}" velocity="${XM430_W350_max_velocity}" />
-      <parent link="arm_link_2" />
-      <child link="arm_link_3" />
-      <dynamics friction="${joint_friction}" damping="${joint_damping}" />
-    </joint>
-    <link name="arm_link_3">
+      <parent link="arm_pitch_link_0" />
+      <child link="arm_pitch_link_1" />
+      <dynamics friction="${joint_friction}" damping="${joint_damping}" />
+    </joint>
+    <link name="arm_pitch_link_1">
       <visual>
         <origin xyz="0.0 0.0 0.0" rpy="0.0 0.0 0.0" />
@@ -174,13 +174,13 @@
       </inertial>
     </link>
-    <joint name="arm_pitch_joint_3" type="revolute">
+    <joint name="arm_pitch_joint_2" type="revolute">
       <origin xyz="-0.1967 -0.004 0.0" rpy="0.0 0.0 0.0" />
       <axis xyz="0 0 1" />
       <limit lower="${-95 * pi / 180}" upper="${95 * pi / 180}" effort="${XM430_W350_max_effort}" velocity="${XM430_W350_max_velocity}" />
-      <parent link="arm_link_3" />
-      <child link="arm_link_4" />
-      <dynamics friction="${joint_friction}" damping="${joint_damping}" />
-    </joint>
-    <link name="arm_link_4">
+      <parent link="arm_pitch_link_1" />
+      <child link="arm_pitch_link_2" />
+      <dynamics friction="${joint_friction}" damping="${joint_damping}" />
+    </joint>
+    <link name="arm_pitch_link_2">
       <visual>
         <origin xyz="0.0 0.0 0.0" rpy="0.0 0.0 0.0" />
@@ -222,9 +222,9 @@
       <axis xyz="0 0 1" />
       <limit lower="${-95 * pi / 180}" upper="${95 * pi / 180}" effort="${XM430_W350_max_effort}" velocity="${XM430_W350_max_velocity}" />
-      <parent link="arm_link_4" />
-      <child link="arm_link_5" />
-      <dynamics friction="${joint_friction}" damping="${joint_damping}" />
-    </joint>
-    <link name="arm_link_5">
+      <parent link="arm_pitch_link_2" />
+      <child link="arm_roll_link" />
+      <dynamics friction="${joint_friction}" damping="${joint_damping}" />
+    </joint>
+    <link name="arm_roll_link">
       <visual>
         <origin xyz="0.0 0.0 0.0" rpy="0.0 0.0 0.0" />
@@ -264,5 +264,5 @@
     <joint name="gripper_mount_joint" type="fixed">
       <origin xyz="0.0 0.0 0.0" rpy="0.0 0.0 0.0" />
-      <parent link="arm_link_5" />
+      <parent link="arm_roll_link" />
       <child link="gripper_palm_link" />
     </joint>
@@ -371,14 +371,14 @@
     </link>
 	  <!-- gripper finger -->
-    <joint name="gripper_finger_joint_1" type="continuous">
+    <joint name="gripper_finger_joint_0" type="continuous">
       <origin xyz="0.0 -0.020125 0.04108" rpy="0.0 ${pi / 2} 0.0" />
       <axis xyz="0 0 1" />
       <limit lower="${-0.95*pi}" upper="${0.95*pi}" effort="${XM430_W350_max_effort}" velocity="${XM430_W350_max_velocity}" />
       <parent link="gripper_palm_link" />
-      <child link="gripper_finger_link_1" />
+      <child link="gripper_finger_link_0" />
       <mimic joint="gripper_servo_joint" multiplier="${8 / 23}" offset="0" />
       <dynamics friction="${joint_friction}" damping="${joint_damping}" />
     </joint>
-    <link name="gripper_finger_link_1">
+    <link name="gripper_finger_link_0">
       <visual>
         <origin xyz="0.0 0.0 0.0" rpy="0.0 0.0 0.0" />
@@ -422,14 +422,14 @@
       </inertial>
     </link>
-    <joint name="gripper_finger_joint_2" type="continuous">
+    <joint name="gripper_finger_joint_1" type="continuous">
       <origin xyz="0.0 0.020125 0.04108" rpy="0.0 ${pi / 2} ${pi}" />
       <axis xyz="0 0 1" />
       <limit lower="${-0.95*pi}" upper="${0.95*pi}" effort="${XM430_W350_max_effort}" velocity="${XM430_W350_max_velocity}" />
       <parent link="gripper_palm_link" />
-      <child link="gripper_finger_link_2" />
+      <child link="gripper_finger_link_1" />
       <mimic joint="gripper_servo_joint" multiplier="${8 / 23}" offset="0" />
       <dynamics friction="${joint_friction}" damping="${joint_damping}" />
     </joint>
-    <link name="gripper_finger_link_2">
+    <link name="gripper_finger_link_1">
       <visual>
         <origin xyz="0.0 0.0 0.0" rpy="0.0 0.0 0.0" />
