Commit message: -Basics working in Gazebo. Tweaking skid steering difficult as not clear how to change parameters (fdir1, mu1, mu2 etc.) properly

File: hector_tracked_vehicles_description/urdf/jasmine_ugv_base.urdf.xacro (robot description, xacro)
@@ -10,18 +10,15 @@
     <property name="base_size_y" value="0.12" />
     <property name="base_size_z" value="0.085" />
-    <property name="wheel_radius" value="0.063" />
+    <property name="wheel_radius" value="0.085" />
     <property name="wheel_length" value="0.02" />
     <property name="wheel_size_y" value="0.05" />
     <property name="total_width" value="0.297" />
     <!--    <property name="wheel_offset_y" value="${(total_width - wheel_size_y) / 2}" />-->
-    <property name="wheel_offset_y" value="0.12350" />
-    <property name="wheel_offset_z_from_base_link" value="-0.029500" />
+    <property name="wheel_offset_y" value="0.1697" />
+    <property name="wheel_offset_z_from_base_link" value="-0.0" />
     <property name="ground_clearance" value="0.05" />
     <property name="top_size_x" value="0.3937" />
     <property name="top_size_y" value="0.3556" />
     <property name="top_size_z" value="0.0020" />
-    <property name="caster_wheel_offset_y" value="0.17" />
-    <property name="caster_support_x" value="0.086" />
-    <property name="caster_support_z" value="0.1095" />
     <macro name="jasmine_ugv_macro">
         <!-- base_footprint is a fictitious link(frame) that is on the ground right below base_link origin,
@@ -59,5 +56,5 @@
         <link name="base_link">
             <inertial>
-                <mass value="3.5" />
+                <mass value="25.0" />
                 <origin xyz="0.0 0.0 0.0" rpy="0 0 0" />
                 <inertia ixx="0.005" ixy="0.0" ixz="0.0"
@@ -66,7 +63,8 @@
             </inertial>
             <visual>
-                <origin xyz="0.0 0.0 0.0" rpy="0 0 0" />
+                <origin xyz="0.0 0.0 -0.085" rpy="0 0 0" />
                 <geometry>
-                    <box size="${base_size_x} ${base_size_y} ${base_size_z}" />
+                    <!--<box size="${base_size_x} ${base_size_y} ${base_size_z}" />-->
+                    <mesh filename="package://hector_tracked_vehicles_description/meshes/jasmine_ugv/jasmine_ugv_simple_colored_v001.dae"/>
                 </geometry>
                 <material name="Grey" >
@@ -82,21 +80,24 @@
         </link>
         <!--	Add wheels using the hlugv_wheel macro -->
-        <tracked_wheel parent="base_link" prefix="left_0" offset_x= "0.15" offset_y = "${wheel_offset_y}" offset_z = "${wheel_offset_z_from_base_link}" reflect="1" />
+        <tracked_wheel parent="base_link" prefix="left_0" offset_x= "0.21100" offset_y = "${wheel_offset_y}" offset_z = "${wheel_offset_z_from_base_link}" reflect="1" />
         <tracked_wheel parent="base_link" prefix="left_1" offset_x= "0.0" offset_y = "${wheel_offset_y}" offset_z = "${wheel_offset_z_from_base_link}" reflect="1" />
-        <tracked_wheel parent="base_link" prefix="left_2" offset_x= "-0.15" offset_y = "${wheel_offset_y}" offset_z = "${wheel_offset_z_from_base_link}" reflect="1" />
-        <tracked_wheel parent="base_link" prefix="right_0" offset_x= "0.15" offset_y = "-${wheel_offset_y}" offset_z = "${wheel_offset_z_from_base_link}" reflect="1" />
-        <tracked_wheel parent="base_link" prefix="right_1" offset_x= "0.0" offset_y = "-${wheel_offset_y}" offset_z = "${wheel_offset_z_from_base_link}" reflect="1" />
-        <tracked_wheel parent="base_link" prefix="right_2" offset_x= "-0.15" offset_y = "-${wheel_offset_y}" offset_z = "${wheel_offset_z_from_base_link}" reflect="1" />
+        <tracked_wheel parent="base_link" prefix="left_2" offset_x= "-0.21100" offset_y = "${wheel_offset_y}" offset_z = "${wheel_offset_z_from_base_link-0.01}" reflect="1" />
+        <tracked_wheel parent="base_link" prefix="left_3" offset_x= "0.10550" offset_y = "${wheel_offset_y}" offset_z = "${wheel_offset_z_from_base_link}" reflect="1" />
+        <tracked_wheel parent="base_link" prefix="left_4" offset_x= "-0.10550" offset_y = "${wheel_offset_y}" offset_z = "${wheel_offset_z_from_base_link}" reflect="1" />
+        <tracked_wheel parent="base_link" prefix="right_0" offset_x= "0.21100" offset_y = "-${wheel_offset_y}" offset_z = "${wheel_offset_z_from_base_link}" reflect="1" />
+        <tracked_wheel parent="base_link" prefix="right_1" offset_x= "0.0" offset_y = "-${wheel_offset_y}" offset_z = "${wheel_offset_z_from_base_link-0.01}" reflect="1" />
+        <tracked_wheel parent="base_link" prefix="right_2" offset_x= "-0.21100" offset_y = "-${wheel_offset_y}" offset_z = "${wheel_offset_z_from_base_link}" reflect="1" />
+        <tracked_wheel parent="base_link" prefix="right_3" offset_x= "-0.10550" offset_y = "-${wheel_offset_y}" offset_z = "${wheel_offset_z_from_base_link}" reflect="1" />
+        <tracked_wheel parent="base_link" prefix="right_4" offset_x= "0.10550" offset_y = "-${wheel_offset_y}" offset_z = "${wheel_offset_z_from_base_link}" reflect="1" />
         <gazebo>
         <plugin name="diffdrive_plugin_multiwheel" filename="libdiffdrive_plugin_multi_wheel.so">
 <!--        <controller:diffdrive_plugin_6w name="differential_drive_controller" plugin="libdiffdrive_plugin_6w.so">-->
                 <alwaysOn>true</alwaysOn>
-                <update>100</update>
                 <updateRate>100.0</updateRate>
-                <leftJoints>left_0_wheel_joint left_1_wheel_joint left_2_wheel_joint</leftJoints>
-                <rightJoints>right_0_wheel_joint right_1_wheel_joint right_2_wheel_joint</rightJoints>
+                <leftJoints>left_0_wheel_joint left_1_wheel_joint left_2_wheel_joint left_3_wheel_joint left_4_wheel_joint</leftJoints>
+                <rightJoints>right_0_wheel_joint right_1_wheel_joint right_2_wheel_joint right_3_wheel_joint right_4_wheel_joint</rightJoints>
                 <wheelSeparation>${wheel_offset_y*2}</wheelSeparation>
                 <wheelDiameter>${wheel_radius*2}</wheelDiameter>
-                <torque>50</torque>
+                <torque>5000</torque>
                 <interface:position name="position_iface_2"/>
                 <robotNamespace>/</robotNamespace>

File: hector_tracked_vehicles_description/urdf/tracked_wheel.urdf.xacro (robot description, xacro)
@@ -7,8 +7,6 @@
     <!-- Properties (Constants) -->
     <xacro:property name="M_PI" value="3.14159" />
-    <xacro:property name="wheel_radius" value="0.063" />
-    <xacro:property name="wheel_size_y" value="0.05" />
-    <xacro:property name="wheel_offset_x" value="0.16" />
-    <xacro:property name="wheel_offset_y" value="0.155" />
+    <!--<xacro:property name="wheel_radius" value="0.185" />-->
+    <!--<xacro:property name="wheel_size_y" value="0.0824" />-->
      <!-- half of wheel width + half of socket width + gap -->
     <xacro:property name="wheel_offset_z" value="-0.112" />
@@ -26,5 +24,5 @@
         <link name="${prefix}_wheel_link">
             <inertial>
-                <mass value="0.2" />
+                <mass value="0.01" />
                 <origin xyz=" 0 0 0 " />
                 <inertia  ixx="0.00012411765597" ixy="0.0" ixz="0.0"
@@ -32,5 +30,5 @@
                           izz="0.00011763977943" />
             </inertial>
-            <visual>
+<!--            <visual>
                 <origin xyz="0 0 0" rpy="${-M_PI/2} 0 0" />
                 <geometry>
@@ -40,5 +38,5 @@
                     <color rgba="0.3 0.3 0.3 1"/>
                 </material>
-            </visual>
+            </visual>-->
             <collision>
                 <origin xyz="0 0 0" rpy="${-M_PI/2} 0 0" />
@@ -46,12 +44,15 @@
                     <cylinder radius="${wheel_radius}" length="${wheel_size_y}" />
                 </geometry>
-                <material name="MTWheelColMat"/>
+                <!--<material name="MTWheelColMat"/>-->
             </collision>
         </link>
         <gazebo reference="${prefix}_wheel_link" >
-            <mu1 value="100.0" />
-            <mu2 value="100.0" />
-            <kp  value="100000.0" />
-            <kd  value="1.0" />
+            <mu1>0.9</mu1>
+            <mu2>0.9</mu2>
+            <kp>100000.0</kp>
+            <kd>1.0</kd>
+            <minDepth>0.001</minDepth>
+<!--            <fdir1>1 0 0</fdir1>-->
+            <maxContacts>1</maxContacts>
             <material>Gazebo/Grey</material>
         </gazebo>

Commit message: -Change parameters in effort to achieve proper steering

File: hector_tracked_vehicles_description/urdf/jasmine_ugv_base.urdf.xacro (robot description, xacro)
@@ -12,5 +12,5 @@
     <property name="wheel_radius" value="0.085" />
     <property name="wheel_length" value="0.02" />
-    <property name="wheel_size_y" value="0.05" />
+    <property name="wheel_size_y" value="0.0825" />
     <property name="total_width" value="0.297" />
     <!--    <property name="wheel_offset_y" value="${(total_width - wheel_size_y) / 2}" />-->
@@ -81,6 +81,6 @@
         <!--	Add wheels using the hlugv_wheel macro -->
         <tracked_wheel parent="base_link" prefix="left_0" offset_x= "0.21100" offset_y = "${wheel_offset_y}" offset_z = "${wheel_offset_z_from_base_link}" reflect="1" />
-        <tracked_wheel parent="base_link" prefix="left_1" offset_x= "0.0" offset_y = "${wheel_offset_y}" offset_z = "${wheel_offset_z_from_base_link}" reflect="1" />
-        <tracked_wheel parent="base_link" prefix="left_2" offset_x= "-0.21100" offset_y = "${wheel_offset_y}" offset_z = "${wheel_offset_z_from_base_link-0.01}" reflect="1" />
+        <tracked_wheel parent="base_link" prefix="left_1" offset_x= "0.0" offset_y = "${wheel_offset_y}" offset_z = "${wheel_offset_z_from_base_link-0.01}" reflect="1" />
+        <tracked_wheel parent="base_link" prefix="left_2" offset_x= "-0.21100" offset_y = "${wheel_offset_y}" offset_z = "${wheel_offset_z_from_base_link}" reflect="1" />
         <tracked_wheel parent="base_link" prefix="left_3" offset_x= "0.10550" offset_y = "${wheel_offset_y}" offset_z = "${wheel_offset_z_from_base_link}" reflect="1" />
         <tracked_wheel parent="base_link" prefix="left_4" offset_x= "-0.10550" offset_y = "${wheel_offset_y}" offset_z = "${wheel_offset_z_from_base_link}" reflect="1" />
@@ -99,5 +99,5 @@
                 <wheelSeparation>${wheel_offset_y*2}</wheelSeparation>
                 <wheelDiameter>${wheel_radius*2}</wheelDiameter>
-                <torque>5000</torque>
+                <torque>50000</torque>
                 <interface:position name="position_iface_2"/>
                 <robotNamespace>/</robotNamespace>

File: hector_tracked_vehicles_description/urdf/tracked_wheel.urdf.xacro (robot description, xacro)
@@ -43,4 +43,5 @@
                 <geometry>
                     <cylinder radius="${wheel_radius}" length="${wheel_size_y}" />
+                    <!--<box size="1.0 0.5 0.1" />-->
                 </geometry>
                 <!--<material name="MTWheelColMat"/>-->
@@ -50,10 +51,11 @@
             <mu1>0.9</mu1>
             <mu2>0.9</mu2>
-            <kp>100000.0</kp>
-            <kd>1.0</kd>
+            <kp>1000000.0</kp>
+            <kd>10.0</kd>
             <minDepth>0.001</minDepth>
-<!--            <fdir1>1 0 0</fdir1>-->
             <maxContacts>1</maxContacts>
             <material>Gazebo/Grey</material>
+            <!--<fdir1>1 0 0</fdir1>-->
+            <!--<maxVel>1.0</maxVel>-->
         </gazebo>
         <transmission type="pr2_mechanism_model/SimpleTransmission" name="${prefix}_wheel_trans">

Commit message: jasmine ugv: Remove base_footprint, fix sdf parameter names, switch off tf publishing for multiwheel plugin

File: hector_tracked_vehicles_description/urdf/jasmine_ugv_base.urdf.xacro (robot description, xacro)
@@ -24,5 +24,5 @@
         <!-- base_footprint is a fictitious link(frame) that is on the ground right below base_link origin,
              navigation stack depends on this frame -->
-        <link name="base_footprint">
+<!--        <link name="base_footprint">
             <inertial>
                 <mass value="0.0001" />
@@ -41,10 +41,4 @@
                 </material>
             </visual>
-            <!--            <collision>
-                <origin xyz="0 0 ${base_size_z/2 + ground_clearance}" rpy="0 0 0" />
-                <geometry>
-                  <box size="0.001 0.001 0.001" />
-                </geometry>
-            </collision>-->
         </link>
         <joint name="base_footprint_joint" type="fixed">
@@ -52,5 +46,5 @@
             <parent link="base_footprint"/>
             <child link="base_link" />
-        </joint>
+        </joint>-->
         <!-- Links and Joints (i.e., the robot) -->
         <link name="base_link">
@@ -92,5 +86,4 @@
         <gazebo>
         <plugin name="diffdrive_plugin_multiwheel" filename="libdiffdrive_plugin_multi_wheel.so">
-<!--        <controller:diffdrive_plugin_6w name="differential_drive_controller" plugin="libdiffdrive_plugin_6w.so">-->
                 <alwaysOn>true</alwaysOn>
                 <updateRate>100.0</updateRate>
@@ -102,5 +95,8 @@
                 <interface:position name="position_iface_2"/>
                 <robotNamespace>/</robotNamespace>
-                <topicName>cmd_vel</topicName>
+                <robotBaseFrame>base_link</robotBaseFrame>
+                <commandTopic>/cmd_vel_raw</commandTopic>
+                <publishOdometryTf>0</publishOdometryTf>
+                <publishOdometryMsg>1</publishOdometryMsg>
         </plugin>
         <plugin name="p3d_base_controller" filename="libgazebo_ros_p3d.so">
