Commit message: hector_tracked_vehicles_description: Added missing xacro namespace prefix to XML tags
See http://wiki.ros.org/xacro#Deprecated_Syntax.

File: hector_tracked_vehicles_description/urdf/jasmine_ugv_base.urdf.xacro (robot description, xacro)
@@ -4,22 +4,22 @@
     xmlns:controller="http://playerstage.sourceforge.net/gazebo/xmlschema/#controller"
     xmlns:interface="http://playerstage.sourceforge.net/gazebo/xmlschema/#interface">
-    <include filename="$(find hector_tracked_vehicles_description)/urdf/tracked_wheel.urdf.xacro" />
+    <xacro:include filename="$(find hector_tracked_vehicles_description)/urdf/tracked_wheel.urdf.xacro" />
     <!-- Properties (Constants) -->
-    <property name="M_PI" value="3.14159"/>
-    <property name="base_size_x" value="0.380" />
-    <property name="base_size_y" value="0.12" />
-    <property name="base_size_z" value="0.085" />
-    <property name="wheel_radius_big" value="0.085" />
-    <property name="wheel_length" value="0.02" />
-    <property name="wheel_size_y" value="0.0825" />
-    <property name="total_width" value="0.297" />
-    <!--    <property name="wheel_offset_y" value="${(total_width - wheel_size_y) / 2}" />-->
-    <property name="wheel_offset_y" value="0.1697" />
-    <property name="wheel_offset_z_from_base_link" value="-0.0" />
-    <property name="ground_clearance" value="0.05" />
-    <property name="top_size_x" value="0.3937" />
-    <property name="top_size_y" value="0.3556" />
-    <property name="top_size_z" value="0.0020" />
-    <macro name="jasmine_ugv_macro">
+    <xacro:property name="M_PI" value="3.14159"/>
+    <xacro:property name="base_size_x" value="0.380" />
+    <xacro:property name="base_size_y" value="0.12" />
+    <xacro:property name="base_size_z" value="0.085" />
+    <xacro:property name="wheel_radius_big" value="0.085" />
+    <xacro:property name="wheel_length" value="0.02" />
+    <xacro:property name="wheel_size_y" value="0.0825" />
+    <xacro:property name="total_width" value="0.297" />
+    <!--    <xacro:property name="wheel_offset_y" value="${(total_width - wheel_size_y) / 2}" />-->
+    <xacro:property name="wheel_offset_y" value="0.1697" />
+    <xacro:property name="wheel_offset_z_from_base_link" value="-0.0" />
+    <xacro:property name="ground_clearance" value="0.05" />
+    <xacro:property name="top_size_x" value="0.3937" />
+    <xacro:property name="top_size_y" value="0.3556" />
+    <xacro:property name="top_size_z" value="0.0020" />
+    <xacro:macro name="jasmine_ugv_macro">
         <!-- base_footprint is a fictitious link(frame) that is on the ground right below base_link origin,
              navigation stack depends on this frame -->
@@ -74,14 +74,14 @@
         </link>
        <!--	Add wheels using the hlugv_wheel macro -->
-        <tracked_wheel parent="base_link" prefix="left_0" offset_x= "0.21100" offset_y = "${wheel_offset_y}" offset_z = "${wheel_offset_z_from_base_link}" reflect="1" wheel_radius="${wheel_radius_big}"/>
-        <tracked_wheel parent="base_link" prefix="left_1" offset_x= "0.0" offset_y = "${wheel_offset_y}" offset_z = "${wheel_offset_z_from_base_link-0.01}" reflect="1" wheel_radius="${wheel_radius_big}"/>
-        <tracked_wheel parent="base_link" prefix="left_2" offset_x= "-0.21100" offset_y = "${wheel_offset_y}" offset_z = "${wheel_offset_z_from_base_link}" reflect="1" wheel_radius="${wheel_radius_big}"/>
-        <tracked_wheel parent="base_link" prefix="left_3" offset_x= "0.10550" offset_y = "${wheel_offset_y}" offset_z = "${wheel_offset_z_from_base_link}" reflect="1" wheel_radius="${wheel_radius_big}"/>
-        <tracked_wheel parent="base_link" prefix="left_4" offset_x= "-0.10550" offset_y = "${wheel_offset_y}" offset_z = "${wheel_offset_z_from_base_link}" reflect="1" wheel_radius="${wheel_radius_big}"/>
-        <tracked_wheel parent="base_link" prefix="right_0" offset_x= "0.21100" offset_y = "-${wheel_offset_y}" offset_z = "${wheel_offset_z_from_base_link}" reflect="1" wheel_radius="${wheel_radius_big}"/>
-        <tracked_wheel parent="base_link" prefix="right_1" offset_x= "0.0" offset_y = "-${wheel_offset_y}" offset_z = "${wheel_offset_z_from_base_link-0.01}" reflect="1" wheel_radius="${wheel_radius_big}"/>
-        <tracked_wheel parent="base_link" prefix="right_2" offset_x= "-0.21100" offset_y = "-${wheel_offset_y}" offset_z = "${wheel_offset_z_from_base_link}" reflect="1" wheel_radius="${wheel_radius_big}"/>
-        <tracked_wheel parent="base_link" prefix="right_3" offset_x= "-0.10550" offset_y = "-${wheel_offset_y}" offset_z = "${wheel_offset_z_from_base_link}" reflect="1" wheel_radius="${wheel_radius_big}"/>
-        <tracked_wheel parent="base_link" prefix="right_4" offset_x= "0.10550" offset_y = "-${wheel_offset_y}" offset_z = "${wheel_offset_z_from_base_link}" reflect="1" wheel_radius="${wheel_radius_big}"/>
+        <xacro:tracked_wheel parent="base_link" prefix="left_0" offset_x= "0.21100" offset_y = "${wheel_offset_y}" offset_z = "${wheel_offset_z_from_base_link}" reflect="1" wheel_radius="${wheel_radius_big}"/>
+        <xacro:tracked_wheel parent="base_link" prefix="left_1" offset_x= "0.0" offset_y = "${wheel_offset_y}" offset_z = "${wheel_offset_z_from_base_link-0.01}" reflect="1" wheel_radius="${wheel_radius_big}"/>
+        <xacro:tracked_wheel parent="base_link" prefix="left_2" offset_x= "-0.21100" offset_y = "${wheel_offset_y}" offset_z = "${wheel_offset_z_from_base_link}" reflect="1" wheel_radius="${wheel_radius_big}"/>
+        <xacro:tracked_wheel parent="base_link" prefix="left_3" offset_x= "0.10550" offset_y = "${wheel_offset_y}" offset_z = "${wheel_offset_z_from_base_link}" reflect="1" wheel_radius="${wheel_radius_big}"/>
+        <xacro:tracked_wheel parent="base_link" prefix="left_4" offset_x= "-0.10550" offset_y = "${wheel_offset_y}" offset_z = "${wheel_offset_z_from_base_link}" reflect="1" wheel_radius="${wheel_radius_big}"/>
+        <xacro:tracked_wheel parent="base_link" prefix="right_0" offset_x= "0.21100" offset_y = "-${wheel_offset_y}" offset_z = "${wheel_offset_z_from_base_link}" reflect="1" wheel_radius="${wheel_radius_big}"/>
+        <xacro:tracked_wheel parent="base_link" prefix="right_1" offset_x= "0.0" offset_y = "-${wheel_offset_y}" offset_z = "${wheel_offset_z_from_base_link-0.01}" reflect="1" wheel_radius="${wheel_radius_big}"/>
+        <xacro:tracked_wheel parent="base_link" prefix="right_2" offset_x= "-0.21100" offset_y = "-${wheel_offset_y}" offset_z = "${wheel_offset_z_from_base_link}" reflect="1" wheel_radius="${wheel_radius_big}"/>
+        <xacro:tracked_wheel parent="base_link" prefix="right_3" offset_x= "-0.10550" offset_y = "-${wheel_offset_y}" offset_z = "${wheel_offset_z_from_base_link}" reflect="1" wheel_radius="${wheel_radius_big}"/>
+        <xacro:tracked_wheel parent="base_link" prefix="right_4" offset_x= "0.10550" offset_y = "-${wheel_offset_y}" offset_z = "${wheel_offset_z_from_base_link}" reflect="1" wheel_radius="${wheel_radius_big}"/>
         <gazebo>
         <plugin name="diffdrive_plugin_multiwheel" filename="libdiffdrive_plugin_multi_wheel.so">
@@ -148,4 +148,4 @@
             <material>HLUGV/Green</material>
         </gazebo>
-    </macro>
+    </xacro:macro>
 </robot>

File: hector_tracked_vehicles_description/urdf/jasmine_ugv_standalone.urdf.xacro (robot description, xacro)
@@ -5,5 +5,5 @@
     xmlns:interface="http://playerstage.sourceforge.net/gazebo/xmlschema/#interface">
     <!-- Included URDF Files -->
-    <include filename="$(find hector_tracked_vehicles_description)/urdf/jasmine_ugv_base.urdf.xacro" />
-    <jasmine_ugv_macro />
+    <xacro:include filename="$(find hector_tracked_vehicles_description)/urdf/jasmine_ugv_base.urdf.xacro" />
+    <xacro:jasmine_ugv_macro />
 </robot>

File: hector_tracked_vehicles_description/urdf/jasmine_ugv_vision_box.urdf.xacro (robot description, xacro)
@@ -9,5 +9,5 @@
     <xacro:include filename="$(find hector_components_description)/urdf/vision_box_common.urdf.xacro"/>
     <xacro:include filename="$(find hector_components_description)/urdf/vision_box_dimensions_hector2.urdf.xacro" />
-    <jasmine_ugv_macro />
+    <xacro:jasmine_ugv_macro />
     <xacro:vision_box parent="base_link" box_type="hector2">
       <origin xyz="-0.05 0 0.11" rpy="0 0 0"/>

File: hector_tracked_vehicles_description/urdf/obelix_2flipper_box.urdf.xacro (robot description, xacro)
@@ -4,13 +4,13 @@
   xmlns:controller="http://playerstage.sourceforge.net/gazebo/xmlschema/#controller"
   xmlns:interface="http://playerstage.sourceforge.net/gazebo/xmlschema/#interface">
-  <property name="flipper_base_mass" value="2.0"/>
-  <property name="flipper_x" value="0.3"/>
-  <property name="flipper_y" value="0.1"/>
-  <property name="flipper_z" value="0.15"/>
+  <xacro:property name="flipper_base_mass" value="2.0"/>
+  <xacro:property name="flipper_x" value="0.3"/>
+  <xacro:property name="flipper_y" value="0.1"/>
+  <xacro:property name="flipper_z" value="0.15"/>
   <!--
   Note macros below are exact copies of each with expection of the
   visual/collision tags.
   -->
-  <macro name="flipper_geom_macro_visual" params="front">
+  <xacro:macro name="flipper_geom_macro_visual" params="front">
     <visual>
       <material name="Grey" >
@@ -34,6 +34,6 @@
       </geometry>
     </visual>
-  </macro>
-  <macro name="flipper_geom_macro_collision" params="front">
+  </xacro:macro>
+  <xacro:macro name="flipper_geom_macro_collision" params="front">
     <collision>
       <origin xyz="0 0 0" rpy="${M_PI*0.5} 0 0" />
@@ -54,10 +54,10 @@
       </geometry>
     </collision>
-  </macro>
-  <macro name="obelix_flipper_macro" params="parent name front *origin">
+  </xacro:macro>
+  <xacro:macro name="obelix_flipper_macro" params="parent name front *origin">
     <!-- front is either 1 (for front flipper) or -1 (for back flipper) -->
     <!-- <joint name="${parent}_${name}_flipper_joint" type="fixed">   -->
     <joint name="${name}_flipper_joint" type="revolute">
-      <insert_block name="origin"/>
+      <xacro:insert_block name="origin"/>
       <axis xyz="0 1 0"/>
       <limit lower="${-90 * M_PI / 180}" upper="${90 * M_PI / 180}"
@@ -68,9 +68,9 @@
     <link name="left_${name}_flipper_base_link">
       <origin xyz="0 0 0" rpy="0 0 0" />
-      <inertial_cuboid_with_pose mass="3" x_length="${flipper_offset_wheel_axis_x}" y_length="${flipper_width}" z_length="${wheel_radius*2}" >
+      <xacro:inertial_cuboid_with_pose mass="3" x_length="${flipper_offset_wheel_axis_x}" y_length="${flipper_width}" z_length="${wheel_radius*2}" >
         <origin xyz="${front*flipper_offset_wheel_axis_x*0.5} 0 0" rpy="0 0 0" />
-      </inertial_cuboid_with_pose>
-      <flipper_geom_macro_visual front="${front}" />
-      <flipper_geom_macro_collision front="${front}" />
+      </xacro:inertial_cuboid_with_pose>
+      <xacro:flipper_geom_macro_visual front="${front}" />
+      <xacro:flipper_geom_macro_collision front="${front}" />
     </link>
     <joint name="right_${name}_flipper_joint" type="fixed">
@@ -81,9 +81,9 @@
     <link name="right_${name}_flipper_base_link">
       <origin xyz="0 0 0" rpy="0 0 0" />
-      <inertial_cuboid_with_pose mass="3" x_length="${flipper_offset_wheel_axis_x}" y_length="${flipper_width}" z_length="${wheel_radius*2}" >
+      <xacro:inertial_cuboid_with_pose mass="3" x_length="${flipper_offset_wheel_axis_x}" y_length="${flipper_width}" z_length="${wheel_radius*2}" >
         <origin xyz="${front*flipper_offset_wheel_axis_x*0.5} 0 0" rpy="0 0 0" />
-      </inertial_cuboid_with_pose>
-      <flipper_geom_macro_visual front="${front}" />
-      <flipper_geom_macro_collision front="${front}" />
+      </xacro:inertial_cuboid_with_pose>
+      <xacro:flipper_geom_macro_visual front="${front}" />
+      <xacro:flipper_geom_macro_collision front="${front}" />
     </link>
     <!--Needed for gazebo-->
@@ -118,4 +118,4 @@
       <maxContacts>1</maxContacts>
     </gazebo>
-  </macro>
+  </xacro:macro>
 </robot>

File: hector_tracked_vehicles_description/urdf/obelix_2flipper_wheel.urdf.xacro (robot description, xacro)
@@ -4,17 +4,17 @@
     xmlns:controller="http://playerstage.sourceforge.net/gazebo/xmlschema/#controller"
     xmlns:interface="http://playerstage.sourceforge.net/gazebo/xmlschema/#interface">
-  <property name="flipper_base_mass" value="2.0"/>
-  <property name="flipper_x" value="0.4"/>
-<property name="flipper_y" value="0.1"/>
-<property name="flipper_z" value="0.1"/>
-<property name="wheel_radius_first" value="0.093" />
-<property name="wheel_radius_second" value="0.09" />
-    <property name="wheel_radius_third" value="0.08" />
-<property name="wheel_intersect_flipper" value="${((flipper_x-2*wheel_radius_first-2*wheel_radius_second-2*wheel_radius_third)/2)}" />
-<property name="wheel_pos_second" value="${2*wheel_radius_first+wheel_intersect_flipper}" />
-    <macro name="obelix_flipper_wheels_macro" params="parent name front *origin">
+  <xacro:property name="flipper_base_mass" value="2.0"/>
+  <xacro:property name="flipper_x" value="0.4"/>
+<xacro:property name="flipper_y" value="0.1"/>
+<xacro:property name="flipper_z" value="0.1"/>
+<xacro:property name="wheel_radius_first" value="0.093" />
+<xacro:property name="wheel_radius_second" value="0.09" />
+    <xacro:property name="wheel_radius_third" value="0.08" />
+<xacro:property name="wheel_intersect_flipper" value="${((flipper_x-2*wheel_radius_first-2*wheel_radius_second-2*wheel_radius_third)/2)}" />
+<xacro:property name="wheel_pos_second" value="${2*wheel_radius_first+wheel_intersect_flipper}" />
+    <xacro:macro name="obelix_flipper_wheels_macro" params="parent name front *origin">
  <!-- front is either 1 (for front flipper) or -1 (for back flipper) -->
 <joint name="${parent}_${name}_flipper_joint" type="revolute">
-<insert_block name="origin"/>
+<xacro:insert_block name="origin"/>
       <axis xyz="0 1 0"/>
       <limit lower="${-90 * M_PI / 180}" upper="${90 * M_PI / 180}"
@@ -33,7 +33,7 @@
       <material>Gazebo/Green</material>
     </gazebo>
- <tracked_wheel parent="left_${name}_flipper_base_link" prefix="first_${name}_left" offset_x= "0" offset_y = "0" offset_z = "0" reflect="1" wheel_radius="${wheel_radius_first}"/>
- <tracked_wheel parent="left_${name}_flipper_base_link" prefix="second_${name}_left" offset_x= "${front*(2*wheel_radius_first+((flipper_x-2*wheel_radius_first-2*wheel_radius_second-2*wheel_radius_third)/2))}" offset_y = "0" offset_z = "0" reflect="1" wheel_radius="${wheel_radius_second}"/>
- <tracked_wheel parent="left_${name}_flipper_base_link" prefix="third_${name}_left" offset_x= "${front*(flipper_x-wheel_radius_third+((flipper_x-2*wheel_radius_first-2*wheel_radius_second-2*wheel_radius_third)/2))}" offset_y = "0" offset_z = "0" reflect="1" wheel_radius="${wheel_radius_second}"/>
+ <xacro:tracked_wheel parent="left_${name}_flipper_base_link" prefix="first_${name}_left" offset_x= "0" offset_y = "0" offset_z = "0" reflect="1" wheel_radius="${wheel_radius_first}"/>
+ <xacro:tracked_wheel parent="left_${name}_flipper_base_link" prefix="second_${name}_left" offset_x= "${front*(2*wheel_radius_first+((flipper_x-2*wheel_radius_first-2*wheel_radius_second-2*wheel_radius_third)/2))}" offset_y = "0" offset_z = "0" reflect="1" wheel_radius="${wheel_radius_second}"/>
+ <xacro:tracked_wheel parent="left_${name}_flipper_base_link" prefix="third_${name}_left" offset_x= "${front*(flipper_x-wheel_radius_third+((flipper_x-2*wheel_radius_first-2*wheel_radius_second-2*wheel_radius_third)/2))}" offset_y = "0" offset_z = "0" reflect="1" wheel_radius="${wheel_radius_second}"/>
 <joint name="right_${name}_flipper_joint" type="fixed">
       <origin xyz="0 ${-2*(base_size_y*0.5+wheel_offset_y+0.5*wheel_size_y)} 0" rpy="0 0 0" />
@@ -44,10 +44,10 @@
 <origin xyz="0 0 0" rpy="0 0 0" />
         </link>
-<tracked_wheel parent="right_${name}_flipper_base_link" prefix="first_${name}_right" offset_x= "0" offset_y = "0" offset_z = "0" reflect="1" wheel_radius="${wheel_radius_first}"/>
-<tracked_wheel parent="right_${name}_flipper_base_link" prefix="second_${name}_right" offset_x= "${front*(2*wheel_radius_first+((flipper_x-2*wheel_radius_first-2*wheel_radius_second-2*wheel_radius_third)/2))}" offset_y = "0" offset_z = "0" reflect="1" wheel_radius="${wheel_radius_second}"/>
-<tracked_wheel parent="right_${name}_flipper_base_link" prefix="third_${name}_right" offset_x= "${front*(flipper_x-wheel_radius_third+((flipper_x-2*wheel_radius_first-2*wheel_radius_second-2*wheel_radius_third)/2))}" offset_y = "0" offset_z = "0" reflect="1" wheel_radius="${wheel_radius_second}"/>
+<xacro:tracked_wheel parent="right_${name}_flipper_base_link" prefix="first_${name}_right" offset_x= "0" offset_y = "0" offset_z = "0" reflect="1" wheel_radius="${wheel_radius_first}"/>
+<xacro:tracked_wheel parent="right_${name}_flipper_base_link" prefix="second_${name}_right" offset_x= "${front*(2*wheel_radius_first+((flipper_x-2*wheel_radius_first-2*wheel_radius_second-2*wheel_radius_third)/2))}" offset_y = "0" offset_z = "0" reflect="1" wheel_radius="${wheel_radius_second}"/>
+<xacro:tracked_wheel parent="right_${name}_flipper_base_link" prefix="third_${name}_right" offset_x= "${front*(flipper_x-wheel_radius_third+((flipper_x-2*wheel_radius_first-2*wheel_radius_second-2*wheel_radius_third)/2))}" offset_y = "0" offset_z = "0" reflect="1" wheel_radius="${wheel_radius_second}"/>
 <gazebo reference="right_${name}_flipper_link">
       <material>Gazebo/Green</material>
     </gazebo>
-    </macro>
+    </xacro:macro>
 </robot>

File: hector_tracked_vehicles_description/urdf/obelix_flipper_box.urdf.xacro (robot description, xacro)
@@ -4,12 +4,12 @@
     xmlns:controller="http://playerstage.sourceforge.net/gazebo/xmlschema/#controller"
     xmlns:interface="http://playerstage.sourceforge.net/gazebo/xmlschema/#interface">
-  <property name="flipper_base_mass" value="2.0"/>
-  <property name="flipper_x" value="0.3"/>
-<property name="flipper_y" value="0.1"/>
-<property name="flipper_z" value="0.1"/>
-    <macro name="obelix_flipper_macro" params="parent name front *origin">
+  <xacro:property name="flipper_base_mass" value="2.0"/>
+  <xacro:property name="flipper_x" value="0.3"/>
+<xacro:property name="flipper_y" value="0.1"/>
+<xacro:property name="flipper_z" value="0.1"/>
+    <xacro:macro name="obelix_flipper_macro" params="parent name front *origin">
  <!-- front is either 1 (for front flipper) or -1 (for back flipper) -->
 <joint name="${name}_flipper_joint" type="revolute">
-<insert_block name="origin"/>
+<xacro:insert_block name="origin"/>
       <axis xyz="0 1 0"/>
       <limit lower="${-90 * M_PI / 180}" upper="${90 * M_PI / 180}"
@@ -50,4 +50,4 @@
       <material>Gazebo/Green</material>
     </gazebo>
-    </macro>
+    </xacro:macro>
 </robot>
