Commit message: hector_tracked_vehicles_description: Added missing xacro namespace prefix to XML tags
See http://wiki.ros.org/xacro#Deprecated_Syntax.

File: hector_tracked_vehicles_description/urdf/obelix_ugv_base.gazebo.xacro (robot description, xacro)
@@ -5,23 +5,23 @@
     xmlns:interface="http://playerstage.sourceforge.net/gazebo/xmlschema/#interface">
     <!-- Included URDF Files -->
-    <include filename="$(find hector_tracked_vehicles_description)/urdf/obelix_2flipper_wheel.urdf.xacro" />
+    <xacro:include filename="$(find hector_tracked_vehicles_description)/urdf/obelix_2flipper_wheel.urdf.xacro" />
   <!-- use for 2*2 flippers -->
-  <obelix_flipper_wheels_macro parent="base_link" name="front" front="1">
+  <xacro:obelix_flipper_wheels_macro parent="base_link" name="front" front="1">
     <origin xyz="${base_size_x*0.5} ${base_size_y*0.5+wheel_offset_y+0.5*wheel_size_y}  0 " rpy="0 0 0"/>
-  </obelix_flipper_wheels_macro >
-  <obelix_flipper_wheels_macro parent="base_link" name="back" front="-1">
+  </xacro:obelix_flipper_wheels_macro >
+  <xacro:obelix_flipper_wheels_macro parent="base_link" name="back" front="-1">
     <origin xyz="${-base_size_x*0.5} ${(base_size_y*0.5+wheel_offset_y+0.5*wheel_size_y)}  0  " rpy="0 0 0"/>
-  </obelix_flipper_wheels_macro >
+  </xacro:obelix_flipper_wheels_macro >
           <!--  Add wheels using the hlugv_wheel macro -->
-        <tracked_wheel parent="base_link" prefix="left_0" offset_x= "0.21100" offset_y = "${wheel_offset_y}" offset_z = "${wheel_offset_z_from_base_link}" reflect="1" wheel_radius="${wheel_radius_big}"/>
-        <tracked_wheel parent="base_link" prefix="left_1" offset_x= "0.0" offset_y = "${wheel_offset_y}" offset_z = "${wheel_offset_z_from_base_link-0.01}" reflect="1" wheel_radius="${wheel_radius_big}"/>
-        <tracked_wheel parent="base_link" prefix="left_2" offset_x= "-0.21100" offset_y = "${wheel_offset_y}" offset_z = "${wheel_offset_z_from_base_link}" reflect="1" wheel_radius="${wheel_radius_big}"/>
-        <tracked_wheel parent="base_link" prefix="left_3" offset_x= "0.10550" offset_y = "${wheel_offset_y}" offset_z = "${wheel_offset_z_from_base_link}" reflect="1" wheel_radius="${wheel_radius_big}"/>
-        <tracked_wheel parent="base_link" prefix="left_4" offset_x= "-0.10550" offset_y = "${wheel_offset_y}" offset_z = "${wheel_offset_z_from_base_link}" reflect="1" wheel_radius="${wheel_radius_big}"/>
-        <tracked_wheel parent="base_link" prefix="right_0" offset_x= "0.21100" offset_y = "-${wheel_offset_y}" offset_z = "${wheel_offset_z_from_base_link}" reflect="1" wheel_radius="${wheel_radius_big}"/>
-        <tracked_wheel parent="base_link" prefix="right_1" offset_x= "0.0" offset_y = "-${wheel_offset_y}" offset_z = "${wheel_offset_z_from_base_link-0.01}" reflect="1" wheel_radius="${wheel_radius_big}"/>
-        <tracked_wheel parent="base_link" prefix="right_2" offset_x= "-0.21100" offset_y = "-${wheel_offset_y}" offset_z = "${wheel_offset_z_from_base_link}" reflect="1" wheel_radius="${wheel_radius_big}"/>
-        <tracked_wheel parent="base_link" prefix="right_3" offset_x= "-0.10550" offset_y = "-${wheel_offset_y}" offset_z = "${wheel_offset_z_from_base_link}" reflect="1" wheel_radius="${wheel_radius_big}"/>
-        <tracked_wheel parent="base_link" prefix="right_4" offset_x= "0.10550" offset_y = "-${wheel_offset_y}" offset_z = "${wheel_offset_z_from_base_link}" reflect="1" wheel_radius="${wheel_radius_big}"/>
+        <xacro:tracked_wheel parent="base_link" prefix="left_0" offset_x= "0.21100" offset_y = "${wheel_offset_y}" offset_z = "${wheel_offset_z_from_base_link}" reflect="1" wheel_radius="${wheel_radius_big}"/>
+        <xacro:tracked_wheel parent="base_link" prefix="left_1" offset_x= "0.0" offset_y = "${wheel_offset_y}" offset_z = "${wheel_offset_z_from_base_link-0.01}" reflect="1" wheel_radius="${wheel_radius_big}"/>
+        <xacro:tracked_wheel parent="base_link" prefix="left_2" offset_x= "-0.21100" offset_y = "${wheel_offset_y}" offset_z = "${wheel_offset_z_from_base_link}" reflect="1" wheel_radius="${wheel_radius_big}"/>
+        <xacro:tracked_wheel parent="base_link" prefix="left_3" offset_x= "0.10550" offset_y = "${wheel_offset_y}" offset_z = "${wheel_offset_z_from_base_link}" reflect="1" wheel_radius="${wheel_radius_big}"/>
+        <xacro:tracked_wheel parent="base_link" prefix="left_4" offset_x= "-0.10550" offset_y = "${wheel_offset_y}" offset_z = "${wheel_offset_z_from_base_link}" reflect="1" wheel_radius="${wheel_radius_big}"/>
+        <xacro:tracked_wheel parent="base_link" prefix="right_0" offset_x= "0.21100" offset_y = "-${wheel_offset_y}" offset_z = "${wheel_offset_z_from_base_link}" reflect="1" wheel_radius="${wheel_radius_big}"/>
+        <xacro:tracked_wheel parent="base_link" prefix="right_1" offset_x= "0.0" offset_y = "-${wheel_offset_y}" offset_z = "${wheel_offset_z_from_base_link-0.01}" reflect="1" wheel_radius="${wheel_radius_big}"/>
+        <xacro:tracked_wheel parent="base_link" prefix="right_2" offset_x= "-0.21100" offset_y = "-${wheel_offset_y}" offset_z = "${wheel_offset_z_from_base_link}" reflect="1" wheel_radius="${wheel_radius_big}"/>
+        <xacro:tracked_wheel parent="base_link" prefix="right_3" offset_x= "-0.10550" offset_y = "-${wheel_offset_y}" offset_z = "${wheel_offset_z_from_base_link}" reflect="1" wheel_radius="${wheel_radius_big}"/>
+        <xacro:tracked_wheel parent="base_link" prefix="right_4" offset_x= "0.10550" offset_y = "-${wheel_offset_y}" offset_z = "${wheel_offset_z_from_base_link}" reflect="1" wheel_radius="${wheel_radius_big}"/>
         <gazebo>
         <plugin name="diffdrive_plugin_multiwheel" filename="libdiffdrive_plugin_multi_wheel.so">

File: hector_tracked_vehicles_description/urdf/obelix_ugv_base.urdf.xacro (robot description, xacro)
@@ -4,35 +4,35 @@
   xmlns:controller="http://playerstage.sourceforge.net/gazebo/xmlschema/#controller"
   xmlns:interface="http://playerstage.sourceforge.net/gazebo/xmlschema/#interface">
-  <include filename="$(find hector_xacro_tools)/urdf/inertia_tensors.urdf.xacro" />
-  <include filename="$(find hector_tracked_vehicles_description)/urdf/tracked_wheel.urdf.xacro" />
+  <xacro:include filename="$(find hector_xacro_tools)/urdf/inertia_tensors.urdf.xacro" />
+  <xacro:include filename="$(find hector_tracked_vehicles_description)/urdf/tracked_wheel.urdf.xacro" />
   <!-- Properties (Constants) -->
-  <property name="M_PI" value="3.14159"/>
-  <property name="base_link_size_x" value="0.52" />
-  <property name="base_link_size_y" value="0.18" />
-  <property name="base_link_size_z" value="0.118" />
-  <property name="wheel_radius_big" value="0.085" />
-  <property name="wheel_offset_x" value="${base_link_size_x*0.5 - 0.042}" />
-  <property name="wheel_offset_z" value="${base_link_size_z*0.5 - 0.065}" />
-  <property name="wheel_radius"   value="0.09" />
-  <property name="track_width"    value="0.1" />
-  <property name="track_offset_y"    value="0.155" />
-  <property name="flipper_width"    value="0.08" />
-  <property name="flipper_offset_y"    value="0.245" />
-  <property name="flipper_offset_wheel_axis_x"    value="0.225" />
-  <property name="wheel_length" value="0.02" />
-  <property name="wheel_size_y" value="0.0825" />
-  <property name="total_width" value="0.297" />
-  <!--    <property name="wheel_offset_y" value="${(total_width - wheel_size_y) / 2}" />-->
-  <property name="wheel_offset_y" value="0.1697" />
-  <property name="wheel_offset_z_from_base_link" value="-0.0" />
-  <property name="ground_clearance" value="0.05" />
-  <property name="top_size_x" value="0.3937" />
-  <property name="top_size_y" value="0.3556" />
-  <property name="top_size_z" value="0.0020" />
+  <xacro:property name="M_PI" value="3.14159"/>
+  <xacro:property name="base_link_size_x" value="0.52" />
+  <xacro:property name="base_link_size_y" value="0.18" />
+  <xacro:property name="base_link_size_z" value="0.118" />
+  <xacro:property name="wheel_radius_big" value="0.085" />
+  <xacro:property name="wheel_offset_x" value="${base_link_size_x*0.5 - 0.042}" />
+  <xacro:property name="wheel_offset_z" value="${base_link_size_z*0.5 - 0.065}" />
+  <xacro:property name="wheel_radius"   value="0.09" />
+  <xacro:property name="track_width"    value="0.1" />
+  <xacro:property name="track_offset_y"    value="0.155" />
+  <xacro:property name="flipper_width"    value="0.08" />
+  <xacro:property name="flipper_offset_y"    value="0.245" />
+  <xacro:property name="flipper_offset_wheel_axis_x"    value="0.225" />
+  <xacro:property name="wheel_length" value="0.02" />
+  <xacro:property name="wheel_size_y" value="0.0825" />
+  <xacro:property name="total_width" value="0.297" />
+  <!--    <xacro:property name="wheel_offset_y" value="${(total_width - wheel_size_y) / 2}" />-->
+  <xacro:property name="wheel_offset_y" value="0.1697" />
+  <xacro:property name="wheel_offset_z_from_base_link" value="-0.0" />
+  <xacro:property name="ground_clearance" value="0.05" />
+  <xacro:property name="top_size_x" value="0.3937" />
+  <xacro:property name="top_size_y" value="0.3556" />
+  <xacro:property name="top_size_z" value="0.0020" />
   <!--
   Note macros below are exact copies of each with expection of the
   visual/collision tags.
   -->
-  <macro name="track_geom_macro_visual" params="offset_y">
+  <xacro:macro name="track_geom_macro_visual" params="offset_y">
     <visual>
       <origin xyz="${wheel_offset_x} ${offset_y} ${wheel_offset_z}" rpy="${M_PI*0.5} 0 0" />
@@ -53,6 +53,6 @@
       </geometry>
     </visual>
-  </macro>
-  <macro name="track_geom_macro_collision" params="offset_y">
+  </xacro:macro>
+  <xacro:macro name="track_geom_macro_collision" params="offset_y">
     <collision>
       <origin xyz="${wheel_offset_x} ${offset_y} ${wheel_offset_z}" rpy="${M_PI*0.5} 0 0" />
@@ -73,11 +73,11 @@
       </geometry>
     </collision>
-  </macro>
-  <macro name="obelix_ugv_macro">
+  </xacro:macro>
+  <xacro:macro name="obelix_ugv_macro">
     <!-- Links and Joints (i.e., the robot) -->
     <link name="base_link">
-      <inertial_cuboid_with_pose mass="40" x_length="${base_link_size_x}" y_length="${base_link_size_y}" z_length="${base_link_size_z}" >
+      <xacro:inertial_cuboid_with_pose mass="40" x_length="${base_link_size_x}" y_length="${base_link_size_y}" z_length="${base_link_size_z}" >
         <origin xyz="0 0.0 0.0" rpy="0 0 0" />
-      </inertial_cuboid_with_pose>
+      </xacro:inertial_cuboid_with_pose>
       <visual>
         <origin xyz="0.0 0.0 0.0" rpy="0 0 0" />
@@ -92,6 +92,6 @@
         </material>
       </visual>
-      <track_geom_macro_visual offset_y="${ track_offset_y}"/>
-      <track_geom_macro_visual offset_y="${-track_offset_y}"/>
+      <xacro:track_geom_macro_visual offset_y="${ track_offset_y}"/>
+      <xacro:track_geom_macro_visual offset_y="${-track_offset_y}"/>
       <collision>
         <origin xyz="0.0 0.0 0.0" rpy="0 0 0" />
@@ -103,7 +103,7 @@
         </geometry>
       </collision>
-      <track_geom_macro_collision offset_y="${ track_offset_y}"/>
-      <track_geom_macro_collision offset_y="${-track_offset_y}"/>
+      <xacro:track_geom_macro_collision offset_y="${ track_offset_y}"/>
+      <xacro:track_geom_macro_collision offset_y="${-track_offset_y}"/>
     </link>
-  </macro>
+  </xacro:macro>
 </robot>

File: hector_tracked_vehicles_description/urdf/obelix_ugv_standalone.urdf.xacro (robot description, xacro)
@@ -5,14 +5,14 @@
        xmlns:interface="http://playerstage.sourceforge.net/gazebo/xmlschema/#interface">
   <!-- Included URDF Files -->
-  <include filename="$(find hector_tracked_vehicles_description)/urdf/obelix_ugv_base.urdf.xacro" />
-  <obelix_ugv_macro />
-  <include filename="$(find hector_tracked_vehicles_description)/urdf/obelix_2flipper_box.urdf.xacro" />
+  <xacro:include filename="$(find hector_tracked_vehicles_description)/urdf/obelix_ugv_base.urdf.xacro" />
+  <xacro:obelix_ugv_macro />
+  <xacro:include filename="$(find hector_tracked_vehicles_description)/urdf/obelix_2flipper_box.urdf.xacro" />
   <!-- use for 2*2 flippers -->
-  <obelix_flipper_macro parent="base_link" name="front" front="1">
+  <xacro:obelix_flipper_macro parent="base_link" name="front" front="1">
     <origin xyz="${wheel_offset_x}  ${flipper_offset_y}  0 " rpy="0 0 0"/>
-  </obelix_flipper_macro >
-  <obelix_flipper_macro parent="base_link" name="rear" front="-1">
+  </xacro:obelix_flipper_macro >
+  <xacro:obelix_flipper_macro parent="base_link" name="rear" front="-1">
     <origin xyz="${-wheel_offset_x}  ${flipper_offset_y}  0  " rpy="0 0 0"/>
-  </obelix_flipper_macro >
+  </xacro:obelix_flipper_macro >
   <gazebo reference="base_link">
     <!--<material>Gazebo/White</material>-->

File: hector_tracked_vehicles_description/urdf/obelix_ugv_standalone_gazebo.urdf.xacro (robot description, xacro)
@@ -5,6 +5,6 @@
     xmlns:interface="http://playerstage.sourceforge.net/gazebo/xmlschema/#interface">
     <!-- Included URDF Files -->
-    <include filename="$(find hector_tracked_vehicles_description)/urdf/obelix_ugv_base.urdf.xacro" />
-    <obelix_ugv_macro />
-    <include filename="$(find hector_tracked_vehicles_description)/urdf/obelix_ugv_base.gazebo.xacro" />
+    <xacro:include filename="$(find hector_tracked_vehicles_description)/urdf/obelix_ugv_base.urdf.xacro" />
+    <xacro:obelix_ugv_macro />
+    <xacro:include filename="$(find hector_tracked_vehicles_description)/urdf/obelix_ugv_base.gazebo.xacro" />
 </robot>

File: hector_tracked_vehicles_description/urdf/obelix_ugv_vision_box.urdf.xacro (robot description, xacro)
@@ -9,5 +9,5 @@
     <xacro:include filename="$(find hector_components_description)/urdf/vision_box_common.urdf.xacro"/>
     <xacro:include filename="$(find hector_components_description)/urdf/vision_box_dimensions_hector2.urdf.xacro" />
-    <!--<obelix_ugv_macro />-->
+    <!--<xacro:obelix_ugv_macro />-->
     <xacro:vision_box parent="base_link" box_type="hector2">
       <origin xyz="-0.05 0 0.11" rpy="0 0 0"/>

File: hector_tracked_vehicles_description/urdf/obelix_ugv_vision_box_small_arm.urdf.xacro (robot description, xacro)
@@ -10,5 +10,5 @@
     <xacro:include filename="$(find hector_components_description)/urdf/vision_box_dimensions_hector2.urdf.xacro" />
     <xacro:include filename="$(find hector_small_arm_description)/urdf/hector_arm_ax12_5dof.urdf.xacro" />
-  <!--<obelix_ugv_macro />-->
+  <!--<xacro:obelix_ugv_macro />-->
   <xacro:vision_box parent="base_link" box_type="hector2">
     <origin xyz="-0.05 0 0.11" rpy="0 0 0"/>

Commit message: Switch to use of forced based move plugin, update model accordingly

File: hector_tracked_vehicles_description/urdf/jasmine_ugv_base.urdf.xacro (robot description, xacro)
@@ -4,12 +4,14 @@
     xmlns:interface="http://www.ros.org/wiki/xacro">
     <xacro:include filename="$(find hector_tracked_vehicles_description)/urdf/tracked_wheel.urdf.xacro" />
+    <xacro:include filename="$(find hector_xacro_tools)/urdf/inertia_tensors.urdf.xacro" />
     <!-- Properties (Constants) -->
     <xacro:property name="M_PI" value="3.14159"/>
-    <xacro:property name="base_size_x" value="0.380" />
+    <xacro:property name="base_size_x" value="0.255" />
     <xacro:property name="base_size_y" value="0.12" />
-    <xacro:property name="base_size_z" value="0.085" />
-    <xacro:property name="wheel_radius_big" value="0.085" />
+    <xacro:property name="base_size_z" value="0.045" />
+    <xacro:property name="wheel_radius_big" value="0.080" />
     <xacro:property name="wheel_length" value="0.02" />
     <xacro:property name="wheel_size_y" value="0.0825" />
+    <xacro:property name="track_width" value="0.0825" />
     <xacro:property name="total_width" value="0.297" />
     <!--    <xacro:property name="wheel_offset_y" value="${(total_width - wheel_size_y) / 2}" />-->
@@ -17,4 +19,5 @@
     <xacro:property name="wheel_offset_z_from_base_link" value="-0.0" />
     <xacro:property name="ground_clearance" value="0.05" />
+    <xacro:property name="flipper_offset_x" value="-0.04" />
     <xacro:property name="top_size_x" value="0.3937" />
     <xacro:property name="top_size_y" value="0.3556" />
@@ -48,11 +51,7 @@
         <!-- Links and Joints (i.e., the robot) -->
         <link name="base_link">
-            <inertial>
-                <mass value="25.0" />
-                <origin xyz="0.0 0.0 0.0" rpy="0 0 0" />
-                <inertia ixx="0.005" ixy="0.0" ixz="0.0"
-                         iyy="0.005" iyz="0.0"
-                         izz="0.005" />
-            </inertial>
+          <xacro:inertial_cuboid_with_pose mass="25" x_length="${base_size_x*2}" y_length="${base_size_y*2}" z_length="${base_size_z*2}" >
+            <origin xyz="0 0 0 " rpy="0 0 0" />
+          </xacro:inertial_cuboid_with_pose>
             <visual>
                 <origin xyz="0.0 0.0 -0.085" rpy="0 0 0" />
@@ -68,9 +67,46 @@
                 <origin xyz="0.0 0.0 0.0" rpy="0 0 0" />
                 <geometry>
-                    <box size="${base_size_x} ${base_size_y} ${base_size_z}" />
+                    <box size="${base_size_x*2} ${base_size_y*2} ${base_size_z*2}" />
                 </geometry>
+            </collision>
+            <collision>
+              <origin xyz="${base_size_x+flipper_offset_x} ${-wheel_offset_y} 0.0" rpy="${M_PI/2} 0 0"/>
+              <geometry>
+                <cylinder length="${track_width}" radius="${wheel_radius_big}"/>
+              </geometry>
+            </collision>
+            <collision>
+              <origin xyz="${-base_size_x-flipper_offset_x}  ${-wheel_offset_y} 0.0" rpy="${M_PI/2} 0 0"/>
+              <geometry>
+                <cylinder length="${track_width}" radius="${wheel_radius_big}"/>
+              </geometry>
+            </collision>
+            <collision>
+              <origin xyz="0 ${-wheel_offset_y} 0.0" rpy="0 0 0"/>
+              <geometry>
+                <box size="${base_size_x*2+flipper_offset_x*2} ${track_width} ${wheel_radius_big*2}"/>
+              </geometry>
+            </collision>
+            <collision>
+              <origin xyz="${base_size_x+flipper_offset_x} ${wheel_offset_y} 0.0" rpy="${M_PI/2} 0 0"/>
+              <geometry>
+                <cylinder length="${track_width}" radius="${wheel_radius_big}"/>
+              </geometry>
+            </collision>
+            <collision>
+              <origin xyz="${-base_size_x-flipper_offset_x}  ${wheel_offset_y} 0.0" rpy="${M_PI/2} 0 0"/>
+              <geometry>
+                <cylinder length="${track_width}" radius="${wheel_radius_big}"/>
+              </geometry>
+            </collision>
+            <collision>
+              <origin xyz="0 ${wheel_offset_y} 0.0" rpy="0 0 0"/>
+              <geometry>
+                <box size="${base_size_x*2+flipper_offset_x*2} ${track_width} ${wheel_radius_big*2}"/>
+              </geometry>
             </collision>
         </link>
        <!--	Add wheels using the hlugv_wheel macro -->
+       <!-- Obsolete, replaced by force-based move macro
         <xacro:tracked_wheel parent="base_link" prefix="left_0" offset_x= "0.21100" offset_y = "${wheel_offset_y}" offset_z = "${wheel_offset_z_from_base_link}" reflect="1" wheel_radius="${wheel_radius_big}"/>
         <xacro:tracked_wheel parent="base_link" prefix="left_1" offset_x= "0.0" offset_y = "${wheel_offset_y}" offset_z = "${wheel_offset_z_from_base_link-0.01}" reflect="1" wheel_radius="${wheel_radius_big}"/>
@@ -99,4 +135,28 @@
                 <publishOdometryMsg>1</publishOdometryMsg>
         </plugin>
+        </gazebo>
+        -->
+    <gazebo reference="base_link">
+      <mu1>0.0</mu1>
+      <mu2>0.0</mu2>
+      <kp>1000000.0</kp>
+      <kd>100.0</kd>
+      <minDepth>0.001</minDepth>
+      <maxVel>1.0</maxVel>
+    </gazebo>
+    <gazebo>
+      <plugin name="force_based_move_controller" filename="libgazebo_ros_force_based_move.so">
+        <commandTopic>/cmd_vel_raw</commandTopic>
+        <odometryTopic>odom</odometryTopic>
+        <odometryFrame>odom</odometryFrame>
+        <odometryRate>20.0</odometryRate>
+        <robotBaseFrame>base_link</robotBaseFrame>
+        <yaw_velocity_p_gain>50</yaw_velocity_p_gain>
+        <x_velocity_p_gain>50</x_velocity_p_gain>
+        <y_velocity_p_gain>50</y_velocity_p_gain>
+        <publishOdometryTf>1</publishOdometryTf>
+      </plugin>
+    </gazebo>
+        <gazebo>
         <plugin name="p3d_base_controller" filename="libgazebo_ros_p3d.so">
           <alwaysOn>true</alwaysOn>
