Commit message: Move tracks and chassis to separate macro

File: hector_tracked_vehicles_description/urdf/jasmine_ugv_base.urdf.xacro (robot description, xacro)
@@ -4,4 +4,5 @@
     xmlns:interface="http://ros.org/wiki/xacro">
     <xacro:include filename="$(find hector_tracked_vehicles_description)/urdf/tracked_wheel.urdf.xacro" />
+    <xacro:include filename="$(find hector_tracked_vehicles_description)/urdf/jasmine_ugv_tracks.urdf.xacro" />
     <xacro:include filename="$(find hector_xacro_tools)/urdf/inertia_tensors.urdf.xacro" />
     <!-- Properties (Constants) -->
@@ -76,77 +77,7 @@
             </visual>
             -->
-            <collision>
-                <origin xyz="0.0 0.0 0.0" rpy="0 0 0" />
-                <geometry>
-                    <box size="${base_size_x*2} ${base_size_y*2} ${base_size_z*2}" />
-                </geometry>
-            </collision>
-            <collision>
-              <origin xyz="${base_size_x+flipper_offset_x} ${-wheel_offset_y} 0.0" rpy="${M_PI/2} 0 0"/>
-              <geometry>
-                <cylinder length="${track_width}" radius="${wheel_radius_big}"/>
-              </geometry>
-            </collision>
-            <collision>
-              <origin xyz="${-base_size_x-flipper_offset_x}  ${-wheel_offset_y} 0.0" rpy="${M_PI/2} 0 0"/>
-              <geometry>
-                <cylinder length="${track_width}" radius="${wheel_radius_big}"/>
-              </geometry>
-            </collision>
-            <collision>
-              <origin xyz="0 ${-wheel_offset_y} 0.0" rpy="0 0 0"/>
-              <geometry>
-                <box size="${base_size_x*2+flipper_offset_x*2} ${track_width} ${wheel_radius_big*2}"/>
-              </geometry>
-            </collision>
-            <collision>
-              <origin xyz="${base_size_x+flipper_offset_x} ${wheel_offset_y} 0.0" rpy="${M_PI/2} 0 0"/>
-              <geometry>
-                <cylinder length="${track_width}" radius="${wheel_radius_big}"/>
-              </geometry>
-            </collision>
-            <collision>
-              <origin xyz="${-base_size_x-flipper_offset_x}  ${wheel_offset_y} 0.0" rpy="${M_PI/2} 0 0"/>
-              <geometry>
-                <cylinder length="${track_width}" radius="${wheel_radius_big}"/>
-              </geometry>
-            </collision>
-            <collision>
-              <origin xyz="0 ${wheel_offset_y} 0.0" rpy="0 0 0"/>
-              <geometry>
-                <box size="${base_size_x*2+flipper_offset_x*2} ${track_width} ${wheel_radius_big*2}"/>
-              </geometry>
-            </collision>
+            <xacro:jasmine_ugv_tracks t_base_size_x="${base_size_x}"  t_base_size_y="${base_size_y}" t_base_size_z="${base_size_z}" t_flipper_offset_x="${flipper_offset_x}" t_wheel_offset_y="${wheel_offset_y}" t_wheel_radius_big="${wheel_radius_big}" t_track_width="${track_width}">
+            </xacro:jasmine_ugv_tracks>
         </link>
-       <!--	Add wheels using the hlugv_wheel macro -->
-       <!-- Obsolete, replaced by force-based move macro
-        <xacro:tracked_wheel parent="base_link" prefix="left_0" offset_x= "0.21100" offset_y = "${wheel_offset_y}" offset_z = "${wheel_offset_z_from_base_link}" reflect="1" wheel_radius="${wheel_radius_big}"/>
-        <xacro:tracked_wheel parent="base_link" prefix="left_1" offset_x= "0.0" offset_y = "${wheel_offset_y}" offset_z = "${wheel_offset_z_from_base_link-0.01}" reflect="1" wheel_radius="${wheel_radius_big}"/>
-        <xacro:tracked_wheel parent="base_link" prefix="left_2" offset_x= "-0.21100" offset_y = "${wheel_offset_y}" offset_z = "${wheel_offset_z_from_base_link}" reflect="1" wheel_radius="${wheel_radius_big}"/>
-        <xacro:tracked_wheel parent="base_link" prefix="left_3" offset_x= "0.10550" offset_y = "${wheel_offset_y}" offset_z = "${wheel_offset_z_from_base_link}" reflect="1" wheel_radius="${wheel_radius_big}"/>
-        <xacro:tracked_wheel parent="base_link" prefix="left_4" offset_x= "-0.10550" offset_y = "${wheel_offset_y}" offset_z = "${wheel_offset_z_from_base_link}" reflect="1" wheel_radius="${wheel_radius_big}"/>
-        <xacro:tracked_wheel parent="base_link" prefix="right_0" offset_x= "0.21100" offset_y = "-${wheel_offset_y}" offset_z = "${wheel_offset_z_from_base_link}" reflect="1" wheel_radius="${wheel_radius_big}"/>
-        <xacro:tracked_wheel parent="base_link" prefix="right_1" offset_x= "0.0" offset_y = "-${wheel_offset_y}" offset_z = "${wheel_offset_z_from_base_link-0.01}" reflect="1" wheel_radius="${wheel_radius_big}"/>
-        <xacro:tracked_wheel parent="base_link" prefix="right_2" offset_x= "-0.21100" offset_y = "-${wheel_offset_y}" offset_z = "${wheel_offset_z_from_base_link}" reflect="1" wheel_radius="${wheel_radius_big}"/>
-        <xacro:tracked_wheel parent="base_link" prefix="right_3" offset_x= "-0.10550" offset_y = "-${wheel_offset_y}" offset_z = "${wheel_offset_z_from_base_link}" reflect="1" wheel_radius="${wheel_radius_big}"/>
-        <xacro:tracked_wheel parent="base_link" prefix="right_4" offset_x= "0.10550" offset_y = "-${wheel_offset_y}" offset_z = "${wheel_offset_z_from_base_link}" reflect="1" wheel_radius="${wheel_radius_big}"/>
-        <gazebo>
-        <plugin name="diffdrive_plugin_multiwheel" filename="libdiffdrive_plugin_multi_wheel.so">
-                <alwaysOn>true</alwaysOn>
-                <updateRate>10.0</updateRate>
-                <leftJoints>left_0_wheel_joint left_1_wheel_joint left_2_wheel_joint left_3_wheel_joint left_4_wheel_joint</leftJoints>
-                <rightJoints>right_0_wheel_joint right_1_wheel_joint right_2_wheel_joint right_3_wheel_joint right_4_wheel_joint</rightJoints>
-                <wheelSeparation>${wheel_offset_y*2}</wheelSeparation>
-                <wheelDiameter>${wheel_radius_big*2}</wheelDiameter>
-                <torque>50000</torque>
-                <interface:position name="position_iface_2"/>
-                <robotNamespace>/</robotNamespace>
-                <robotBaseFrame>base_link</robotBaseFrame>
-                <commandTopic>/cmd_vel_raw</commandTopic>
-                <publishOdometryTf>0</publishOdometryTf>
-                <publishOdometryMsg>1</publishOdometryMsg>
-        </plugin>
-        </gazebo>
-        -->
     <gazebo reference="base_link">
       <mu1>0.0</mu1>
@@ -169,56 +100,27 @@
         <publishOdometryTf>1</publishOdometryTf>
       </plugin>
+      <plugin name="p3d_base_controller" filename="libgazebo_ros_p3d.so">
+        <alwaysOn>true</alwaysOn>
+        <updateRate>50.0</updateRate>
+        <bodyName>base_link</bodyName>
+        <topicName>ground_truth/state</topicName>
+        <gaussianNoise>0.01</gaussianNoise>
+        <frameName>world</frameName>
+        <xyzOffsets>0 0 0</xyzOffsets>
+        <rpyOffsets>0 0 0</rpyOffsets>
+      </plugin>
+      <plugin name="imu_controller" filename="libhector_gazebo_ros_imu.so">
+        <alwaysOn>true</alwaysOn>
+        <updateRate>50.0</updateRate>
+        <bodyName>base_link</bodyName>
+        <topicName>imu_quat</topicName>
+        <accelDrift>0.0 0.0 0.0</accelDrift>
+        <accelGaussianNoise>0.1 0.1 0.1</accelGaussianNoise>
+        <rateDrift>0.0 0.0 0.0</rateDrift>
+        <rateGaussianNoise>0.05 0.05 0.05</rateGaussianNoise>
+        <headingDrift>0.0</headingDrift>
+        <headingGaussianNoise>0.05</headingGaussianNoise>
+      </plugin>
     </gazebo>
-        <gazebo>
-        <plugin name="p3d_base_controller" filename="libgazebo_ros_p3d.so">
-          <alwaysOn>true</alwaysOn>
-          <updateRate>50.0</updateRate>
-          <bodyName>base_link</bodyName>
-          <topicName>ground_truth/state</topicName>
-          <gaussianNoise>0.01</gaussianNoise>
-          <frameName>world</frameName>
-          <xyzOffsets>0 0 0</xyzOffsets>
-          <rpyOffsets>0 0 0</rpyOffsets>
-        </plugin>
-        <plugin name="imu_controller" filename="libhector_gazebo_ros_imu.so">
-          <alwaysOn>true</alwaysOn>
-          <updateRate>50.0</updateRate>
-          <bodyName>base_link</bodyName>
-          <topicName>imu_quat</topicName>
-          <accelDrift>0.0 0.0 0.0</accelDrift>
-          <accelGaussianNoise>0.1 0.1 0.1</accelGaussianNoise>
-          <rateDrift>0.0 0.0 0.0</rateDrift>
-          <rateGaussianNoise>0.05 0.05 0.05</rateGaussianNoise>
-          <headingDrift>0.0</headingDrift>
-          <headingGaussianNoise>0.05</headingGaussianNoise>
-        </plugin>
-<!--        <plugin name="gazebo_ros_controller_manager" filename="libgazebo_ros_controller_manager.so">
-          <alwaysOn>true</alwaysOn>
-          <updateRate>1000.0</updateRate>
-        </plugin>-->
-           <!--
-            <canonicalBody>base_footprint</canonicalBody>
-            <controller:gazebo_ros_controller_manager name="gazebo_ros_controller_manager" plugin="libgazebo_ros_controller_manager.so">
-                <alwaysOn>true</alwaysOn>
-                <updateRate>100.0</updateRate>
-                <interface:audio name="gazebo_ros_controller_manager_dummy_iface" />
-            </controller:gazebo_ros_controller_manager>
-            <controller:gazebo_ros_imu name="imu_controller" plugin="libgazebo_ros_imu.so">
-                <alwaysOn>true</alwaysOn>
-                <updateRate>50</updateRate>
-                <bodyName>base_link</bodyName>
-                <topicName>hlugv_imu</topicName>
-                <gaussianNoise>0.1</gaussianNoise>
-                <xyzOffsets>0 0 0</xyzOffsets>
-                <rpyOffsets>0 0 0</rpyOffsets>
-                <interface:position name="imu_position"/>
-            </controller:gazebo_ros_imu>
-            -->
-        </gazebo>
-        <!--
-        <gazebo reference="base_link">
-            <material>HLUGV/Green</material>
-        </gazebo>
-        -->
     </xacro:macro>
 </robot>

Commit message: Move box for sensor head filtering up

File: hector_tracked_vehicles_description/urdf/jasmine_ugv_base.urdf.xacro (robot description, xacro)
@@ -87,5 +87,5 @@
               </xacro:jasmine_ugv_tracks>
               <collision>
-                <origin xyz="0.2 0.04 0.13" rpy="0 0 0" />
+                <origin xyz="0.2 0.04 0.15" rpy="0 0 0" />
                 <geometry>
                     <box size="${0.1} ${0.2} ${0.15}" />

Commit message: Further updates for self filter URDF setup

File: hector_tracked_vehicles_description/urdf/jasmine_ugv_base.urdf.xacro (robot description, xacro)
@@ -100,5 +100,4 @@
             <xacro:if value="$(arg add_raycast_self_filter_geom)">
               <xacro:jasmine_ugv_tracks t_base_size_x="${base_size_x}"  t_base_size_y="${base_size_y}" t_base_size_z="${base_size_z}" t_flipper_offset_x="${flipper_offset_x}" t_wheel_offset_y="${wheel_offset_y}" t_wheel_radius_big="${wheel_radius_big*1.3}" t_track_width="${track_width}">
-                  <xacro:arg name="use_cylinder_geoms" default="$(arg add_containment_self_filter_geom)"/>
               </xacro:jasmine_ugv_tracks>
             </xacro:if>

File: hector_tracked_vehicles_description/urdf/jasmine_ugv_tracks.urdf.xacro (robot description, xacro)
@@ -6,11 +6,24 @@
     <xacro:macro name="jasmine_ugv_tracks" params="t_base_size_x t_base_size_y t_base_size_z t_flipper_offset_x t_wheel_offset_y t_wheel_radius_big t_track_width">
             <xacro:arg name="add_raycast_self_filter_geom" default="false"/>
+            <xacro:arg name="add_containment_self_filter_geom" default="false"/>
             <xacro:unless value="$(arg add_raycast_self_filter_geom)">
-              <collision>
-                <origin xyz="0.0 0.0 0.0" rpy="0 0 0" />
-                <geometry>
-                  <box size="${t_base_size_x*2} ${t_base_size_y*2} ${t_base_size_z*2}" />
-                </geometry>
-              </collision>
+              <!--Make base geom larger for containment filter-->
+              <xacro:unless value="$(arg add_containment_self_filter_geom)">
+                <collision>
+                  <origin xyz="0.0 0.0 0.0" rpy="0 0 0" />
+                  <geometry>
+                    <box size="${t_base_size_x*2} ${t_base_size_y*2} ${t_base_size_z*2}" />
+                  </geometry>
+                </collision>
+              </xacro:unless>
+              <xacro:if value="$(arg add_containment_self_filter_geom)">
+                <collision>
+                  <origin xyz="0.0 0.0 ${t_base_size_z*2}" rpy="0 0 0" />
+                  <geometry>
+                    <box size="${t_base_size_x*2} ${t_base_size_y*2} ${t_base_size_z*4}" />
+                  </geometry>
+                </collision>
+              </xacro:if>
+              <!--/Make base geom larger for containment filter-->
               <collision>
                 <origin xyz="0 ${-t_wheel_offset_y} 0.0" rpy="0 0 0"/>
