Commit message: used new chassis and track macros

File: hector_tracked_vehicles_description/urdf/jasmine_ugv_base.urdf.xacro (robot description, xacro)
@@ -15,42 +15,10 @@
     <xacro:property name="wheel_size_y" value="0.0825" />
     <xacro:property name="track_width" value="0.0825" />
-    <xacro:property name="total_width" value="0.297" />
-    <!--    <xacro:property name="wheel_offset_y" value="${(total_width - wheel_size_y) / 2}" />-->
     <xacro:property name="wheel_offset_y" value="0.1697" />
-    <xacro:property name="wheel_offset_z_from_base_link" value="-0.0" />
-    <xacro:property name="ground_clearance" value="0.05" />
     <xacro:property name="flipper_offset_x" value="-0.04" />
-    <xacro:property name="top_size_x" value="0.3937" />
-    <xacro:property name="top_size_y" value="0.3556" />
-    <xacro:property name="top_size_z" value="0.0020" />
     <xacro:macro name="jasmine_ugv_macro">
         <xacro:arg name="add_default_geom" default="true"/>
         <xacro:arg name="add_containment_self_filter_geom" default="false"/>
         <xacro:arg name="add_raycast_self_filter_geom" default="false"/>
-        <!-- base_footprint is a fictitious link(frame) that is on the ground right below base_link origin,
-             navigation stack depends on this frame -->
-<!--        <link name="base_footprint">
-            <inertial>
-                <mass value="0.0001" />
-                <origin xyz="0 0 0" />
-                <inertia ixx="0.0001" ixy="0.0" ixz="0.0"
-                         iyy="0.0001" iyz="0.0"
-                         izz="0.0001" />
-            </inertial>
-            <visual>
-                <origin xyz="0 0 0" rpy="0 0 0" />
-                <geometry>
-                    <box size="0.001 0.001 0.001" />
-                </geometry>
-                <material name="Green" >
-                    <color rgba="0 0.8 0 1"/>
-                </material>
-            </visual>
-        </link>
-        <joint name="base_footprint_joint" type="fixed">
-            <origin xyz="0 0 ${base_size_z/2 + 0.051}" rpy="0 0 0" />
-            <parent link="base_footprint"/>
-            <child link="base_link" />
-        </joint>-->
         <!-- Links and Joints (i.e., the robot) -->
         <link name="base_link">
@@ -80,70 +48,70 @@
             </visual>
             -->
-            <xacro:if value="$(arg add_default_geom)">
+<!--            <xacro:if value="$(arg add_default_geom)">
               <xacro:jasmine_ugv_tracks t_base_size_x="${base_size_x}"  t_base_size_y="${base_size_y}" t_base_size_z="${base_size_z}" t_flipper_offset_x="${flipper_offset_x}" t_wheel_offset_y="${wheel_offset_y}" t_wheel_radius_big="${wheel_radius_big}" t_track_width="${track_width}">
               </xacro:jasmine_ugv_tracks>
-            </xacro:if>
-            <!--Make tracks larger for self filtering-->
-            <xacro:if value="$(arg add_containment_self_filter_geom)">
+            </xacro:if>-->
+            <!--Make tracks larger for containment self filtering-->
+<!--            <xacro:if value="$(arg add_containment_self_filter_geom)">
               <xacro:jasmine_ugv_tracks t_base_size_x="${base_size_x}"  t_base_size_y="${base_size_y}" t_base_size_z="${base_size_z}" t_flipper_offset_x="${flipper_offset_x}" t_wheel_offset_y="${wheel_offset_y}" t_wheel_radius_big="${wheel_radius_big*1.3}" t_track_width="${track_width}">
               </xacro:jasmine_ugv_tracks>
-              <!--
-              <collision>
-                <origin xyz="0.2 0.04 0.15" rpy="0 0 0" />
-                <geometry>
-                    <box size="${0.1} ${0.2} ${0.15}" />
-                </geometry>
-              </collision>
-              -->
-            </xacro:if>
-            <!--Make tracks larger for self filtering-->
-            <xacro:if value="$(arg add_raycast_self_filter_geom)">
+            </xacro:if>-->
+            <!--Make tracks larger for raycast self filtering-->
+<!--            <xacro:if value="$(arg add_raycast_self_filter_geom)">
               <xacro:jasmine_ugv_tracks t_base_size_x="${base_size_x}"  t_base_size_y="${base_size_y}" t_base_size_z="${base_size_z}" t_flipper_offset_x="${flipper_offset_x}" t_wheel_offset_y="${wheel_offset_y}" t_wheel_radius_big="${wheel_radius_big*1.3}" t_track_width="${track_width}">
               </xacro:jasmine_ugv_tracks>
-            </xacro:if>
+            </xacro:if>-->
+            <!-- Chassis geometry -->
+            <xacro:jasmine_ugv_chassis_geom t_base_size_x="${base_size_x}"  t_base_size_y="${base_size_y}" t_base_size_z="${base_size_z}"/>
         </link>
-    <gazebo reference="base_link">
-      <mu1>0.0</mu1>
-      <mu2>0.0</mu2>
-      <kp>1000000.0</kp>
-      <kd>100.0</kd>
-      <minDepth>0.001</minDepth>
-      <maxVel>1.0</maxVel>
-    </gazebo>
-    <gazebo>
-      <plugin name="force_based_move_controller" filename="libgazebo_ros_force_based_move.so">
-        <commandTopic>/cmd_vel_raw</commandTopic>
-        <odometryTopic>odom</odometryTopic>
-        <odometryFrame>odom</odometryFrame>
-        <odometryRate>20.0</odometryRate>
-        <robotBaseFrame>base_link</robotBaseFrame>
-        <yaw_velocity_p_gain>500</yaw_velocity_p_gain>
-        <x_velocity_p_gain>3000</x_velocity_p_gain>
-        <y_velocity_p_gain>3000</y_velocity_p_gain>
-        <publishOdometryTf>1</publishOdometryTf>
-      </plugin>
-      <plugin name="p3d_base_controller" filename="libgazebo_ros_p3d.so">
-        <alwaysOn>true</alwaysOn>
-        <updateRate>50.0</updateRate>
-        <bodyName>base_link</bodyName>
-        <topicName>ground_truth/state</topicName>
-        <gaussianNoise>0.01</gaussianNoise>
-        <frameName>world</frameName>
-        <xyzOffsets>0 0 0</xyzOffsets>
-        <rpyOffsets>0 0 0</rpyOffsets>
-      </plugin>
-      <plugin name="imu_controller" filename="libhector_gazebo_ros_imu.so">
-        <alwaysOn>true</alwaysOn>
-        <updateRate>50.0</updateRate>
-        <bodyName>base_link</bodyName>
-        <topicName>imu_quat</topicName>
-        <accelDrift>0.0 0.0 0.0</accelDrift>
-        <accelGaussianNoise>0.1 0.1 0.1</accelGaussianNoise>
-        <rateDrift>0.0 0.0 0.0</rateDrift>
-        <rateGaussianNoise>0.05 0.05 0.05</rateGaussianNoise>
-        <headingDrift>0.0</headingDrift>
-        <headingGaussianNoise>0.05</headingGaussianNoise>
-      </plugin>
-    </gazebo>
+        <xacro:jasmine_ugv_track_link name="left_flipper" parent="base_link" t_wheel_radius_big="${wheel_radius_big}" t_track_width="${track_width}" t_track_length="${base_size_x*2+flipper_offset_x*2}">
+          <origin xyz="0 ${wheel_offset_y} 0 " rpy="0 0 0" />
+        </xacro:jasmine_ugv_track_link>
+        <xacro:jasmine_ugv_track_link name="right_flipper" parent="base_link" t_wheel_radius_big="${wheel_radius_big}" t_track_width="${track_width}" t_track_length="${base_size_x*2+flipper_offset_x*2}">
+          <origin xyz="0 ${-wheel_offset_y} 0 " rpy="0 0 0" />
+        </xacro:jasmine_ugv_track_link>
+        <gazebo reference="base_link">
+          <mu1>0.0</mu1>
+          <mu2>0.0</mu2>
+          <kp>1000000.0</kp>
+          <kd>100.0</kd>
+          <minDepth>0.001</minDepth>
+          <maxVel>1.0</maxVel>
+        </gazebo>
+        <gazebo>
+          <plugin name="force_based_move_controller" filename="libgazebo_ros_force_based_move.so">
+            <commandTopic>/cmd_vel_raw</commandTopic>
+            <odometryTopic>odom</odometryTopic>
+            <odometryFrame>odom</odometryFrame>
+            <odometryRate>20.0</odometryRate>
+            <robotBaseFrame>base_link</robotBaseFrame>
+            <yaw_velocity_p_gain>500</yaw_velocity_p_gain>
+            <x_velocity_p_gain>3000</x_velocity_p_gain>
+            <y_velocity_p_gain>3000</y_velocity_p_gain>
+            <publishOdometryTf>1</publishOdometryTf>
+          </plugin>
+          <plugin name="p3d_base_controller" filename="libgazebo_ros_p3d.so">
+            <alwaysOn>true</alwaysOn>
+            <updateRate>50.0</updateRate>
+            <bodyName>base_link</bodyName>
+            <topicName>ground_truth/state</topicName>
+            <gaussianNoise>0.01</gaussianNoise>
+            <frameName>world</frameName>
+            <xyzOffsets>0 0 0</xyzOffsets>
+            <rpyOffsets>0 0 0</rpyOffsets>
+          </plugin>
+          <plugin name="imu_controller" filename="libhector_gazebo_ros_imu.so">
+            <alwaysOn>true</alwaysOn>
+            <updateRate>50.0</updateRate>
+            <bodyName>base_link</bodyName>
+            <topicName>imu_quat</topicName>
+            <accelDrift>0.0 0.0 0.0</accelDrift>
+            <accelGaussianNoise>0.1 0.1 0.1</accelGaussianNoise>
+            <rateDrift>0.0 0.0 0.0</rateDrift>
+            <rateGaussianNoise>0.05 0.05 0.05</rateGaussianNoise>
+            <headingDrift>0.0</headingDrift>
+            <headingGaussianNoise>0.05</headingGaussianNoise>
+          </plugin>
+        </gazebo>
     </xacro:macro>
 </robot>

File: hector_tracked_vehicles_description/urdf/jasmine_ugv_tracks.urdf.xacro (robot description, xacro)
@@ -5,29 +5,27 @@
     <xacro:property name="M_PI" value="3.14159"/>
     <xacro:macro name="jasmine_ugv_chassis_geom" params="t_base_size_x t_base_size_y t_base_size_z t_offset_z:=0">
+      <xacro:arg name="add_default_geom" default="true"/>
       <xacro:arg name="add_raycast_self_filter_geom" default="false"/>
       <xacro:arg name="add_containment_self_filter_geom" default="false"/>
-      <!-- Non-raycast -->
-      <xacro:unless value="$(arg add_raycast_self_filter_geom)">
-        <xacro:unless value="$(arg add_containment_self_filter_geom)">
-          <!-- Standard-->
-          <collision>
-            <origin xyz="0.0 0.0 ${t_offset_z}" rpy="0 0 0" />
-            <geometry>
-              <box size="${t_base_size_x*2} ${t_base_size_y*2} ${t_base_size_z*2}" />
-            </geometry>
-          </collision>
-        </xacro:unless>
-        <!--Make base geom larger for containment filter-->
-        <xacro:if value="$(arg add_containment_self_filter_geom)">
-          <!-- Containment self filtering-->
-          <collision>
-            <origin xyz="0.0 0.0 ${t_base_size_z*2+t_offset_z}" rpy="0 0 0" />
-            <geometry>
-              <box size="${t_base_size_x*2} ${t_base_size_y*2} ${t_base_size_z*4}" />
-            </geometry>
-          </collision>
-        </xacro:if>
-      </xacro:unless>
-      <!-- Chassis geometry for raycast self filter -->
+      <!-- Default geom-->
+      <xacro:if value="$(arg add_default_geom)">
+        <collision>
+          <origin xyz="0.0 0.0 ${t_offset_z}" rpy="0 0 0" />
+          <geometry>
+            <box size="${t_base_size_x*2} ${t_base_size_y*2} ${t_base_size_z*2}" />
+          </geometry>
+        </collision>
+      </xacro:if>
+      <!-- Containment self-filter geom -->
+      <xacro:if value="$(arg add_containment_self_filter_geom)">
+        <!-- Containment self filtering-->
+        <collision>
+          <origin xyz="0.0 0.0 ${t_base_size_z*2+t_offset_z}" rpy="0 0 0" />
+          <geometry>
+            <box size="${t_base_size_x*2} ${t_base_size_y*2} ${t_base_size_z*4}" />
+          </geometry>
+        </collision>
+      </xacro:if>
+      <!-- Raycast self-filter geom -->
       <!-- Does not use boxes as raycast filtering is broken as of 27.03.2019 -->
       <xacro:if value="$(arg add_raycast_self_filter_geom)">
@@ -47,4 +45,5 @@
     </xacro:macro>
     <xacro:macro name="jasmine_ugv_track_link" params="name parent t_wheel_radius_big t_track_width t_track_length *origin">
+      <xacro:arg name="add_default_geom" default="true"/>
       <xacro:arg name="add_raycast_self_filter_geom" default="false"/>
       <xacro:arg name="add_containment_self_filter_geom" default="false"/>
@@ -56,12 +55,10 @@
       <link name="${name}_link">
         <!-- TODO intertial -->
-        <inertial>
-          <origin xyz="0 0 0" rpy="0 0 0"/>
-          <mass value="2"/>
-          <inertia ixx="1.0" ixy="0.0" ixz="0.0" iyy="1.0" iyz="0.0" izz="1.0"/>
-        </inertial>
+        <xacro:inertial_cuboid_with_pose mass="2" x_length="${t_track_length}" y_length="${t_track_width}" z_length="${t_wheel_radius_big*2}" >
+          <origin xyz="0 0 0 " rpy="0 0 0" />
+        </xacro:inertial_cuboid_with_pose>
         <!-- Collision geom -->
-        <!-- Non-raycast Track -->
-        <xacro:unless value="$(arg add_raycast_self_filter_geom)">
+        <!-- Standard track geom -->
+        <xacro:if value="$(arg add_default_geom)">
           <collision>
             <origin xyz="0 0 0" rpy="0 0 0"/>
@@ -70,6 +67,6 @@
             </geometry>
           </collision>
-        </xacro:unless>
-        <!-- Track geometry for raycast self filter -->
+        </xacro:if>
+        <!-- Raycast self-filter track geom -->
         <!-- Does not use boxes as raycast filtering is broken as of 27.03.2019 -->
         <xacro:if value="$(arg add_raycast_self_filter_geom)">

Commit message: added padding for self-filtering, adjusted weight

File: hector_tracked_vehicles_description/urdf/jasmine_ugv_base.urdf.xacro (robot description, xacro)
@@ -23,5 +23,5 @@
         <!-- Links and Joints (i.e., the robot) -->
         <link name="base_link">
-          <xacro:inertial_cuboid_with_pose mass="25" x_length="${base_size_x*2}" y_length="${base_size_y*2}" z_length="${base_size_z*2}" >
+          <xacro:inertial_cuboid_with_pose mass="10" x_length="${base_size_x*2}" y_length="${base_size_y*2}" z_length="${base_size_z*2}" >
             <origin xyz="0 0 0 " rpy="0 0 0" />
           </xacro:inertial_cuboid_with_pose>
@@ -48,25 +48,11 @@
             </visual>
             -->
-<!--            <xacro:if value="$(arg add_default_geom)">
-              <xacro:jasmine_ugv_tracks t_base_size_x="${base_size_x}"  t_base_size_y="${base_size_y}" t_base_size_z="${base_size_z}" t_flipper_offset_x="${flipper_offset_x}" t_wheel_offset_y="${wheel_offset_y}" t_wheel_radius_big="${wheel_radius_big}" t_track_width="${track_width}">
-              </xacro:jasmine_ugv_tracks>
-            </xacro:if>-->
-            <!--Make tracks larger for containment self filtering-->
-<!--            <xacro:if value="$(arg add_containment_self_filter_geom)">
-              <xacro:jasmine_ugv_tracks t_base_size_x="${base_size_x}"  t_base_size_y="${base_size_y}" t_base_size_z="${base_size_z}" t_flipper_offset_x="${flipper_offset_x}" t_wheel_offset_y="${wheel_offset_y}" t_wheel_radius_big="${wheel_radius_big*1.3}" t_track_width="${track_width}">
-              </xacro:jasmine_ugv_tracks>
-            </xacro:if>-->
-            <!--Make tracks larger for raycast self filtering-->
-<!--            <xacro:if value="$(arg add_raycast_self_filter_geom)">
-              <xacro:jasmine_ugv_tracks t_base_size_x="${base_size_x}"  t_base_size_y="${base_size_y}" t_base_size_z="${base_size_z}" t_flipper_offset_x="${flipper_offset_x}" t_wheel_offset_y="${wheel_offset_y}" t_wheel_radius_big="${wheel_radius_big*1.3}" t_track_width="${track_width}">
-              </xacro:jasmine_ugv_tracks>
-            </xacro:if>-->
             <!-- Chassis geometry -->
             <xacro:jasmine_ugv_chassis_geom t_base_size_x="${base_size_x}"  t_base_size_y="${base_size_y}" t_base_size_z="${base_size_z}"/>
         </link>
-        <xacro:jasmine_ugv_track_link name="left_flipper" parent="base_link" t_wheel_radius_big="${wheel_radius_big}" t_track_width="${track_width}" t_track_length="${base_size_x*2+flipper_offset_x*2}">
+        <xacro:jasmine_ugv_track_link name="left_track" parent="base_link" t_wheel_radius_big="${wheel_radius_big}" t_track_width="${track_width}" t_track_length="${base_size_x*2+flipper_offset_x*2}">
           <origin xyz="0 ${wheel_offset_y} 0 " rpy="0 0 0" />
         </xacro:jasmine_ugv_track_link>
-        <xacro:jasmine_ugv_track_link name="right_flipper" parent="base_link" t_wheel_radius_big="${wheel_radius_big}" t_track_width="${track_width}" t_track_length="${base_size_x*2+flipper_offset_x*2}">
+        <xacro:jasmine_ugv_track_link name="right_track" parent="base_link" t_wheel_radius_big="${wheel_radius_big}" t_track_width="${track_width}" t_track_length="${base_size_x*2+flipper_offset_x*2}">
           <origin xyz="0 ${-wheel_offset_y} 0 " rpy="0 0 0" />
         </xacro:jasmine_ugv_track_link>

File: hector_tracked_vehicles_description/urdf/jasmine_ugv_tracks.urdf.xacro (robot description, xacro)
@@ -48,4 +48,13 @@
       <xacro:arg name="add_raycast_self_filter_geom" default="false"/>
       <xacro:arg name="add_containment_self_filter_geom" default="false"/>
+      <xacro:if value="$(arg add_default_geom)">
+        <xacro:property name="collision_factor" value="1.0" />
+      </xacro:if>
+      <xacro:if value="$(arg add_containment_self_filter_geom)">
+        <xacro:property name="collision_factor" value="1.3" />
+      </xacro:if>
+      <xacro:if value="$(arg add_raycast_self_filter_geom)">
+        <xacro:property name="collision_factor" value="1.3" />
+      </xacro:if>
       <joint name="${name}_fixed_joint" type="fixed">
         <xacro:insert_block name="origin"/>
@@ -54,15 +63,14 @@
       </joint>
       <link name="${name}_link">
-        <!-- TODO intertial -->
-        <xacro:inertial_cuboid_with_pose mass="2" x_length="${t_track_length}" y_length="${t_track_width}" z_length="${t_wheel_radius_big*2}" >
+        <xacro:inertial_cuboid_with_pose mass="5" x_length="${t_track_length}" y_length="${t_track_width}" z_length="${t_wheel_radius_big*2}" >
           <origin xyz="0 0 0 " rpy="0 0 0" />
         </xacro:inertial_cuboid_with_pose>
         <!-- Collision geom -->
         <!-- Standard track geom -->
-        <xacro:if value="$(arg add_default_geom)">
+        <xacro:if value="$(eval add_default_geom or add_containment_self_filter_geom)">
           <collision>
             <origin xyz="0 0 0" rpy="0 0 0"/>
             <geometry>
-              <box size="${t_track_length} ${t_track_width} ${t_wheel_radius_big*2}"/>
+              <box size="${t_track_length} ${t_track_width} ${collision_factor * t_wheel_radius_big*2}"/>
             </geometry>
           </collision>
@@ -74,5 +82,5 @@
             <origin xyz="0 0 0" rpy="0 ${M_PI*0.5} 0"/>
             <geometry>
-              <cylinder length="${t_track_length}" radius="${t_wheel_radius_big}"/>
+              <cylinder length="${t_track_length + 0.08}" radius="${collision_factor * t_wheel_radius_big}"/>
               <!--<box size="${t_base_size_x*2+t_flipper_offset_x*2} ${t_track_width} ${t_wheel_radius_big*2}"/>-->
             </geometry>
@@ -83,5 +91,5 @@
           <origin xyz="${t_track_length / 2.0} 0 0" rpy="${M_PI/2} 0 0"/>
           <geometry>
-            <cylinder length="${t_track_width}" radius="${t_wheel_radius_big}"/>
+            <cylinder length="${t_track_width}" radius="${collision_factor * t_wheel_radius_big}"/>
           </geometry>
         </collision>
@@ -90,5 +98,5 @@
           <origin xyz="${-t_track_length / 2.0} 0 0" rpy="${M_PI/2} 0 0"/>
           <geometry>
-            <cylinder length="${t_track_width}" radius="${t_wheel_radius_big}"/>
+            <cylinder length="${t_track_width}" radius="${collision_factor * t_wheel_radius_big}"/>
           </geometry>
         </collision>

Commit message: Added chassis_link, base_link is now empty

File: hector_tracked_vehicles_description/urdf/jasmine_ugv_base.urdf.xacro (robot description, xacro)
@@ -22,6 +22,10 @@
         <xacro:arg name="add_containment_self_filter_geom" default="false"/>
         <xacro:arg name="add_raycast_self_filter_geom" default="false"/>
-        <!-- Links and Joints (i.e., the robot) -->
-        <link name="base_link">
+        <link name="base_link"/>
+        <joint name="chassis_joint" type="fixed">
+          <parent link="base_link"/>
+          <child link="chassis_link"/>
+        </joint>
+        <link name="chassis_link">
           <xacro:inertial_cuboid_with_pose mass="10" x_length="${base_size_x*2}" y_length="${base_size_y*2}" z_length="${base_size_z*2}" >
             <origin xyz="0 0 0 " rpy="0 0 0" />
@@ -52,8 +56,8 @@
             <xacro:jasmine_ugv_chassis_geom t_base_size_x="${base_size_x}"  t_base_size_y="${base_size_y}" t_base_size_z="${base_size_z}"/>
         </link>
-        <xacro:jasmine_ugv_track_link name="left_track" parent="base_link" t_wheel_radius_big="${wheel_radius_big}" t_track_width="${track_width}" t_track_length="${base_size_x*2+flipper_offset_x*2}">
+        <xacro:jasmine_ugv_track_link name="left_track" parent="chassis_link" t_wheel_radius_big="${wheel_radius_big}" t_track_width="${track_width}" t_track_length="${base_size_x*2+flipper_offset_x*2}">
           <origin xyz="0 ${wheel_offset_y} 0 " rpy="0 0 0" />
         </xacro:jasmine_ugv_track_link>
-        <xacro:jasmine_ugv_track_link name="right_track" parent="base_link" t_wheel_radius_big="${wheel_radius_big}" t_track_width="${track_width}" t_track_length="${base_size_x*2+flipper_offset_x*2}">
+        <xacro:jasmine_ugv_track_link name="right_track" parent="chassis_link" t_wheel_radius_big="${wheel_radius_big}" t_track_width="${track_width}" t_track_length="${base_size_x*2+flipper_offset_x*2}">
           <origin xyz="0 ${-wheel_offset_y} 0 " rpy="0 0 0" />
         </xacro:jasmine_ugv_track_link>
