Commit message: added imu link

File: hector_tracked_vehicles_description/urdf/jasmine_2018_structure_addons.urdf.xacro (robot description, xacro)
@@ -25,4 +25,9 @@
       <child link="structure_addons_link"/>
     </joint>
+     <joint name="imu_link_joint" type="fixed">
+      <origin xyz="0 0 0.5" rpy="0 0 0"/>
+      <parent link="${parent}" />
+      <child link="imu_link"/>
+    </joint>
     <link name="structure_addons_link">
       <xacro:inertial_sphere mass="0.1" diameter="0.07"/>
@@ -233,4 +238,6 @@
         </material>
       </collision>
+    </link>
+    <link name="imu_link">
     </link>
     <gazebo reference="structure_addons_link">

Commit message: Switch to using non-box geoms as work-around for https://github.com/ros-planning/geometric_shapes/issues/86 Add macro use to generate different models for different filters

File: hector_tracked_vehicles_description/urdf/jasmine_2018_structure_addons.urdf.xacro (robot description, xacro)
@@ -19,5 +19,6 @@
   <xacro:property name="handle_height" value="0.016"/>
   <xacro:property name="handle_y" value="0.138"/>
-  <xacro:macro name="jasmine_2018_structure_addons_macro" params="parent *origin">
+  <xacro:macro name="jasmine_2018_structure_addons_macro" params="parent *origin alu_profile_collision_size_factor">
+    <xacro:arg name="add_containment_self_filter_geom" default="false"/>
     <joint name="structure_addon_joint" type="fixed">
       <xacro:insert_block name="origin"/>
@@ -117,4 +118,5 @@
       </visual>
       <!--Handles-->
+      <!--
       <visual>
         <origin xyz="0 ${ (computer_box_width/2+handle_width/2)} ${handle_y}" rpy="0 0 0"/>
@@ -135,5 +137,7 @@
         </material>
       </visual>
+      -->
       <!-- Computer box-->
+      <xacro:unless value="$(arg add_containment_self_filter_geom)">
       <collision>
         <origin xyz="0 0 ${computer_box_height/2}" rpy="0 0 0"/>
@@ -149,5 +153,6 @@
         <origin xyz="${ (computer_box_length/2-alu_profile_side_length/2)} ${ (computer_box_width/2-alu_profile_side_length/2)} ${computer_box_height/2 + top_protection_bottom/2}" rpy="0 0 0"/>
         <geometry>
-          <box size="${alu_profile_side_length} ${alu_profile_side_length} ${top_protection_bottom-computer_box_height}"/>
+          <!--<box size="${alu_profile_side_length} ${alu_profile_side_length} ${top_protection_bottom-computer_box_height}"/>-->
+          <cylinder length="${top_protection_bottom-computer_box_height}" radius="${alu_profile_side_length*0.5*alu_profile_collision_size_factor}"/>
         </geometry>
         <material name="Grey">
@@ -158,5 +163,6 @@
         <origin xyz="${-(computer_box_length/2-alu_profile_side_length/2)} ${ (computer_box_width/2-alu_profile_side_length/2)} ${computer_box_height/2 + top_protection_bottom/2}" rpy="0 0 0"/>
         <geometry>
-          <box size="${alu_profile_side_length} ${alu_profile_side_length} ${top_protection_bottom-computer_box_height}"/>
+          <!--<box size="${alu_profile_side_length} ${alu_profile_side_length} ${top_protection_bottom-computer_box_height}"/>-->
+          <cylinder length="${top_protection_bottom-computer_box_height}" radius="${alu_profile_side_length*0.5*alu_profile_collision_size_factor}"/>
         </geometry>
         <material name="Grey">
@@ -167,5 +173,6 @@
         <origin xyz="${-(computer_box_length/2-alu_profile_side_length/2)} ${-(computer_box_width/2-alu_profile_side_length/2)} ${computer_box_height/2 + top_protection_bottom/2}" rpy="0 0 0"/>
         <geometry>
-          <box size="${alu_profile_side_length} ${alu_profile_side_length} ${top_protection_bottom-computer_box_height}"/>
+          <!--<box size="${alu_profile_side_length} ${alu_profile_side_length} ${top_protection_bottom-computer_box_height}"/>-->
+          <cylinder length="${top_protection_bottom-computer_box_height}" radius="${alu_profile_side_length*0.5*alu_profile_collision_size_factor}"/>
         </geometry>
         <material name="Grey">
@@ -176,5 +183,6 @@
         <origin xyz="${ (computer_box_length/2-alu_profile_side_length/2)} ${-(computer_box_width/2-alu_profile_side_length/2)} ${computer_box_height/2 + top_protection_bottom/2}" rpy="0 0 0"/>
         <geometry>
-          <box size="${alu_profile_side_length} ${alu_profile_side_length} ${top_protection_bottom-computer_box_height}"/>
+          <!--<box size="${alu_profile_side_length} ${alu_profile_side_length} ${top_protection_bottom-computer_box_height}"/>-->
+          <cylinder length="${top_protection_bottom-computer_box_height}" radius="${alu_profile_side_length*0.5*alu_profile_collision_size_factor}"/>
         </geometry>
         <material name="Grey">
@@ -184,34 +192,38 @@
       <!--Top geom-->
       <collision>
-        <origin xyz="0 ${ (computer_box_width/2-alu_profile_side_length/2)} ${top_protection_bottom + alu_profile_side_length/2}" rpy="0 0 0"/>
-        <geometry>
-          <box size="${computer_box_length} ${alu_profile_side_length} ${alu_profile_side_length}"/>
-        </geometry>
-        <material name="Grey">
-          <color rgba="0.5 0.5 0.5 1"/>
-        </material>
-      </collision>
-      <collision>
-        <origin xyz="0 ${-(computer_box_width/2-alu_profile_side_length/2)} ${top_protection_bottom + alu_profile_side_length/2}" rpy="0 0 0"/>
-        <geometry>
-          <box size="${computer_box_length} ${alu_profile_side_length} ${alu_profile_side_length}"/>
-        </geometry>
-        <material name="Grey">
-          <color rgba="0.5 0.5 0.5 1"/>
-        </material>
-      </collision>
-      <collision>
-        <origin xyz="${ (computer_box_length/2-alu_profile_side_length/2)} 0 ${top_protection_bottom + alu_profile_side_length/2}" rpy="0 0 0"/>
-        <geometry>
-          <box size="${alu_profile_side_length} ${computer_box_width}  ${alu_profile_side_length}"/>
-        </geometry>
-        <material name="Grey">
-          <color rgba="0.5 0.5 0.5 1"/>
-        </material>
-      </collision>
-      <collision>
-        <origin xyz="${-(computer_box_length/2-alu_profile_side_length/2)} 0 ${top_protection_bottom + alu_profile_side_length/2}" rpy="0 0 0"/>
-        <geometry>
-          <box size="${alu_profile_side_length} ${computer_box_width}  ${alu_profile_side_length}"/>
+        <origin xyz="0 ${ (computer_box_width/2-alu_profile_side_length/2)} ${top_protection_bottom + alu_profile_side_length/2}" rpy="0 ${M_PI*0.5} 0"/>
+        <geometry>
+          <!--<box size="${computer_box_length} ${alu_profile_side_length} ${alu_profile_side_length}"/>-->
+          <cylinder length="${computer_box_length}" radius="${alu_profile_side_length*0.5*alu_profile_collision_size_factor}"/>
+        </geometry>
+        <material name="Grey">
+          <color rgba="0.5 0.5 0.5 1"/>
+        </material>
+      </collision>
+      <collision>
+        <origin xyz="0 ${-(computer_box_width/2-alu_profile_side_length/2)} ${top_protection_bottom + alu_profile_side_length/2}" rpy="0 ${M_PI*0.5} 0"/>
+        <geometry>
+          <!--<box size="${computer_box_length} ${alu_profile_side_length} ${alu_profile_side_length}"/>-->
+          <cylinder length="${computer_box_length}" radius="${alu_profile_side_length*0.5*alu_profile_collision_size_factor}"/>
+        </geometry>
+        <material name="Grey">
+          <color rgba="0.5 0.5 0.5 1"/>
+        </material>
+      </collision>
+      <collision>
+        <origin xyz="${ (computer_box_length/2-alu_profile_side_length/2)} 0 ${top_protection_bottom + alu_profile_side_length/2}" rpy="${M_PI*0.5} ${M_PI*0.5} 0"/>
+        <geometry>
+          <!--<box size="${alu_profile_side_length} ${computer_box_width}  ${alu_profile_side_length}"/>-->
+          <cylinder length="${computer_box_width}" radius="${alu_profile_side_length*0.5*alu_profile_collision_size_factor}"/>
+        </geometry>
+        <material name="Grey">
+          <color rgba="0.5 0.5 0.5 1"/>
+        </material>
+      </collision>
+      <collision>
+        <origin xyz="${-(computer_box_length/2-alu_profile_side_length/2)} 0 ${top_protection_bottom + alu_profile_side_length/2}" rpy="${M_PI*0.5} ${M_PI*0.5} 0"/>
+        <geometry>
+          <!--<box size="${alu_profile_side_length} ${computer_box_width}  ${alu_profile_side_length}"/>-->
+          <cylinder length="${computer_box_width}" radius="${alu_profile_side_length*0.5*alu_profile_collision_size_factor}"/>
         </geometry>
         <material name="Grey">
@@ -220,4 +232,5 @@
       </collision>
       <!--Handles-->
+      <!--
       <collision>
         <origin xyz="0 ${ (computer_box_width/2+handle_width/2)} ${handle_y}" rpy="0 0 0"/>
@@ -238,4 +251,17 @@
         </material>
       </collision>
+      -->
+      </xacro:unless>
+      <xacro:if value="$(arg add_containment_self_filter_geom)">
+      <collision>
+        <origin xyz="0 0 ${computer_box_height/2 + top_protection_bottom/2}" rpy="0 0 0"/>
+        <geometry>
+          <box size="${computer_box_length} ${computer_box_width} ${top_protection_bottom}"/>
+        </geometry>
+        <material name="Grey">
+          <color rgba="0.5 0.5 0.5 1"/>
+        </material>
+      </collision>
+      </xacro:if>
     </link>
     <link name="imu_link">

File: hector_tracked_vehicles_description/urdf/jasmine_2018_ugv.urdf.xacro (robot description, xacro)
@@ -12,7 +12,11 @@
     </xacro:property>
     -->
-    <xacro:arg name="add_self_filter_geom" default="false"/>
+    <xacro:arg name="add_default_geom" default="true"/>
+    <xacro:arg name="add_containment_self_filter_geom" default="false"/>
+    <xacro:arg name="add_raycast_self_filter_geom" default="false"/>
     <xacro:jasmine_ugv_macro>
-      <xacro:arg name="add_self_filter_geom_" default="$(arg add_self_filter_geom)"/>
+<!--      <xacro:arg name="add_default_geom" default="$(arg add_default_geom)"/>
+      <xacro:arg name="add_containment_self_filter_geom_" default="$(arg add_containment_self_filter_geom)"/>
+      <xacro:arg name="add_raycast_self_filter_geom" default="$(arg add_raycast_self_filter_geom)"/>-->
     </xacro:jasmine_ugv_macro>
     <!--
@@ -24,5 +28,5 @@
       <origin xyz="${+0.18 } 0.04 ${0.05}" rpy="0.0 -0.0 ${0.0}"/>
     </xacro:tracker_sensor_head_macro>
-    <xacro:jasmine_2018_structure_addons_macro parent="base_link">
+    <xacro:jasmine_2018_structure_addons_macro parent="base_link" alu_profile_collision_size_factor="1.5">
      <origin xyz="0 0 0" rpy="0 0 0"/>
     </xacro:jasmine_2018_structure_addons_macro>

File: hector_tracked_vehicles_description/urdf/jasmine_ugv_base.urdf.xacro (robot description, xacro)
@@ -25,5 +25,7 @@
     <xacro:property name="top_size_z" value="0.0020" />
     <xacro:macro name="jasmine_ugv_macro">
-        <xacro:arg name="add_self_filter_geom" default="false"/>
+        <xacro:arg name="add_default_geom" default="true"/>
+        <xacro:arg name="add_containment_self_filter_geom" default="false"/>
+        <xacro:arg name="add_raycast_self_filter_geom" default="false"/>
         <!-- base_footprint is a fictitious link(frame) that is on the ground right below base_link origin,
              navigation stack depends on this frame -->
@@ -78,12 +80,13 @@
             </visual>
             -->
-            <xacro:unless value="$(arg add_self_filter_geom)">
+            <xacro:if value="$(arg add_default_geom)">
               <xacro:jasmine_ugv_tracks t_base_size_x="${base_size_x}"  t_base_size_y="${base_size_y}" t_base_size_z="${base_size_z}" t_flipper_offset_x="${flipper_offset_x}" t_wheel_offset_y="${wheel_offset_y}" t_wheel_radius_big="${wheel_radius_big}" t_track_width="${track_width}">
               </xacro:jasmine_ugv_tracks>
-            </xacro:unless>
+            </xacro:if>
             <!--Make tracks larger for self filtering-->
-            <xacro:if value="$(arg add_self_filter_geom)">
+            <xacro:if value="$(arg add_containment_self_filter_geom)">
               <xacro:jasmine_ugv_tracks t_base_size_x="${base_size_x}"  t_base_size_y="${base_size_y}" t_base_size_z="${base_size_z}" t_flipper_offset_x="${flipper_offset_x}" t_wheel_offset_y="${wheel_offset_y}" t_wheel_radius_big="${wheel_radius_big*1.3}" t_track_width="${track_width}">
               </xacro:jasmine_ugv_tracks>
+              <!--
               <collision>
                 <origin xyz="0.2 0.04 0.15" rpy="0 0 0" />
@@ -92,4 +95,11 @@
                 </geometry>
               </collision>
+              -->
+            </xacro:if>
+            <!--Make tracks larger for self filtering-->
+            <xacro:if value="$(arg add_raycast_self_filter_geom)">
+              <xacro:jasmine_ugv_tracks t_base_size_x="${base_size_x}"  t_base_size_y="${base_size_y}" t_base_size_z="${base_size_z}" t_flipper_offset_x="${flipper_offset_x}" t_wheel_offset_y="${wheel_offset_y}" t_wheel_radius_big="${wheel_radius_big*1.3}" t_track_width="${track_width}">
+                  <xacro:arg name="use_cylinder_geoms" default="$(arg add_containment_self_filter_geom)"/>
+              </xacro:jasmine_ugv_tracks>
             </xacro:if>
         </link>

File: hector_tracked_vehicles_description/urdf/jasmine_ugv_tracks.urdf.xacro (robot description, xacro)
@@ -5,10 +5,53 @@
     <xacro:property name="M_PI" value="3.14159"/>
     <xacro:macro name="jasmine_ugv_tracks" params="t_base_size_x t_base_size_y t_base_size_z t_flipper_offset_x t_wheel_offset_y t_wheel_radius_big t_track_width">
-            <collision>
+            <xacro:arg name="add_raycast_self_filter_geom" default="false"/>
+            <xacro:unless value="$(arg add_raycast_self_filter_geom)">
+              <collision>
                 <origin xyz="0.0 0.0 0.0" rpy="0 0 0" />
                 <geometry>
-                    <box size="${t_base_size_x*2} ${t_base_size_y*2} ${t_base_size_z*2}" />
+                  <box size="${t_base_size_x*2} ${t_base_size_y*2} ${t_base_size_z*2}" />
                 </geometry>
-            </collision>
+              </collision>
+              <collision>
+                <origin xyz="0 ${-t_wheel_offset_y} 0.0" rpy="0 0 0"/>
+                <geometry>
+                  <box size="${t_base_size_x*2+t_flipper_offset_x*2} ${t_track_width} ${t_wheel_radius_big*2}"/>
+                </geometry>
+              </collision>
+              <collision>
+                <origin xyz="0 ${t_wheel_offset_y} 0.0" rpy="0 0 0"/>
+                <geometry>
+                  <box size="${t_base_size_x*2+t_flipper_offset_x*2} ${t_track_width} ${t_wheel_radius_big*2}"/>
+                </geometry>
+              </collision>
+            </xacro:unless>
+            <xacro:if value="$(arg add_raycast_self_filter_geom)">
+              <collision>
+                <origin xyz="0.0 0.07 0.0" rpy="0 ${M_PI*0.5} 0" />
+                <geometry>
+                  <cylinder length="${t_base_size_x*2}" radius="${t_base_size_z*1.6}"/>
+                </geometry>
+              </collision>
+              <collision>
+                <origin xyz="0.0 -0.07 0.0" rpy="0 ${M_PI*0.5} 0" />
+                <geometry>
+                  <cylinder length="${t_base_size_x*2}" radius="${t_base_size_z*1.6}"/>
+                </geometry>
+              </collision>
+              <collision>
+                <origin xyz="0 ${-t_wheel_offset_y} 0.0" rpy="0 ${M_PI*0.5} 0"/>
+                <geometry>
+                  <cylinder length="${t_base_size_x*2}" radius="${t_wheel_radius_big}"/>
+                  <!--<box size="${t_base_size_x*2+t_flipper_offset_x*2} ${t_track_width} ${t_wheel_radius_big*2}"/>-->
+                </geometry>
+              </collision>
+              <collision>
+                <origin xyz="0 ${t_wheel_offset_y} 0.0" rpy="0 ${M_PI*0.5} 0"/>
+                <geometry>
+                  <cylinder length="${t_base_size_x*2}" radius="${t_wheel_radius_big}"/>
+                  <!--<box size="${t_base_size_x*2+t_flipper_offset_x*2} ${t_track_width} ${t_wheel_radius_big*2}"/>-->
+                </geometry>
+              </collision>
+            </xacro:if>
             <collision>
               <origin xyz="${t_base_size_x+t_flipper_offset_x} ${-t_wheel_offset_y} 0.0" rpy="${M_PI/2} 0 0"/>
@@ -21,10 +64,4 @@
               <geometry>
                 <cylinder length="${t_track_width}" radius="${t_wheel_radius_big}"/>
-              </geometry>
-            </collision>
-            <collision>
-              <origin xyz="0 ${-t_wheel_offset_y} 0.0" rpy="0 0 0"/>
-              <geometry>
-                <box size="${t_base_size_x*2+t_flipper_offset_x*2} ${t_track_width} ${t_wheel_radius_big*2}"/>
               </geometry>
             </collision>
@@ -41,10 +78,4 @@
               </geometry>
             </collision>
-            <collision>
-              <origin xyz="0 ${t_wheel_offset_y} 0.0" rpy="0 0 0"/>
-              <geometry>
-                <box size="${t_base_size_x*2+t_flipper_offset_x*2} ${t_track_width} ${t_wheel_radius_big*2}"/>
-              </geometry>
-            </collision>
     </xacro:macro>
 </robot>

Commit message: Update self filter model

File: hector_tracked_vehicles_description/urdf/jasmine_2018_structure_addons.urdf.xacro (robot description, xacro)
@@ -263,4 +263,13 @@
         </material>
       </collision>
+      <collision>
+        <origin xyz="-0.18 0 ${computer_box_height/2+0.07}" rpy="0 0 0"/>
+        <geometry>
+          <box size="${computer_box_length} ${computer_box_width*1.95} ${0.3}"/>
+        </geometry>
+        <material name="Grey">
+          <color rgba="0.5 0.5 0.5 1"/>
+        </material>
+      </collision>
       </xacro:if>
     </link>

Commit message: Make name of structure addons param

File: hector_tracked_vehicles_description/urdf/jasmine_2018_structure_addons.urdf.xacro (robot description, xacro)
@@ -19,10 +19,10 @@
   <xacro:property name="handle_height" value="0.016"/>
   <xacro:property name="handle_y" value="0.138"/>
-  <xacro:macro name="jasmine_2018_structure_addons_macro" params="parent *origin alu_profile_collision_size_factor">
+  <xacro:macro name="jasmine_2018_structure_addons_macro" params="parent *origin alu_profile_collision_size_factor name:='autonomy_box'">
     <xacro:arg name="add_containment_self_filter_geom" default="false"/>
-    <joint name="structure_addon_joint" type="fixed">
+    <joint name="${name}_joint" type="fixed">
       <xacro:insert_block name="origin"/>
       <parent link="${parent}" />
-      <child link="structure_addons_link"/>
+      <child link="${name}_link"/>
     </joint>
      <joint name="imu_link_joint" type="fixed">
@@ -31,5 +31,5 @@
       <child link="imu_link"/>
     </joint>
-    <link name="structure_addons_link">
+    <link name="${name}_link">
       <xacro:inertial_sphere mass="0.1" diameter="0.07"/>
       <!-- Computer box-->

Commit message: fixed rotated imu and lidar

File: hector_tracked_vehicles_description/urdf/jasmine_2018_structure_addons.urdf.xacro (robot description, xacro)
@@ -27,5 +27,5 @@
     </joint>
      <joint name="imu_link_joint" type="fixed">
-      <origin xyz="0 0 0.5" rpy="0 0 0"/>
+      <origin xyz="0 0 0.5" rpy="0 0 ${M_PI/2}"/>
       <parent link="${parent}" />
       <child link="imu_link"/>

File: hector_tracked_vehicles_description/urdf/jasmine_2018_ugv.urdf.xacro (robot description, xacro)
@@ -38,5 +38,5 @@
     <xacro:spinning_sensor_mount_macro parent="base_link"  name="spin_lidar" scaling="0.001">
       <!-- the angles are due to ground calibration with tud tracker vlp16 -->
-      <origin xyz="${+0.0 } 0.0 ${0.27 + 0.0944673}" rpy="0.0 0.0 0"/>
+      <origin xyz="${+0.0 } 0.0 ${0.27 + 0.0944673}" rpy="0.0 0.0 ${M_PI}"/>
     </xacro:spinning_sensor_mount_macro>
     <xacro:realsense_d435_camera_comprehensive_params name="manipulation_rgbd_cam" parent="base_link" image_topic="image_rect_color" depth_points_topic="depth/points" min_range="0.3" max_range="9.0" update_rate="20">
