Commit message: Add nodelet manager for theta Add theta model to jasmine 2018

File: hector_tracked_vehicles_description/urdf/jasmine_2018_ugv.urdf.xacro (robot description, xacro)
@@ -21,3 +21,7 @@
       <origin xyz="${+0.0 } 0.0 ${0.15}" rpy="0.0052159 -0.00553223 ${M_PI*0.64}"/>
     </xacro:spinning_sensor_mount_macro>
+    <xacro:include filename="$(find hector_sensors_description)/urdf/ricoh_theta.urdf.xacro"/>
+    <xacro:ricoh_theta_camera name="ricoh_theta" cam_front_name="right" cam_rear_name="left" parent="base_link" ros_topic="image_raw" cam_info_topic="camera_info" update_rate="10" res_x="640" res_y="640" image_format="R8G8B8" fov="${M_PI}">
+      <origin xyz="0.1 0.0 0.6" rpy="0 0 0"/>
+    </xacro:ricoh_theta_camera>
 </robot>

Commit message: Add primitive-based version of current structure addons setup

File: hector_tracked_vehicles_description/urdf/jasmine_2018_ugv.urdf.xacro (robot description, xacro)
@@ -3,4 +3,5 @@
     <!-- Included URDF Files -->
     <xacro:include filename="$(find hector_tracked_vehicles_description)/urdf/jasmine_ugv_base.urdf.xacro" />
+    <xacro:include filename="$(find hector_tracked_vehicles_description)/urdf/jasmine_2018_structure_addons.urdf.xacro" />
     <xacro:include filename="$(find hector_components_description)/urdf/vlp16_mount.urdf.xacro.xml"/>
     <xacro:include filename="$(find hector_components_description)/urdf/tracker_sensor_head.urdf.xacro.xml"/>
@@ -17,7 +18,10 @@
       <origin xyz="${+0.18 } 0.0 ${0.05}" rpy="0.0 -0.0 ${0.0}"/>
     </xacro:tracker_sensor_head_macro>
+    <xacro:jasmine_2018_structure_addons_macro parent="base_link">
+     <origin xyz="0 0 0" rpy="0 0 0"/>
+    </xacro:jasmine_2018_structure_addons_macro>
     <xacro:spinning_sensor_mount_macro parent="base_link"  name="spin_lidar" scaling="0.001">
       <!-- the angles are due to ground calibration with tud tracker vlp16 -->
-      <origin xyz="${+0.0 } 0.0 ${0.15}" rpy="0.0052159 -0.00553223 ${M_PI*0.64}"/>
+      <origin xyz="${+0.0 } 0.0 ${0.27}" rpy="0.0052159 -0.00553223 ${M_PI*0.64}"/>
     </xacro:spinning_sensor_mount_macro>
     <xacro:include filename="$(find hector_sensors_description)/urdf/ricoh_theta.urdf.xacro"/>

File: hector_tracked_vehicles_description/urdf/jasmine_ugv_base.urdf.xacro (robot description, xacro)
@@ -64,4 +64,16 @@
                 </material>
             </visual>
+            <!--Optional visualization of detailed mesh-->
+            <!--
+            <visual>
+                <origin xyz="0.0 0.0 -0.049" rpy="0 0 0" />
+                <geometry>
+                    <mesh filename="package://hector_tracked_vehicles_description/meshes/jasmine_ugv/jasmine_2018_chassis_low_poly_velodyne.stl" scale="0.001 0.001 0.001"/>
+                </geometry>
+                <material name="Grey" >
+                    <color rgba="0.8 0.8 0.8 1"/>
+                </material>
+            </visual>
+            -->
             <collision>
                 <origin xyz="0.0 0.0 0.0" rpy="0 0 0" />

Commit message: Changed theta mount to actual mount location

File: hector_tracked_vehicles_description/urdf/jasmine_2018_ugv.urdf.xacro (robot description, xacro)
@@ -27,5 +27,5 @@
     <xacro:include filename="$(find hector_sensors_description)/urdf/ricoh_theta.urdf.xacro"/>
     <xacro:ricoh_theta_camera name="ricoh_theta" cam_front_name="right" cam_rear_name="left" parent="base_link" ros_topic="image_raw" cam_info_topic="camera_info" update_rate="10" res_x="640" res_y="640" image_format="R8G8B8" fov="${M_PI}">
-      <origin xyz="0.1 0.0 0.6" rpy="0 0 0"/>
+      <origin xyz="0.0 0.0 0.595" rpy="0 0 0"/>
     </xacro:ricoh_theta_camera>
 </robot>

Commit message: Remove vlp16 offset

File: hector_tracked_vehicles_description/urdf/jasmine_2018_ugv.urdf.xacro (robot description, xacro)
@@ -23,5 +23,5 @@
     <xacro:spinning_sensor_mount_macro parent="base_link"  name="spin_lidar" scaling="0.001">
       <!-- the angles are due to ground calibration with tud tracker vlp16 -->
-      <origin xyz="${+0.0 } 0.0 ${0.27}" rpy="0.0052159 -0.00553223 ${M_PI*0.64}"/>
+      <origin xyz="${+0.0 } 0.0 ${0.27}" rpy="0.0052159 -0.00553223 ${0.0}"/>
     </xacro:spinning_sensor_mount_macro>
     <xacro:include filename="$(find hector_sensors_description)/urdf/ricoh_theta.urdf.xacro"/>

Commit message: added spin lidar offset

File: hector_tracked_vehicles_description/urdf/jasmine_2018_ugv.urdf.xacro (robot description, xacro)
@@ -23,5 +23,5 @@
     <xacro:spinning_sensor_mount_macro parent="base_link"  name="spin_lidar" scaling="0.001">
       <!-- the angles are due to ground calibration with tud tracker vlp16 -->
-      <origin xyz="${+0.0 } 0.0 ${0.27}" rpy="0.0052159 -0.00553223 ${0.0}"/>
+      <origin xyz="${+0.0 } 0.0 ${0.27}" rpy="0.0052159 -0.00553223 -1.85"/>
     </xacro:spinning_sensor_mount_macro>
     <xacro:include filename="$(find hector_sensors_description)/urdf/ricoh_theta.urdf.xacro"/>

Commit message: changed offset again

File: hector_tracked_vehicles_description/urdf/jasmine_2018_ugv.urdf.xacro (robot description, xacro)
@@ -23,5 +23,5 @@
     <xacro:spinning_sensor_mount_macro parent="base_link"  name="spin_lidar" scaling="0.001">
       <!-- the angles are due to ground calibration with tud tracker vlp16 -->
-      <origin xyz="${+0.0 } 0.0 ${0.27}" rpy="0.0052159 -0.00553223 -1.85"/>
+      <origin xyz="${+0.0 } 0.0 ${0.27}" rpy="0.0052159 -0.00553223 1.85"/>
     </xacro:spinning_sensor_mount_macro>
     <xacro:include filename="$(find hector_sensors_description)/urdf/ricoh_theta.urdf.xacro"/>

Commit message: changed offset back to 0

File: hector_tracked_vehicles_description/urdf/jasmine_2018_ugv.urdf.xacro (robot description, xacro)
@@ -23,5 +23,5 @@
     <xacro:spinning_sensor_mount_macro parent="base_link"  name="spin_lidar" scaling="0.001">
       <!-- the angles are due to ground calibration with tud tracker vlp16 -->
-      <origin xyz="${+0.0 } 0.0 ${0.27}" rpy="0.0052159 -0.00553223 1.85"/>
+      <origin xyz="${+0.0 } 0.0 ${0.27}" rpy="0.0052159 -0.00553223 0"/>
     </xacro:spinning_sensor_mount_macro>
     <xacro:include filename="$(find hector_sensors_description)/urdf/ricoh_theta.urdf.xacro"/>

Commit message: Update calibration setup for jasmine

File: hector_tracked_vehicles_description/urdf/jasmine_2018_ugv.urdf.xacro (robot description, xacro)
@@ -6,7 +6,10 @@
     <xacro:include filename="$(find hector_components_description)/urdf/vlp16_mount.urdf.xacro.xml"/>
     <xacro:include filename="$(find hector_components_description)/urdf/tracker_sensor_head.urdf.xacro.xml"/>
+    <xacro:include filename="$(find hector_tracked_vehicles_description)/calibrations/spin_lidar_calibration.urdf.xacro"/>
+    <!--
     <xacro:property name="vlp16_calibration">
       <origin xyz="0.0 0.0 0.09446" rpy="${M_PI*0.250} 0.0 ${M_PI}"/>
     </xacro:property>
+    -->
     <xacro:arg name="add_self_filter_geom" default="false"/>
     <xacro:jasmine_ugv_macro>
@@ -26,5 +29,5 @@
     <xacro:spinning_sensor_mount_macro parent="base_link"  name="spin_lidar" scaling="0.001">
       <!-- the angles are due to ground calibration with tud tracker vlp16 -->
-      <origin xyz="${+0.0 } 0.0 ${0.27}" rpy="0.0052159 -0.00553223 0"/>
+      <origin xyz="${+0.0 } 0.0 ${0.27}" rpy="0.0 0.0 0"/>
     </xacro:spinning_sensor_mount_macro>
     <xacro:include filename="$(find hector_sensors_description)/urdf/ricoh_theta.urdf.xacro"/>

Commit message: Adjust cam position to reflect real robot setup

File: hector_tracked_vehicles_description/urdf/jasmine_2018_ugv.urdf.xacro (robot description, xacro)
@@ -22,5 +22,5 @@
     -->
     <xacro:tracker_sensor_head_macro parent="base_link">
-      <origin xyz="${+0.18 } 0.0 ${0.05}" rpy="0.0 -0.0 ${0.0}"/>
+      <origin xyz="${+0.18 } 0.04 ${0.05}" rpy="0.0 -0.0 ${0.0}"/>
     </xacro:tracker_sensor_head_macro>
     <xacro:jasmine_2018_structure_addons_macro parent="base_link">

Commit message: add an arm to jasmine

File: hector_tracked_vehicles_description/urdf/jasmine_2018_ugv.urdf.xacro (robot description, xacro)
@@ -7,4 +7,5 @@
     <xacro:include filename="$(find hector_components_description)/urdf/tracker_sensor_head.urdf.xacro.xml"/>
     <xacro:include filename="$(find hector_tracked_vehicles_description)/calibrations/spin_lidar_calibration.urdf.xacro"/>
+    <xacro:include filename="$(find hector_tracked_vehicles_description)/urdf/jasmine_2018_ugv_arm.urdf.xacro" />
     <!--
     <xacro:property name="vlp16_calibration">
@@ -21,4 +22,7 @@
     </xacro:vision_box>
     -->
+    <xacro:manipulator_arm_macro parent="base_link">
+      <origin xyz="-0.1618 -0.06875 0.01315" rpy="0.0 0.0 ${M_PI/2}" />
+    </xacro:manipulator_arm_macro>
     <xacro:tracker_sensor_head_macro parent="base_link">
       <origin xyz="${+0.18 } 0.04 ${0.05}" rpy="0.0 -0.0 ${0.0}"/>

Commit message: camera lidar calibration

File: hector_tracked_vehicles_description/urdf/jasmine_2018_ugv.urdf.xacro (robot description, xacro)
@@ -37,5 +37,5 @@
     <xacro:include filename="$(find hector_sensors_description)/urdf/ricoh_theta.urdf.xacro"/>
     <xacro:ricoh_theta_camera name="ricoh_theta" cam_front_name="right" cam_rear_name="left" parent="base_link" ros_topic="image_raw" cam_info_topic="camera_info" update_rate="10" res_x="640" res_y="640" image_format="R8G8B8" fov="${M_PI}">
-      <origin xyz="0.0 0.0 0.595" rpy="0 0 0"/>
+      <origin xyz="0.0 0.0 0.595" rpy="0.02 0 0"/>
     </xacro:ricoh_theta_camera>
 </robot>

Commit message: add the manipulation rgbd cam

File: hector_tracked_vehicles_description/urdf/jasmine_2018_ugv.urdf.xacro (robot description, xacro)
@@ -8,5 +8,6 @@
     <xacro:include filename="$(find hector_tracked_vehicles_description)/calibrations/spin_lidar_calibration.urdf.xacro"/>
     <xacro:include filename="$(find hector_tracked_vehicles_description)/urdf/jasmine_2018_ugv_arm.urdf.xacro" />
-    <!--
+    <xacro:include filename="$(find hector_sensors_description)/urdf/realsense_d435_camera.urdf.xacro"/>
+    <!--file
     <xacro:property name="vlp16_calibration">
       <origin xyz="0.0 0.0 0.09446" rpy="${M_PI*0.250} 0.0 ${M_PI}"/>
@@ -39,4 +40,7 @@
       <origin xyz="${+0.0 } 0.0 ${0.27 + 0.0944673}" rpy="0.0 0.0 0"/>
     </xacro:spinning_sensor_mount_macro>
+    <xacro:realsense_d435_camera_comprehensive_params name="manipulation_rgbd_cam" parent="base_link" image_topic="image_rect_color" depth_points_topic="depth/points" min_range="0.3" max_range="9.0" update_rate="20">
+      <origin xyz="-0.08 -0.005 0.454" rpy="0.0 ${25*M_PI/180.0} ${M_PI}"/>
+    </xacro:realsense_d435_camera_comprehensive_params>
     <xacro:include filename="$(find hector_sensors_description)/urdf/ricoh_theta.urdf.xacro"/>
     <xacro:ricoh_theta_camera name="ricoh_theta" cam_front_name="right" cam_rear_name="left" parent="base_link" ros_topic="image_raw" cam_info_topic="camera_info" update_rate="10" res_x="640" res_y="640" image_format="R8G8B8" fov="${M_PI}">

Commit message: added insta360

File: hector_tracked_vehicles_description/urdf/jasmine_2018_ugv.urdf.xacro (robot description, xacro)
@@ -43,7 +43,9 @@
       <origin xyz="-0.08 -0.005 0.454" rpy="0.0 ${25*M_PI/180.0} ${M_PI}"/>
     </xacro:realsense_d435_camera_comprehensive_params>
-    <xacro:include filename="$(find hector_sensors_description)/urdf/ricoh_theta.urdf.xacro"/>
-    <xacro:ricoh_theta_camera name="ricoh_theta" cam_front_name="right" cam_rear_name="left" parent="base_link" ros_topic="image_raw" cam_info_topic="camera_info" update_rate="10" res_x="640" res_y="640" image_format="R8G8B8" fov="${M_PI}">
-      <origin xyz="0.0 0.0 0.595" rpy="0.02 0 0"/>
-    </xacro:ricoh_theta_camera>
+    <xacro:include filename="$(find hector_sensors_description)/urdf/camera360.urdf.xacro"/>
+    <xacro:camera360 name="camera360" right_cam_name="right" left_cam_name="left" parent="base_link" ros_topic="image_raw" update_rate="10" res_x="1504" res_y="1504" image_format="R8G8B8" fov="${M_PI}">
+      <origin xyz="0.0 0.0 0.595" rpy="0.0 0 0"/>
+      <origin xyz="0.00009742  0.00061696 -0.03850784" rpy="3.1373499 -0.0021358 -3.1279404"/>
+<!--       <origin xyz="0.03850784 0 0" rpy="0 0 ${M_PI}"/> -->
+    </xacro:camera360>
 </robot>

Commit message: fix inertias and COMs

File: hector_tracked_vehicles_description/urdf/jasmine_2018_ugv.urdf.xacro (robot description, xacro)
@@ -41,5 +41,5 @@
     </xacro:spinning_sensor_mount_macro>
     <xacro:realsense_d435_camera_comprehensive_params name="manipulation_rgbd_cam" parent="base_link" image_topic="image_rect_color" depth_points_topic="depth/points" min_range="0.3" max_range="9.0" update_rate="20">
-      <origin xyz="-0.08 -0.005 0.454" rpy="0.0 ${25*M_PI/180.0} ${M_PI}"/>
+      <origin xyz="-0.08 -0.03 0.454" rpy="0.0 ${25*M_PI/180.0} ${M_PI}"/>
     </xacro:realsense_d435_camera_comprehensive_params>
     <xacro:include filename="$(find hector_sensors_description)/urdf/ricoh_theta.urdf.xacro"/>

File: hector_tracked_vehicles_description/urdf/jasmine_2018_ugv_arm.urdf.xacro (robot description, xacro)
@@ -35,9 +35,9 @@
       </collision>
       <inertial>
-        <origin xyz="-0.0129 0.00024 0.01759" rpy="0.0 0.0 0.0" />
+        <origin xyz="0.0129 0.00024 0.01759" rpy="0.0 0.0 0.0" />
         <mass value="0.082" />
-        <inertia ixx="48.546e-06"   ixy="-0.218e-06"    ixz="-0.416e-06"
-                                    iyy="25.118e-06"    iyz="17.510e-06"
-                                                        izz="4.077e-06" />
+        <inertia ixx="4.8545E-5"   ixy="-2.17E-7"    ixz="-4.16E-7"
+                                    iyy="2.5118E-5"    iyz="1.751E-5"
+                                                        izz="4.077E-6" />
       </inertial>
     </link>
@@ -67,9 +67,9 @@
       </collision>
       <inertial>
-        <origin xyz="0.00023 -0.00056 0.026" rpy="0.0 0.0 0.0" />
-        <mass value="0.088" />
-        <inertia ixx="13.346e-06"   ixy="0.224e-06"     ixz="0.323e-06"
-                                    iyy="7.757e-06"     iyz="0.438e-06"
-                                                        izz="14.284e-06" />
+        <origin xyz="0.0 -0.00064 0.03439" rpy="0.0 0.0 0.0" />
+        <mass value="0.176" />
+        <inertia ixx="-9.361E-6"   ixy="0.0"     ixz="0.0"
+                                    iyy="-1.1746E-5"     iyz="2.42E-7"
+                                                        izz="4.445E-6" />
       </inertial>
     </link>
@@ -117,9 +117,9 @@
       </collision>
       <inertial>
-        <origin xyz="0.00746 0.12016 0.00036" rpy="0.0 ${pi} 0.0" />
-        <mass value="0.136" />
-        <inertia ixx="267.630e-06"    ixy="25.927e-06"    ixz="-0.339e-06"
-                                      iyy="21.769e-06"    iyz="1.571e-06"
-                                                          izz="260.554e-06" />
+        <origin xyz="0.00692 0.18362 0.00028" rpy="0.0 0.0 0.0" />
+        <mass value="0.172" />
+        <inertia ixx="0.001359662"    ixy="7.8685E-5"    ixz="-2.1E-7"
+                                      iyy="3.584E-5"    iyz="3.533E-6"
+                                                          izz="0.00134845" />
       </inertial>
     </link>
@@ -167,9 +167,9 @@
       </collision>
       <inertial>
-        <origin xyz="-0.11166 0.00016 0.00038" rpy="0.0 0.0 0.0" />
-        <mass value="0.127" />
-        <inertia ixx="19.832e-06"   ixy="-0.793e-06"      ixz="-0.724e-06"
-                                    iyy="215.338e-06"     iyz="-0.221e-06"
-                                                          izz="207.743e-06" />
+        <origin xyz="-0.14163 -0.00294 0.00033" rpy="0.0 0.0 0.0" />
+        <mass value="0.147" />
+        <inertia ixx="2.3437E-5"   ixy="7.946E-6"      ixz="-1.54E-6"
+                                    iyy="0.00051703"     iyz="-2.64E-7"
+                                                          izz="0.000506424" />
       </inertial>
     </link>
@@ -211,9 +211,9 @@
       </collision>
       <inertial>
-        <origin xyz="-0.11166 0.00016 0.00038" rpy="0.0 0.0 0.0" />
-        <mass value="0.127" />
-        <inertia ixx="19.832e-06"   ixy="-0.793e-06"      ixz="-0.724e-06"
-                                    iyy="215.338e-06"     iyz="-0.221e-06"
-                                                          izz="207.743e-06" />
+        <origin xyz="-0.0475 -0.0002 0.00076" rpy="0.0 0.0 0.0" />
+        <mass value="0.09715" />
+        <inertia ixx="1e-6"   ixy="-0.000017591"      ixz="0.000000113"
+                                    iyy="1e-6"     iyz="-0.000000215"
+                                                          izz="1e-6" />
       </inertial>
     </link>
@@ -255,9 +255,9 @@
       </collision>
       <inertial>
-        <origin xyz="-0.11166 0.00016 0.00038" rpy="0.0 0.0 0.0" />
-        <mass value="0.127" />
-        <inertia ixx="19.832e-06"   ixy="-0.793e-06"      ixz="-0.724e-06"
-                                    iyy="215.338e-06"     iyz="-0.221e-06"
-                                                          izz="207.743e-06" />
+        <origin xyz="0.00003 0.00453 0.01105" rpy="0.0 0.0 0.0" />
+        <mass value="0.012667" />
+        <inertia ixx="0.000009292"   ixy="0.000000012"      ixz="0.000000008"
+                                    iyy="0.000003471"     iyz="0.000000621"
+                                                          izz="0.00000707" />
       </inertial>
     </link>
@@ -320,9 +320,9 @@
       </collision>
       <inertial>
-        <origin xyz="-0.04663 -0.00051 -0.00234" rpy="0.0 0.0 0.0" />
+        <origin xyz="0.00018 0.00265 0.03088" rpy="0.0 0.0 0.0" />
         <mass value="0.155" />
-        <inertia ixx="114.015e-06"    ixy="17.253e-06"    ixz="-1.650e-06"
-                                      iyy="70.718e-06"    iyz="0.750e-06"
-                                                          izz="141.557e-06" />
+        <inertia ixx="0.000058905"    ixy="-0.000001039"    ixz="-0.000015872"
+                                      iyy="0.000129197"    iyz="-0.000002084"
+                                                          izz="0.000106087" />
       </inertial>
     </link>
@@ -333,5 +333,5 @@
       <parent link="gripper_palm_link" />
       <child link="gripper_servo_link" />
-      <dynamics friction="0" damping="0" />
+      <dynamics friction="${0.01*joint_friction}" damping="${0.01*joint_damping}" />
     </joint>
     <link name="gripper_servo_link">
@@ -339,7 +339,7 @@
         <origin xyz="0.0 0.0 0.0" rpy="0.0 0.0 0.0" />
         <mass value="0.001" />
-        <inertia ixx="1.0e-05" ixy="0.0"     ixz="0.0"
-                              iyy="1.0e-05"  iyz="0.0"
-                                            izz="1.0e-05" />
+        <inertia ixx="1.0e-06" ixy="0.0"     ixz="0.0"
+                              iyy="1.0e-06"  iyz="0.0"
+                                            izz="1.0e-06" />
       </inertial>
       <visual>
@@ -421,9 +421,9 @@
       </collision>
       <inertial>
-        <origin xyz="0.01764 -0.04373 0.0" rpy="0.0 0.0 ${90 * pi / 180}" />
+        <origin xyz="0.00029 0.05281 0.05788" rpy="0.0 0.0 ${90 * pi / 180}" />
         <mass value="0.029" />
-        <inertia ixx="0.000025065339"   ixy="-0.000009627959" ixz="2.8255e-8"
-                                        iyy="0.000022245643"  iyz="5.37e-10"
-                                                              izz="0.000027220956" />
+        <inertia ixx="0.00006267"   ixy="-0.000021787" ixz="-0.000000201"
+                                        iyy="0.000044811"  iyz="0.00000006"
+                                                              izz="0.000065514" />
       </inertial>
     </link>
@@ -472,11 +472,12 @@
       </collision>
       <inertial>
-        <origin xyz="0.01764 -0.04373 0.0" rpy="0.0 0.0 ${90 * pi / 180}" />
+        <origin xyz="0.00029 0.05281 0.05788" rpy="0.0 0.0 ${90 * pi / 180}" />
         <mass value="0.029" />
-        <inertia ixx="0.000025065339" ixy="-0.000009627959" ixz="2.8255e-8"
-                                      iyy="0.000022245643"  iyz="5.37e-10"
-                                                            izz="0.000027220956" />
-      </inertial>
-    </link>
+        <inertia ixx="0.00006267"   ixy="-0.000021787" ixz="-0.000000201"
+                                        iyy="0.000044811"  iyz="0.00000006"
+                                                              izz="0.000065514" />
+      </inertial>
+    </link>
+    <xacro:generic_camera name="gripper_cam" parent="gripper_palm_link" ros_topic="/gripper_cam/image_raw" cam_info_topic="/gripper_cam/camera_info" update_rate="15" res_x="640" res_y="480" image_format="B8G8R8" hfov="60">
   </xacro:macro>
 </robot>

Commit message: updated height of the insta360

File: hector_tracked_vehicles_description/urdf/jasmine_2018_ugv.urdf.xacro (robot description, xacro)
@@ -45,5 +45,5 @@
     <xacro:include filename="$(find hector_sensors_description)/urdf/camera360.urdf.xacro"/>
     <xacro:camera360 name="camera360" right_cam_name="right" left_cam_name="left" parent="base_link" ros_topic="image_raw" update_rate="10" res_x="1504" res_y="1504" image_format="R8G8B8" fov="${M_PI}">
-      <origin xyz="0.0 0.0 0.595" rpy="0.0 0 0"/>
+      <origin xyz="0.0 0.0 0.58" rpy="0.0 0 0"/>
       <origin xyz="0.00009742  0.00061696 -0.03850784" rpy="3.1373499 -0.0021358 -3.1279404"/>
 <!--       <origin xyz="0.03850784 0 0" rpy="0 0 ${M_PI}"/> -->

Commit message: move D435

File: hector_tracked_vehicles_description/urdf/jasmine_2018_ugv.urdf.xacro (robot description, xacro)
@@ -41,5 +41,5 @@
     </xacro:spinning_sensor_mount_macro>
     <xacro:realsense_d435_camera_comprehensive_params name="manipulation_rgbd_cam" parent="base_link" image_topic="image_rect_color" depth_points_topic="depth/points" min_range="0.3" max_range="9.0" update_rate="20">
-      <origin xyz="-0.08 -0.005 0.454" rpy="0.0 ${25*M_PI/180.0} ${M_PI}"/>
+      <origin xyz="-0.08 -0.0085 0.454" rpy="0.0 ${25*M_PI/180.0} ${M_PI}"/>
     </xacro:realsense_d435_camera_comprehensive_params>
     <xacro:include filename="$(find hector_sensors_description)/urdf/camera360.urdf.xacro"/>
