Commit message: added dist between cameras parameter

File: hector_tracked_vehicles_description/urdf/jasmine_2018_ugv.urdf.xacro (robot description, xacro)
@@ -44,7 +44,7 @@
     </xacro:realsense_d435_camera_comprehensive_params>
     <xacro:include filename="$(find hector_sensors_description)/urdf/camera360.urdf.xacro"/>
-    <xacro:camera360 name="camera360" right_cam_name="right" left_cam_name="left" parent="base_link" ros_topic="image_raw" update_rate="10" res_x="1504" res_y="1504" image_format="R8G8B8" fov="${M_PI}">
-      <origin xyz="0.0 0.0 0.58" rpy="0.0 0 0"/>
-      <origin xyz="0.00009742  0.00061696 -0.03850784" rpy="3.1373499 -0.0021358 -3.1279404"/>
+    <xacro:camera360 name="camera360" right_cam_name="right" left_cam_name="left" parent="base_link" dist_between_cameras="-0.03850784" ros_topic="image_raw" update_rate="10" res_x="1504" res_y="1504" image_format="R8G8B8" fov="${M_PI}">
+      <origin xyz="0.0 0.0 0.58" rpy="0.0 0 0"/> <!-- base_link to camera mount transform -->
+      <origin xyz="0.00009742  0.00061696 -0.03850784" rpy="3.1373499 -0.0021358 -3.1279404"/> <!-- cam to cam transform (calibration by kalibr) -->
 <!--       <origin xyz="0.03850784 0 0" rpy="0 0 ${M_PI}"/> -->
     </xacro:camera360>

Commit message: ground calibration

File: hector_tracked_vehicles_description/urdf/jasmine_2018_ugv.urdf.xacro (robot description, xacro)
@@ -22,4 +22,17 @@
       <xacro:arg name="add_raycast_self_filter_geom" default="$(arg add_raycast_self_filter_geom)"/>-->
     </xacro:jasmine_ugv_macro>
+    <!-- Helper links to view robot from front and side with top-down ortho in rviz -->
+<!--    <joint name="base_link_side_joint" type="fixed">
+      <origin xyz="0 0 0" rpy="${M_PI/2} 0 0" />
+      <parent link="base_link"/>
+      <child link="base_link_side" />
+    </joint>
+    <link name="base_link_side"/>
+    <joint name="base_link_front_joint" type="fixed">
+      <origin xyz="0 0 0" rpy=" 0 ${-M_PI/2} 0" />
+      <parent link="base_link"/>
+      <child link="base_link_front" />
+    </joint>
+    <link name="base_link_front"/>-->
     <!--
     <xacro:vision_box parent="base_link" box_type="hector2">
@@ -37,6 +50,6 @@
     </xacro:jasmine_2018_structure_addons_macro>
     <xacro:spinning_sensor_mount_macro parent="base_link"  name="spin_lidar" scaling="0.001">
-      <!-- the angles are due to ground calibration with tud tracker vlp16 -->
-      <origin xyz="${+0.0 } 0.0 ${0.27 + 0.0944673}" rpy="0.0 0.0 ${M_PI}"/>
+      <!-- the angles are due to ground calibration with jasmine (06.10.2018) -->
+      <origin xyz="${+0.0 } 0.0 ${0.27 + 0.0944673}" rpy="-0.00116843 0.00539346 ${M_PI}"/>
     </xacro:spinning_sensor_mount_macro>
     <xacro:realsense_d435_camera_comprehensive_params name="manipulation_rgbd_cam" parent="base_link" image_topic="image_rect_color" depth_points_topic="depth/points" min_range="0.3" max_range="9.0" update_rate="20">

Commit message: add yaw offset of sensor head

File: hector_tracked_vehicles_description/urdf/jasmine_2018_ugv.urdf.xacro (robot description, xacro)
@@ -44,5 +44,5 @@
     </xacro:manipulator_arm_macro>
     <xacro:tracker_sensor_head_macro parent="base_link">
-      <origin xyz="${+0.18 } 0.04 ${0.05}" rpy="0.0 -0.0 ${0.0}"/>
+      <origin xyz="${+0.18 } 0.04 ${0.05}" rpy="0.0 -0.0 -0.187273829"/>
     </xacro:tracker_sensor_head_macro>
     <xacro:jasmine_2018_structure_addons_macro parent="base_link" alu_profile_collision_size_factor="2.0">

Commit message: camera lidar calibration

File: hector_tracked_vehicles_description/urdf/jasmine_2018_ugv.urdf.xacro (robot description, xacro)
@@ -58,5 +58,5 @@
     <xacro:include filename="$(find hector_sensors_description)/urdf/camera360.urdf.xacro"/>
     <xacro:camera360 name="camera360" right_cam_name="right" left_cam_name="left" parent="base_link" dist_between_cameras="-0.03850784" ros_topic="image_raw" update_rate="10" res_x="1504" res_y="1504" image_format="R8G8B8" fov="${M_PI}">
-      <origin xyz="0.0 0.0 0.58" rpy="0.0 0 0"/> <!-- base_link to camera mount transform -->
+      <origin xyz="0.0 0.0 0.59" rpy="0.0 0.01 -0.04"/> <!-- base_link to camera mount transform -->
       <origin xyz="0.00009742  0.00061696 -0.03850784" rpy="3.1373499 -0.0021358 -3.1279404"/> <!-- cam to cam transform (calibration by kalibr) -->
 <!--       <origin xyz="0.03850784 0 0" rpy="0 0 ${M_PI}"/> -->

Commit message: Revert "add yaw offset of sensor head"
This reverts commit adf61492ead0921775c23e45526781a062b51f1b.

File: hector_tracked_vehicles_description/urdf/jasmine_2018_ugv.urdf.xacro (robot description, xacro)
@@ -44,5 +44,5 @@
     </xacro:manipulator_arm_macro>
     <xacro:tracker_sensor_head_macro parent="base_link">
-      <origin xyz="${+0.18 } 0.04 ${0.05}" rpy="0.0 -0.0 -0.187273829"/>
+      <origin xyz="${+0.18 } 0.04 ${0.05}" rpy="0.0 -0.0 ${0.0}"/>
     </xacro:tracker_sensor_head_macro>
     <xacro:jasmine_2018_structure_addons_macro parent="base_link" alu_profile_collision_size_factor="2.0">

Commit message: rotate the lidar 180°

File: hector_tracked_vehicles_description/urdf/jasmine_2018_ugv.urdf.xacro (robot description, xacro)
@@ -51,5 +51,5 @@
     <xacro:spinning_sensor_mount_macro parent="base_link"  name="spin_lidar" scaling="0.001">
       <!-- the angles are due to ground calibration with jasmine (06.10.2018) -->
-      <origin xyz="${+0.0 } 0.0 ${0.27 + 0.0944673}" rpy="-0.00116843 0.00539346 ${M_PI}"/>
+      <origin xyz="${+0.0 } 0.0 ${0.27 + 0.0944673}" rpy="-0.00116843 0.00539346 0"/>
     </xacro:spinning_sensor_mount_macro>
     <xacro:realsense_d435_camera_comprehensive_params name="manipulation_rgbd_cam" parent="base_link" image_topic="image_rect_color" depth_points_topic="depth/points" min_range="0.3" max_range="9.0" update_rate="20">

Commit message: fixed autonomy box height

File: hector_tracked_vehicles_description/urdf/jasmine_2018_ugv.urdf.xacro (robot description, xacro)
@@ -42,5 +42,5 @@
     </xacro:tracker_sensor_head_macro>
     <xacro:jasmine_2018_structure_addons_macro parent="base_link" alu_profile_collision_size_factor="2.0">
-     <origin xyz="0 0 0" rpy="0 0 0"/>
+     <origin xyz="0 0 0.029" rpy="0 0 0"/>
     </xacro:jasmine_2018_structure_addons_macro>
     <xacro:realsense_d435_camera_comprehensive_params name="manipulation_rgbd_cam" parent="base_link" image_topic="image_rect_color" depth_points_topic="depth/points" min_range="0.3" max_range="9.0" update_rate="20">

Commit message: moved autonomy box down

File: hector_tracked_vehicles_description/urdf/jasmine_2018_ugv.urdf.xacro (robot description, xacro)
@@ -42,5 +42,5 @@
     </xacro:tracker_sensor_head_macro>
     <xacro:jasmine_2018_structure_addons_macro parent="base_link" alu_profile_collision_size_factor="2.0">
-     <origin xyz="0 0 0.029" rpy="0 0 0"/>
+     <origin xyz="0 0 0.025" rpy="0 0 0"/>
     </xacro:jasmine_2018_structure_addons_macro>
 <!--    <xacro:realsense_d435_camera_comprehensive_params name="manipulation_rgbd_cam" parent="base_link" image_topic="image_rect_color" depth_points_topic="depth/points" min_range="0.3" max_range="9.0" update_rate="20">

Commit message: moved autonomy box

File: hector_tracked_vehicles_description/urdf/jasmine_2018_ugv.urdf.xacro (robot description, xacro)
@@ -42,5 +42,5 @@
     </xacro:tracker_sensor_head_macro>
     <xacro:jasmine_2018_structure_addons_macro parent="base_link" alu_profile_collision_size_factor="2.0">
-     <origin xyz="0 0 0.025" rpy="0 0 0"/>
+     <origin xyz="${base_size_x - 0.12 - computer_box_width/2} 0 0.025" rpy="0 0 0"/>
     </xacro:jasmine_2018_structure_addons_macro>
 <!--    <xacro:realsense_d435_camera_comprehensive_params name="manipulation_rgbd_cam" parent="base_link" image_topic="image_rect_color" depth_points_topic="depth/points" min_range="0.3" max_range="9.0" update_rate="20">

Commit message: add xm430 sensor head and fix the component's height of the base plate

File: hector_tracked_vehicles_description/urdf/jasmine_2018_ugv.urdf.xacro (robot description, xacro)
@@ -5,5 +5,5 @@
     <xacro:include filename="$(find hector_tracked_vehicles_description)/urdf/jasmine_2018_structure_addons.urdf.xacro" />
     <xacro:include filename="$(find hector_components_description)/urdf/vlp16_mount.urdf.xacro.xml"/>
-    <xacro:include filename="$(find hector_components_description)/urdf/tracker_sensor_head.urdf.xacro.xml"/>
+    <xacro:include filename="$(find hector_components_description)/urdf/xm430_sensor_head.urdf.xacro.xml"/>
     <xacro:include filename="$(find hector_tracked_vehicles_description)/calibrations/spin_lidar_calibration.urdf.xacro"/>
     <xacro:include filename="$(find hector_tracked_vehicles_description)/urdf/jasmine_2018_ugv_arm.urdf.xacro" />
@@ -14,4 +14,5 @@
     </xacro:property>
     -->
+    <xacro:property name="base_link_to_base_plate_dist" value="0.059"/>
     <xacro:arg name="add_default_geom" default="true"/>
     <xacro:arg name="add_containment_self_filter_geom" default="false"/>
@@ -36,11 +37,11 @@
     <link name="base_link_front"/>-->
     <xacro:manipulator_arm_macro parent="base_link">
-      <origin xyz="-0.1618 -0.06875 0.01315" rpy="0.0 0.0 ${M_PI/2}" />
+      <origin xyz="-0.1618 -0.06875 ${0.097-base_link_to_base_plate_dist}" rpy="0.0 0.0 ${M_PI/2}" />
     </xacro:manipulator_arm_macro>
-    <xacro:tracker_sensor_head_macro parent="base_link">
-      <origin xyz="${+0.18 } 0.04 ${0.05}" rpy="0.0 -0.0 ${0.0}"/>
-    </xacro:tracker_sensor_head_macro>
+    <xacro:xm430_sensor_head_macro parent="base_link" name="sensor_head">
+      <origin xyz="0.225 0.0 ${0.077-base_link_to_base_plate_dist}" rpy="0.0 0.0 0.0"/>
+    </xacro:xm430_sensor_head_macro>
     <xacro:jasmine_2018_structure_addons_macro parent="base_link" alu_profile_collision_size_factor="2.0">
-     <origin xyz="0 0 0.025" rpy="0 0 0"/>
+     <origin xyz="0 0 ${0.084-base_link_to_base_plate_dist}" rpy="0 0 0"/>
     </xacro:jasmine_2018_structure_addons_macro>
 <!--    <xacro:realsense_d435_camera_comprehensive_params name="manipulation_rgbd_cam" parent="base_link" image_topic="image_rect_color" depth_points_topic="depth/points" min_range="0.3" max_range="9.0" update_rate="20">

Commit message: increased raycast self filter geom size of chassis increased collision size of chassis according to measurements of marius

File: hector_tracked_vehicles_description/urdf/jasmine_2018_ugv.urdf.xacro (robot description, xacro)
@@ -14,5 +14,4 @@
     </xacro:property>
     -->
-    <xacro:property name="base_link_to_base_plate_dist" value="0.059"/>
     <xacro:arg name="add_default_geom" default="true"/>
     <xacro:arg name="add_containment_self_filter_geom" default="false"/>
@@ -37,11 +36,11 @@
     <link name="base_link_front"/>-->
     <xacro:manipulator_arm_macro parent="base_link">
-      <origin xyz="-0.1618 -0.06875 ${0.097-base_link_to_base_plate_dist}" rpy="0.0 0.0 ${M_PI/2}" />
+      <origin xyz="-0.1618 -0.06875 ${0.097-base_size_z}" rpy="0.0 0.0 ${M_PI/2}" />
     </xacro:manipulator_arm_macro>
     <xacro:xm430_sensor_head_macro parent="base_link" name="sensor_head">
-      <origin xyz="0.225 0.0 ${0.077-base_link_to_base_plate_dist}" rpy="0.0 0.0 0.0"/>
+      <origin xyz="0.225 0.0 ${0.077-base_size_z}" rpy="0.0 0.0 0.0"/>
     </xacro:xm430_sensor_head_macro>
     <xacro:jasmine_2018_structure_addons_macro parent="base_link" alu_profile_collision_size_factor="2.0">
-     <origin xyz="${base_size_x - 0.12 - computer_box_width/2} 0 ${0.084-base_link_to_base_plate_dist}" rpy="0 0 0"/>
+     <origin xyz="${base_size_x - 0.12 - computer_box_width/2} 0 ${0.084-base_size_z}" rpy="0 0 0"/>
     </xacro:jasmine_2018_structure_addons_macro>
 <!--    <xacro:realsense_d435_camera_comprehensive_params name="manipulation_rgbd_cam" parent="base_link" image_topic="image_rect_color" depth_points_topic="depth/points" min_range="0.3" max_range="9.0" update_rate="20">

File: hector_tracked_vehicles_description/urdf/jasmine_ugv_base.urdf.xacro (robot description, xacro)
@@ -11,5 +11,5 @@
     <xacro:property name="base_size_x" value="0.255" />
     <xacro:property name="base_size_y" value="0.12" />
-    <xacro:property name="base_size_z" value="0.045" />
+    <xacro:property name="base_size_z" value="0.059" />
     <xacro:property name="wheel_radius_big" value="0.080" />
     <xacro:property name="wheel_length" value="0.02" />

File: hector_tracked_vehicles_description/urdf/jasmine_ugv_tracks.urdf.xacro (robot description, xacro)
@@ -27,11 +27,19 @@
         </collision>
       </xacro:if>
+      <xacro:property name="collision_factor" value="2" />
+      <xacro:property name="collision_cylinder_length_factor" value="1.1" />
       <!-- Raycast self-filter geom -->
       <!-- Does not use boxes as raycast filtering is broken as of 27.03.2019 -->
       <xacro:if value="$(arg add_raycast_self_filter_geom)">
         <collision>
+          <origin xyz="0.0 0.0 ${t_offset_z}" rpy="0 ${M_PI*0.5} 0" />
+          <geometry>
+            <cylinder length="${t_base_size_x*2 * collision_cylinder_length_factor}" radius="${t_base_size_z*collision_factor}"/>
+          </geometry>
+        </collision>
+        <collision>
           <origin xyz="0.0 0.07 ${t_offset_z}" rpy="0 ${M_PI*0.5} 0" />
           <geometry>
-            <cylinder length="${t_base_size_x*2}" radius="${t_base_size_z*1.6}"/>
+            <cylinder length="${t_base_size_x*2 * collision_cylinder_length_factor}" radius="${t_base_size_z*collision_factor}"/>
           </geometry>
         </collision>
@@ -39,5 +47,5 @@
           <origin xyz="0.0 -0.07 ${t_offset_z}" rpy="0 ${M_PI*0.5} 0" />
           <geometry>
-            <cylinder length="${t_base_size_x*2}" radius="${t_base_size_z*1.6}"/>
+            <cylinder length="${t_base_size_x*2 * collision_cylinder_length_factor}" radius="${t_base_size_z*collision_factor}"/>
           </geometry>
         </collision>

Commit message: started the urdf for the dynamixel pro arm upgrade

File: hector_tracked_vehicles_description/urdf/jasmine_2018_ugv.urdf.xacro (robot description, xacro)
@@ -36,5 +36,5 @@
     <link name="base_link_front"/>-->
     <xacro:manipulator_arm_macro parent="base_link">
-      <origin xyz="-0.1618 -0.06875 ${0.097-base_size_z}" rpy="0.0 0.0 ${M_PI/2}" />
+      <origin xyz="-0.1618 -0.06875 ${0.077-base_size_z}" rpy="0.0 0.0 ${M_PI/2}" />
     </xacro:manipulator_arm_macro>
     <xacro:xm430_sensor_head_macro parent="base_link" name="sensor_head">

File: hector_tracked_vehicles_description/urdf/jasmine_2018_ugv_arm.urdf.xacro (robot description, xacro)
@@ -69,5 +69,5 @@
     </link>
     <joint name="arm_yaw_joint" type="revolute">
-      <origin xyz="0.0 0 0.036" rpy="0.0 0.0 ${pi / 2}" />
+      <origin xyz="0.0 0 0.086" rpy="0.0 0.0 ${pi / 2}" />
       <axis xyz="0 0 1" />
       <limit lower="${-pi / 2}" upper="${pi / 2}" effort="${XM430_W350_max_effort}" velocity="${XM430_W350_max_velocity}" />
@@ -109,5 +109,5 @@
     </link>
     <joint name="arm_pitch_joint_0" type="revolute">
-      <origin xyz="0.0 0.0 0.0515" rpy=" ${pi/2} 0.0 0.0" />
+      <origin xyz="0.0 0.0 0.0275" rpy=" ${pi/2} 0.0 0.0" />
       <axis xyz="0 0 1" />
       <limit lower="${-pi / 2}" upper="${pi / 2}" effort="${XM540_W270_max_effort}" velocity="${XM540_W270_max_velocity}" />
@@ -167,5 +167,5 @@
     </link>
     <joint name="arm_pitch_joint_1" type="revolute">
-      <origin xyz="0.026 0.2517 0.0" rpy="0.0 0.0 ${-pi}" />
+      <origin xyz="0.031 0.2505 0.0" rpy="0.0 0.0 ${-pi}" />
       <axis xyz="0 0 1" />
       <limit lower="${-pi/2}" upper="${pi/2}" effort="${XM430_W350_max_effort}" velocity="${XM430_W350_max_velocity}" />
@@ -225,5 +225,5 @@
     </link>
     <joint name="arm_pitch_joint_2" type="revolute">
-      <origin xyz="-0.1967 -0.004 0.0" rpy="0.0 0.0 0.0" />
+      <origin xyz="-0.2017 -0.002 0.0" rpy="0.0 0.0 0.0" />
       <axis xyz="0 0 1" />
       <limit lower="${-pi / 2}" upper="${pi / 2}" effort="${XM430_W350_max_effort}" velocity="${XM430_W350_max_velocity}" />

Commit message: updated urdf

File: hector_tracked_vehicles_description/urdf/jasmine_2018_ugv.urdf.xacro (robot description, xacro)
@@ -36,5 +36,5 @@
     <link name="base_link_front"/>-->
     <xacro:manipulator_arm_macro parent="base_link">
-      <origin xyz="-0.1618 -0.06875 ${0.077-base_size_z}" rpy="0.0 0.0 ${M_PI/2}" />
+      <origin xyz="-0.136 -0.06875 ${0.077-base_size_z}" rpy="0.0 0.0 ${M_PI/2}" />
     </xacro:manipulator_arm_macro>
     <xacro:xm430_sensor_head_macro parent="base_link" name="sensor_head">

File: hector_tracked_vehicles_description/urdf/jasmine_2018_ugv_arm.urdf.xacro (robot description, xacro)
@@ -109,5 +109,5 @@
     </link>
     <joint name="arm_pitch_joint_0" type="revolute">
-      <origin xyz="0.0 0.0 0.0275" rpy=" ${pi/2} 0.0 0.0" />
+      <origin xyz="0.0 0.0 0.027" rpy=" ${pi/2} 0.0 0.0" />
       <axis xyz="0 0 1" />
       <limit lower="${-pi / 2}" upper="${pi / 2}" effort="${XM540_W270_max_effort}" velocity="${XM540_W270_max_velocity}" />
@@ -167,5 +167,5 @@
     </link>
     <joint name="arm_pitch_joint_1" type="revolute">
-      <origin xyz="0.031 0.2505 0.0" rpy="0.0 0.0 ${-pi}" />
+      <origin xyz="0.031 0.2545 0.0" rpy="0.0 0.0 ${-pi}" />
       <axis xyz="0 0 1" />
       <limit lower="${-pi/2}" upper="${pi/2}" effort="${XM430_W350_max_effort}" velocity="${XM430_W350_max_velocity}" />
