Commit message: fix the gripper links

File: hector_tracked_vehicles_description/urdf/jasmine_2018_ugv_arm.urdf.xacro (robot description, xacro)
@@ -328,7 +328,7 @@
     </link>
     <joint name="gripper_servo_joint" type="revolute">
-      <origin xyz="-0.04225 0.0 -0.016" rpy="${pi/2} 0 0.0" />
-      <axis xyz="0 0 1" />
-      <limit lower="-1.6" upper="${105 * M_PI / 180}" effort="${XM430_W350_max_effort}" velocity="${XM430_W350_max_velocity}" />
+      <origin xyz="0.024 0.01612 0.01625" rpy="${pi/2} 0.0 ${pi / 2}" />
+      <axis xyz="0 0 1" />
+      <limit lower="${-190 / 180 * M_PI}" upper="0.0" effort="${XM430_W350_max_effort}" velocity="${XM430_W350_max_velocity}" />
       <parent link="gripper_palm_link" />
       <child link="gripper_servo_link" />
@@ -343,6 +343,12 @@
                                             izz="1.0e-05" />
       </inertial>
-      <collision>
-        <origin xyz="0 0.0 0.0275" rpy="0.0 0.0 0.0" />
+      <visual>
+        <origin xyz="0 0.0 0.0" rpy="0.0 0.0 0.0" />
+        <geometry>
+          <cylinder length="0.01" radius="0.01" />
+        </geometry>
+      </visual>
+      <collision>
+        <origin xyz="0 0.0 0.0" rpy="0.0 0.0 0.0" />
         <geometry>
           <cylinder length="0.01" radius="0.01" />
@@ -352,5 +358,5 @@
     <!-- virtual endeffector joint -->
     <joint name="gripper_grasp" type="fixed">
-      <origin xyz="-0.14 0.0 0.0" rpy="0.0 0.0 0.0"/>
+      <origin xyz="0.0 0.0 0.15" rpy="0.0 0.0 0.0"/>
       <parent link="gripper_palm_link"/>
       <child link="gripper_grasp_link"/>

Commit message: renamed gripper_mount_joint removed mass of grasp link

File: hector_tracked_vehicles_description/urdf/jasmine_2018_ugv_arm.urdf.xacro (robot description, xacro)
@@ -262,10 +262,10 @@
       </inertial>
     </link>
-    <joint name="gripper_mount_joint" type="fixed">
+    <joint name="gripper_palm_joint" type="fixed">
       <origin xyz="0.0 0.0 0.0" rpy="0.0 0.0 0.0" />
       <parent link="arm_roll_link" />
       <child link="gripper_palm_link" />
     </joint>
-       <link name="gripper_palm_link">
+    <link name="gripper_palm_link">
       <visual>
         <origin xyz="0.0 0.0 0.0" rpy="0.0 0.0 0.0" />
@@ -357,5 +357,5 @@
     </link>
     <!-- virtual endeffector joint -->
-    <joint name="gripper_grasp" type="fixed">
+    <joint name="gripper_grasp_joint" type="fixed">
       <origin xyz="0.0 0.0 0.15" rpy="0.0 0.0 0.0"/>
       <parent link="gripper_palm_link"/>
@@ -363,16 +363,16 @@
     </joint>
     <link name="gripper_grasp_link">
-    <visual>
-      <origin xyz="0.0 0.0 0.0" rpy="0.0 0.0 0.0"/>
-      <geometry>
-        <sphere radius="0.005" />
-      </geometry>
-      <material name="red"/>
-    </visual>
-    <inertial>
-      <origin xyz="0.0 0.0 0.0" rpy="0.0 0.0 0.0"/>
-      <mass value="0.0001"/>
-    <inertia ixx="1.0e-10" ixy="0.0" ixz="0.0" iyy="1.0e-10" iyz="0.0" izz="1.0e-10" />
-    </inertial>
+<!--      <visual>
+        <origin xyz="0.0 0.0 0.0" rpy="0.0 0.0 0.0"/>
+        <geometry>
+          <sphere radius="0.005" />
+        </geometry>
+        <material name="red"/>
+      </visual>
+      <inertial>
+        <origin xyz="0.0 0.0 0.0" rpy="0.0 0.0 0.0"/>
+        <mass value="0.0001"/>
+      <inertia ixx="1.0e-10" ixy="0.0" ixz="0.0" iyy="1.0e-10" iyz="0.0" izz="1.0e-10" />
+      </inertial>-->
     </link>
 	  <!-- gripper finger -->

Commit message: adjust the joint limits

File: hector_tracked_vehicles_description/urdf/jasmine_2018_ugv_arm.urdf.xacro (robot description, xacro)
@@ -43,7 +43,7 @@
     </link>
     <joint name="arm_yaw_joint" type="revolute">
-      <origin xyz="0.0 0 0.036" rpy="0.0 0.0 ${pi}" />
-      <axis xyz="0 0 1" />
-      <limit lower="${-pi+0.001}" upper="${pi-0.001}" effort="${XM430_W350_max_effort}" velocity="${XM430_W350_max_velocity}" />
+      <origin xyz="0.0 0 0.036" rpy="0.0 0.0 ${pi / 2}" />
+      <axis xyz="0 0 1" />
+      <limit lower="${-pi / 2}" upper="${pi / 2}" effort="${XM430_W350_max_effort}" velocity="${XM430_W350_max_velocity}" />
       <parent link="arm_base_link" />
       <child link="arm_yaw_link" />
@@ -77,5 +77,5 @@
       <origin xyz="0.0 0.0 0.0515" rpy=" ${pi/2} 0.0 0.0" />
       <axis xyz="0 0 1" />
-      <limit lower="${-100 * pi / 180}" upper="${100 * pi / 180}" effort="${XM540_W270_max_effort}" velocity="${XM540_W270_max_velocity}" />
+      <limit lower="${-pi / 2}" upper="${pi / 2}" effort="${XM540_W270_max_effort}" velocity="${XM540_W270_max_velocity}" />
       <parent link="arm_yaw_link" />
       <child link="arm_pitch_link_0" />
@@ -125,7 +125,8 @@
     </link>
     <joint name="arm_pitch_joint_1" type="revolute">
-      <origin xyz="0.026 0.2517 0.0" rpy="0.0 0.0 ${-pi/2}" />
-      <axis xyz="0 0 1" />
-      <limit lower="${-180 * pi / 180}" upper="${25 * pi / 180}" effort="${XM430_W350_max_effort}" velocity="${XM430_W350_max_velocity}" />
+      <origin xyz="0.026 0.2517 0.0" rpy="0.0 0.0 ${-pi}" />
+      <axis xyz="0 0 1" />
+      <limit lower="${-pi/2}" upper="${
+             pi/2}" effort="${XM430_W350_max_effort}" velocity="${XM430_W350_max_velocity}" />
       <parent link="arm_pitch_link_0" />
       <child link="arm_pitch_link_1" />
@@ -177,5 +178,5 @@
       <origin xyz="-0.1967 -0.004 0.0" rpy="0.0 0.0 0.0" />
       <axis xyz="0 0 1" />
-      <limit lower="${-95 * pi / 180}" upper="${95 * pi / 180}" effort="${XM430_W350_max_effort}" velocity="${XM430_W350_max_velocity}" />
+      <limit lower="${-pi / 2}" upper="${pi / 2}" effort="${XM430_W350_max_effort}" velocity="${XM430_W350_max_velocity}" />
       <parent link="arm_pitch_link_1" />
       <child link="arm_pitch_link_2" />
@@ -219,7 +220,7 @@
     </link>
     <joint name="arm_roll_joint" type="revolute">
-      <origin xyz="-0.073 0.0 -0.012" rpy="0 ${-pi/2} 0.0" />
-      <axis xyz="0 0 1" />
-      <limit lower="${-95 * pi / 180}" upper="${95 * pi / 180}" effort="${XM430_W350_max_effort}" velocity="${XM430_W350_max_velocity}" />
+      <origin xyz="-0.073 0.0 -0.012" rpy="${pi/2} 0.0 ${-pi/2}" />
+      <axis xyz="0 0 1" />
+      <limit lower="${-3/4*pi}" upper="${3/4*pi}" effort="${XM430_W350_max_effort}" velocity="${XM430_W350_max_velocity}" />
       <parent link="arm_pitch_link_2" />
       <child link="arm_roll_link" />

Commit message: adjust the urdf towards the real arm

File: hector_tracked_vehicles_description/urdf/jasmine_2018_ugv_arm.urdf.xacro (robot description, xacro)
@@ -127,6 +127,5 @@
       <origin xyz="0.026 0.2517 0.0" rpy="0.0 0.0 ${-pi}" />
       <axis xyz="0 0 1" />
-      <limit lower="${-pi/2}" upper="${
-             pi/2}" effort="${XM430_W350_max_effort}" velocity="${XM430_W350_max_velocity}" />
+      <limit lower="${-pi/2}" upper="${pi/2}" effort="${XM430_W350_max_effort}" velocity="${XM430_W350_max_velocity}" />
       <parent link="arm_pitch_link_0" />
       <child link="arm_pitch_link_1" />
@@ -222,5 +221,5 @@
       <origin xyz="-0.073 0.0 -0.012" rpy="${pi/2} 0.0 ${-pi/2}" />
       <axis xyz="0 0 1" />
-      <limit lower="${-3/4*pi}" upper="${3/4*pi}" effort="${XM430_W350_max_effort}" velocity="${XM430_W350_max_velocity}" />
+      <limit lower="${-pi/2}" upper="${pi}" effort="${XM430_W350_max_effort}" velocity="${XM430_W350_max_velocity}" />
       <parent link="arm_pitch_link_2" />
       <child link="arm_roll_link" />
@@ -331,5 +330,5 @@
       <origin xyz="0.024 0.01612 0.01625" rpy="${pi/2} 0.0 ${pi / 2}" />
       <axis xyz="0 0 1" />
-      <limit lower="${-190 / 180 * M_PI}" upper="0.0" effort="${XM430_W350_max_effort}" velocity="${XM430_W350_max_velocity}" />
+      <limit lower="${-M_PI/2}" upper="${112 * M_PI/ 180}" effort="${XM430_W350_max_effort}" velocity="${XM430_W350_max_velocity}" />
       <parent link="gripper_palm_link" />
       <child link="gripper_servo_link" />
@@ -384,5 +383,5 @@
       <parent link="gripper_palm_link" />
       <child link="gripper_finger_link_0" />
-      <mimic joint="gripper_servo_joint" multiplier="${8 / 23}" offset="0" />
+      <mimic joint="gripper_servo_joint" multiplier="${-8 / 23}" offset="${-M_PI/2 * 8/23}" />
       <dynamics friction="${joint_friction}" damping="${joint_damping}" />
     </joint>
@@ -435,5 +434,5 @@
       <parent link="gripper_palm_link" />
       <child link="gripper_finger_link_1" />
-      <mimic joint="gripper_servo_joint" multiplier="${8 / 23}" offset="0" />
+      <mimic joint="gripper_servo_joint" multiplier="${-8 / 23}" offset="${-M_PI/2 * 8/23}" />
       <dynamics friction="${joint_friction}" damping="${joint_damping}" />
     </joint>

Commit message: update roll servo limits

File: hector_tracked_vehicles_description/urdf/jasmine_2018_ugv_arm.urdf.xacro (robot description, xacro)
@@ -221,5 +221,5 @@
       <origin xyz="-0.073 0.0 -0.012" rpy="${pi/2} 0.0 ${-pi/2}" />
       <axis xyz="0 0 1" />
-      <limit lower="${-pi/2}" upper="${pi}" effort="${XM430_W350_max_effort}" velocity="${XM430_W350_max_velocity}" />
+      <limit lower="${-pi}" upper="${162.976*pi/180}" effort="${XM430_W350_max_effort}" velocity="${XM430_W350_max_velocity}" />
       <parent link="arm_pitch_link_2" />
       <child link="arm_roll_link" />

Commit message: added gripper cam

File: hector_tracked_vehicles_description/urdf/jasmine_2018_ugv_arm.urdf.xacro (robot description, xacro)
@@ -6,4 +6,5 @@
   xmlns:xacro="http://ros.org/wiki/xacro">
   <xacro:include filename="$(find hector_tracked_vehicles_description)/urdf/jasmine_2018_ugv_arm.gazebo.xacro" />
+  <xacro:include filename="$(find hector_sensors_description)/urdf/generic_camera.urdf.xacro" />
   <xacro:property name="XM430_W350_max_effort" value="4.1" />
   <xacro:property name="XM540_W270_max_effort" value="10.6" />
@@ -479,4 +480,7 @@
       </inertial>
     </link>
+    <xacro:generic_camera name="gripper_cam" parent="gripper_palm_link" ros_topic="/gripper_cam/image_raw" cam_info_topic="/gripper_cam/camera_info" update_rate="15" res_x="1024" res_y="1024" image_format="rgb8" hfov="60">
+      <origin xyz="0 0 0" rpy="${-pi/2} ${-pi/2} ${-pi/2}"/>
+    </xacro:generic_camera>
   </xacro:macro>
 </robot>

Commit message: rotated gripper cam

File: hector_tracked_vehicles_description/urdf/jasmine_2018_ugv_arm.urdf.xacro (robot description, xacro)
@@ -481,5 +481,5 @@
     </link>
     <xacro:generic_camera name="gripper_cam" parent="gripper_palm_link" ros_topic="/gripper_cam/image_raw" cam_info_topic="/gripper_cam/camera_info" update_rate="15" res_x="1024" res_y="1024" image_format="rgb8" hfov="60">
-      <origin xyz="0 0 0" rpy="${-pi/2} ${-pi/2} ${-pi/2}"/>
+      <origin xyz="0 0 0" rpy="${pi/2} ${-pi/2} ${-pi/2}"/>
     </xacro:generic_camera>
   </xacro:macro>

Commit message: rotated gripper cam #2

File: hector_tracked_vehicles_description/urdf/jasmine_2018_ugv_arm.urdf.xacro (robot description, xacro)
@@ -481,5 +481,5 @@
     </link>
     <xacro:generic_camera name="gripper_cam" parent="gripper_palm_link" ros_topic="/gripper_cam/image_raw" cam_info_topic="/gripper_cam/camera_info" update_rate="15" res_x="1024" res_y="1024" image_format="rgb8" hfov="60">
-      <origin xyz="0 0 0" rpy="${pi/2} ${-pi/2} ${-pi/2}"/>
+      <origin xyz="0 0 0" rpy="0 ${-pi/2} ${-pi/2}"/>
     </xacro:generic_camera>
   </xacro:macro>

Commit message: rotated gripper #3

File: hector_tracked_vehicles_description/urdf/jasmine_2018_ugv_arm.urdf.xacro (robot description, xacro)
@@ -481,5 +481,5 @@
     </link>
     <xacro:generic_camera name="gripper_cam" parent="gripper_palm_link" ros_topic="/gripper_cam/image_raw" cam_info_topic="/gripper_cam/camera_info" update_rate="15" res_x="1024" res_y="1024" image_format="rgb8" hfov="60">
-      <origin xyz="0 0 0" rpy="0 ${-pi/2} ${-pi/2}"/>
+      <origin xyz="0 0 0" rpy="${pi} ${-pi/2} ${-pi/2}"/>
     </xacro:generic_camera>
   </xacro:macro>

Commit message: adjusted gripper cam position

File: hector_tracked_vehicles_description/urdf/jasmine_2018_ugv_arm.urdf.xacro (robot description, xacro)
@@ -481,5 +481,5 @@
     </link>
     <xacro:generic_camera name="gripper_cam" parent="gripper_palm_link" ros_topic="/gripper_cam/image_raw" cam_info_topic="/gripper_cam/camera_info" update_rate="15" res_x="640" res_y="480" image_format="R8G8B8" hfov="60">
-      <origin xyz="0 0 0" rpy="${pi} ${-pi/2} ${-pi/2}"/>
+      <origin xyz="0 0 ${0.034 + 0.02}" rpy="${pi} ${-pi/2} ${-pi/2}"/>
     </xacro:generic_camera>
   </xacro:macro>

Commit message: added touch tool to urdf

File: hector_tracked_vehicles_description/urdf/jasmine_2018_ugv_arm.urdf.xacro (robot description, xacro)
@@ -480,7 +480,22 @@
       </inertial>
     </link>
+    <xacro:property name="servo_width" value="0.034" />
+    <xacro:property name="touch_tool_length" value="0.109" />
     <xacro:generic_camera name="gripper_cam" parent="gripper_palm_link" ros_topic="/gripper_cam/image_raw" cam_info_topic="/gripper_cam/camera_info" update_rate="15" res_x="640" res_y="480" image_format="R8G8B8" hfov="60">
-      <origin xyz="0 0 ${0.034 + 0.02}" rpy="${pi} ${-pi/2} ${-pi/2}"/>
+      <origin xyz="0 0 ${servo_width + 0.02}" rpy="${pi} ${-pi/2} ${-pi/2}"/>
     </xacro:generic_camera>
+    <joint name="touch_tool_joint" type="fixed">
+      <origin xyz="0.012 0.0 ${servo_width + touch_tool_length}" rpy="0.0 0.0 0.0"/>
+      <parent link="gripper_palm_link"/>
+      <child link="touch_tool_link"/>
+    </joint>
+    <link name="touch_tool_link">
+      <visual>
+        <origin xyz="0 0 ${-touch_tool_length/2}" rpy="0 0 0"/>
+        <geometry>
+          <cylinder radius="0.001" length="${touch_tool_length}"/>
+        </geometry>
+      </visual>
+    </link>
   </xacro:macro>
 </robot>

Commit message: increased arm motor strength removed dynamics tags fixed inertial tags of gripper

File: hector_tracked_vehicles_description/urdf/jasmine_2018_ugv_arm.urdf.xacro (robot description, xacro)
@@ -7,6 +7,9 @@
   <xacro:include filename="$(find hector_tracked_vehicles_description)/urdf/jasmine_2018_ugv_arm.gazebo.xacro" />
   <xacro:include filename="$(find hector_sensors_description)/urdf/generic_camera.urdf.xacro" />
-  <xacro:property name="XM430_W350_max_effort" value="4.1" />
-  <xacro:property name="XM540_W270_max_effort" value="10.6" />
+  <xacro:include filename="$(find hector_xacro_tools)/urdf/inertia_tensors.urdf.xacro" />
+<!--  <xacro:property name="XM430_W350_max_effort" value="4.1" />
+  <xacro:property name="XM540_W270_max_effort" value="10.6" />-->
+  <xacro:property name="XM430_W350_max_effort" value="1000" />
+  <xacro:property name="XM540_W270_max_effort" value="1000" />
   <xacro:property name="XM430_W350_max_velocity" value="4.81710873" />
   <xacro:property name="XM540_W270_max_velocity" value="3.1415926499999998" />
@@ -49,5 +52,5 @@
       <parent link="arm_base_link" />
       <child link="arm_yaw_link" />
-      <dynamics friction="${joint_friction}" damping="${joint_damping}" />
+<!--       <dynamics friction="${joint_friction}" damping="${joint_damping}" /> -->
     </joint>
     <link name="arm_yaw_link">
@@ -81,5 +84,5 @@
       <parent link="arm_yaw_link" />
       <child link="arm_pitch_link_0" />
-      <dynamics friction="${joint_friction}" damping="${joint_damping}" />
+<!--       <dynamics friction="${joint_friction}" damping="${joint_damping}" /> -->
     </joint>
     <link name="arm_pitch_link_0">
@@ -111,5 +114,5 @@
         </geometry>
      </collision>
-    <collision>
+      <collision>
         <origin xyz="0.0 0.13 0.0" rpy="0.0 0.0 0.0" />
         <geometry>
@@ -131,5 +134,5 @@
       <parent link="arm_pitch_link_0" />
       <child link="arm_pitch_link_1" />
-      <dynamics friction="${joint_friction}" damping="${joint_damping}" />
+<!--       <dynamics friction="${joint_friction}" damping="${joint_damping}" /> -->
     </joint>
     <link name="arm_pitch_link_1">
@@ -181,5 +184,5 @@
       <parent link="arm_pitch_link_1" />
       <child link="arm_pitch_link_2" />
-      <dynamics friction="${joint_friction}" damping="${joint_damping}" />
+<!--       <dynamics friction="${joint_friction}" damping="${joint_damping}" /> -->
     </joint>
     <link name="arm_pitch_link_2">
@@ -211,5 +214,5 @@
         </geometry>
       </collision>
-      <inertial>
+<!--      <inertial>
         <origin xyz="-0.11166 0.00016 0.00038" rpy="0.0 0.0 0.0" />
         <mass value="0.127" />
@@ -217,5 +220,8 @@
                                     iyy="215.338e-06"     iyz="-0.221e-06"
                                                           izz="207.743e-06" />
-      </inertial>
+      </inertial>-->
+      <xacro:inertial_cuboid_with_pose mass="0.1" x_length="0.05" y_length="0.05" z_length="0.05" >
+        <origin xyz="-0.05 0 0" rpy="0.0 0.0 0.0" />
+      </xacro:inertial_cuboid_with_pose>
     </link>
     <joint name="arm_roll_joint" type="revolute">
@@ -225,5 +231,5 @@
       <parent link="arm_pitch_link_2" />
       <child link="arm_roll_link" />
-      <dynamics friction="${joint_friction}" damping="${joint_damping}" />
+<!--       <dynamics friction="${joint_friction}" damping="${joint_damping}" /> -->
     </joint>
     <link name="arm_roll_link">
@@ -255,5 +261,5 @@
         </geometry>
       </collision>
-      <inertial>
+<!--      <inertial>
         <origin xyz="-0.11166 0.00016 0.00038" rpy="0.0 0.0 0.0" />
         <mass value="0.127" />
@@ -261,5 +267,8 @@
                                     iyy="215.338e-06"     iyz="-0.221e-06"
                                                           izz="207.743e-06" />
-      </inertial>
+      </inertial>-->
+      <xacro:inertial_cuboid_with_pose mass="0.01" x_length="0.03" y_length="0.03" z_length="0.03" >
+        <origin xyz="0 0 0" rpy="0 0 0" />
+      </xacro:inertial_cuboid_with_pose>
     </link>
     <joint name="gripper_palm_joint" type="fixed">
@@ -320,5 +329,5 @@
         </geometry>
       </collision>
-      <inertial>
+<!--      <inertial>
         <origin xyz="-0.04663 -0.00051 -0.00234" rpy="0.0 0.0 0.0" />
         <mass value="0.155" />
@@ -326,5 +335,8 @@
                                       iyy="70.718e-06"    iyz="0.750e-06"
                                                           izz="141.557e-06" />
-      </inertial>
+      </inertial>-->
+      <xacro:inertial_cuboid_with_pose mass="0.155" x_length="0.05" y_length="0.05" z_length="0.05" >
+        <origin xyz="0 0 0.05" rpy="0.0 0.0 0.0" />
+      </xacro:inertial_cuboid_with_pose>
     </link>
     <joint name="gripper_servo_joint" type="revolute">
@@ -334,8 +346,8 @@
       <parent link="gripper_palm_link" />
       <child link="gripper_servo_link" />
-      <dynamics friction="0" damping="0" />
+<!--       <dynamics friction="0" damping="0" /> -->
     </joint>
     <link name="gripper_servo_link">
-      <inertial>
+<!--      <inertial>
         <origin xyz="0.0 0.0 0.0" rpy="0.0 0.0 0.0" />
         <mass value="0.001" />
@@ -343,5 +355,8 @@
                               iyy="1.0e-05"  iyz="0.0"
                                             izz="1.0e-05" />
-      </inertial>
+      </inertial>-->
+      <xacro:inertial_cuboid_with_pose mass="0.01" x_length="0.05" y_length="0.05" z_length="0.05" >
+        <origin xyz="0 0 0" rpy="0 0 0" />
+      </xacro:inertial_cuboid_with_pose>
       <visual>
         <origin xyz="0 0.0 0.0" rpy="0.0 0.0 0.0" />
@@ -364,16 +379,4 @@
     </joint>
     <link name="gripper_grasp_link">
-<!--      <visual>
-        <origin xyz="0.0 0.0 0.0" rpy="0.0 0.0 0.0"/>
-        <geometry>
-          <sphere radius="0.005" />
-        </geometry>
-        <material name="red"/>
-      </visual>
-      <inertial>
-        <origin xyz="0.0 0.0 0.0" rpy="0.0 0.0 0.0"/>
-        <mass value="0.0001"/>
-      <inertia ixx="1.0e-10" ixy="0.0" ixz="0.0" iyy="1.0e-10" iyz="0.0" izz="1.0e-10" />
-      </inertial>-->
     </link>
 	  <!-- gripper finger -->
@@ -422,5 +425,5 @@
       </collision>
       <inertial>
-        <origin xyz="0.01764 -0.04373 0.0" rpy="0.0 0.0 ${90 * pi / 180}" />
+        <origin xyz="-0.03 -0.05 0.0" rpy="0.0 0.0 ${pi}" />
         <mass value="0.029" />
         <inertia ixx="0.000025065339"   ixy="-0.000009627959" ixz="2.8255e-8"
@@ -473,5 +476,5 @@
       </collision>
       <inertial>
-        <origin xyz="0.01764 -0.04373 0.0" rpy="0.0 0.0 ${90 * pi / 180}" />
+        <origin xyz="-0.03 -0.05 0.0" rpy="0.0 0.0 ${pi}" />
         <mass value="0.029" />
         <inertia ixx="0.000025065339" ixy="-0.000009627959" ixz="2.8255e-8"

Commit message: added folded arm self filter containment geom

File: hector_tracked_vehicles_description/urdf/jasmine_2018_ugv_arm.urdf.xacro (robot description, xacro)
@@ -14,4 +14,5 @@
   <xacro:property name="joint_friction" value="0.5" />
   <xacro:macro name="manipulator_arm_macro" params="parent *origin">
+    <xacro:arg name="add_containment_self_filter_geom" default="false"/>
     <joint name="arm_base_joint" type="fixed">
       <xacro:insert_block name="origin" />
@@ -35,4 +36,15 @@
         </geometry>
       </collision>
+      <xacro:if value="$(arg add_containment_self_filter_geom)">
+        <collision>
+          <origin xyz="${0.06875} ${-1*(-0.18 + 0.1618)} ${0.15/2+0.07-0.01315}" rpy="0 0 0"/>
+          <geometry>
+            <box size="${0.19*1.95} ${0.19} ${0.3}"/>
+          </geometry>
+          <material name="Grey">
+            <color rgba="0.5 0.5 0.5 1"/>
+          </material>
+        </collision>
+      </xacro:if>
       <inertial>
         <origin xyz="-0.0129 0.00024 0.01759" rpy="0.0 0.0 0.0" />
