Commit message: added raycast self filter geom to arm

File: hector_tracked_vehicles_description/urdf/jasmine_2018_ugv_arm.urdf.xacro (robot description, xacro)
@@ -17,5 +17,7 @@
   <xacro:property name="joint_friction" value="0.5" />
   <xacro:macro name="manipulator_arm_macro" params="parent *origin">
+    <xacro:arg name="add_default_geom" default="true"/>
     <xacro:arg name="add_containment_self_filter_geom" default="false"/>
+    <xacro:arg name="add_raycast_self_filter_geom" default="false"/>
     <joint name="arm_base_joint" type="fixed">
       <xacro:insert_block name="origin" />
@@ -50,4 +52,12 @@
         </collision>
       </xacro:if>
+      <xacro:if value="$(arg add_raycast_self_filter_geom)">
+        <collision>
+          <origin xyz="0.0125 0.0 0.02" rpy="0 ${M_PI*0.5} 0" />
+          <geometry>
+            <cylinder length="0.055" radius="0.03"/>
+          </geometry>
+        </collision>
+      </xacro:if>
       <inertial>
         <origin xyz="-0.0129 0.00024 0.01759" rpy="0.0 0.0 0.0" />
@@ -82,4 +92,12 @@
         </geometry>
       </collision>
+      <xacro:if value="$(arg add_raycast_self_filter_geom)">
+        <collision>
+          <origin xyz="0.0 -0.0025 0.035" rpy="0 0 0" />
+          <geometry>
+            <cylinder length="0.07" radius="0.04"/>
+          </geometry>
+        </collision>
+      </xacro:if>
       <inertial>
         <origin xyz="0.00023 -0.00056 0.026" rpy="0.0 0.0 0.0" />
@@ -132,4 +150,12 @@
         </geometry>
       </collision>
+      <xacro:if value="$(arg add_raycast_self_filter_geom)">
+        <collision>
+          <origin xyz="0.0 0.13 0.0" rpy="${M_PI*0.5} 0 0" />
+          <geometry>
+            <cylinder length="${0.2 + 0.09}" radius="0.03"/>
+          </geometry>
+        </collision>
+      </xacro:if>
       <inertial>
         <origin xyz="0.00746 0.12016 0.00036" rpy="0.0 ${pi} 0.0" />
@@ -182,4 +208,12 @@
         </geometry>
       </collision>
+      <xacro:if value="$(arg add_raycast_self_filter_geom)">
+        <collision>
+          <origin xyz="-0.09 0.0 0.0" rpy="0 ${M_PI*0.5} 0" />
+          <geometry>
+            <cylinder length="${0.14 + 0.08}" radius="0.03"/>
+          </geometry>
+        </collision>
+      </xacro:if>
       <inertial>
         <origin xyz="-0.11166 0.00016 0.00038" rpy="0.0 0.0 0.0" />
@@ -226,4 +260,12 @@
         </geometry>
       </collision>
+      <xacro:if value="$(arg add_raycast_self_filter_geom)">
+        <collision>
+          <origin xyz="-0.045 0.0 0.0" rpy="0 ${M_PI*0.5} 0" />
+          <geometry>
+            <cylinder length="${0.05}" radius="0.03"/>
+          </geometry>
+        </collision>
+      </xacro:if>
 <!--      <inertial>
         <origin xyz="-0.11166 0.00016 0.00038" rpy="0.0 0.0 0.0" />

Commit message: updated collision geometry

File: hector_tracked_vehicles_description/urdf/jasmine_2018_ugv_arm.urdf.xacro (robot description, xacro)
@@ -36,7 +36,7 @@
       </visual>
       <collision>
-        <origin xyz="0.0125 0.0 0.02" rpy="0.0 0.0 0.0" />
-        <geometry>
-          <box size="0.055 0.03 0.04" />
+        <origin xyz="0.0 0.0 0.044" rpy="0.0 0.0 0.0" />
+        <geometry>
+          <box size="0.042 0.042 0.084" />
         </geometry>
       </collision>
@@ -87,7 +87,13 @@
       </visual>
       <collision>
-        <origin xyz="0.0 -0.0025 0.035" rpy="0.0 0.0 0.0" />
-        <geometry>
-          <box size="0.04 0.055 0.07" />
+        <origin xyz="0.0 0.0 0.027" rpy="0.0 0.0 0.0" />
+        <geometry>
+          <box size="0.042 0.089 0.042" />
+        </geometry>
+      </collision>
+      <collision>
+        <origin xyz="0.0 0.0 0.0075" rpy="0.0 0.0 0.0" />
+        <geometry>
+          <box size="0.05 0.042 0.015" />
         </geometry>
       </collision>
@@ -127,25 +133,31 @@
       </visual>
       <collision>
-        <origin xyz="0.0 0.01 0.025" rpy="0.0 0.0 0.0" />
-        <geometry>
-          <box size="0.035 0.045 0.01" />
-        </geometry>
-      </collision>
-      <collision>
-        <origin xyz="0.0 0.01 -0.025" rpy="0.0 0.0 0.0" />
-        <geometry>
-          <box size="0.035 0.045 0.01" />
+        <origin xyz="0.0 0.01 0.045" rpy="0.0 0.0 0.0" />
+        <geometry>
+          <box size="0.045 0.06 0.01" />
+        </geometry>
+      </collision>
+      <collision>
+        <origin xyz="0.0 0.01 -0.045" rpy="0.0 0.0 0.0" />
+        <geometry>
+          <box size="0.045 0.06 0.01" />
         </geometry>
       </collision>
      <collision>
-        <origin xyz="0.01 0.25 0.0" rpy="0.0 0.0 0.0" />
-        <geometry>
-          <box size="0.06 0.04 0.04" />
+        <origin xyz="0.0 0.0325 0.0" rpy="0.0 0.0 0.0" />
+        <geometry>
+          <box size="0.042 0.015 0.09" />
         </geometry>
      </collision>
       <collision>
-        <origin xyz="0.0 0.13 0.0" rpy="0.0 0.0 0.0" />
-        <geometry>
-          <box size="0.04 0.2 0.04" />
+        <origin xyz="0.0 0.135 0.0" rpy="0.0 0.0 0.0" />
+        <geometry>
+          <box size="0.035 0.2 0.055" />
+        </geometry>
+      </collision>
+      <collision>
+        <origin xyz="0.015 0.252 0.0" rpy="0.0 0.0 0.0" />
+        <geometry>
+          <box size="0.06 0.0425 0.05" />
         </geometry>
       </collision>
@@ -185,13 +197,13 @@
       </visual>
       <collision>
-        <origin xyz="-0.01 0.0 0.02" rpy="0.0 0.0 0.0" />
-        <geometry>
-          <box size="0.04 0.03 0.0075" />
-        </geometry>
-      </collision>
-      <collision>
-        <origin xyz="-0.01 0.0 -0.02" rpy="0.0 0.0 0.0" />
-        <geometry>
-          <box size="0.04 0.03 0.0075" />
+        <origin xyz="-0.0125 0.0 0.0275" rpy="0.0 0.0 0.0" />
+        <geometry>
+          <box size="0.04 0.03 0.01" />
+        </geometry>
+      </collision>
+      <collision>
+        <origin xyz="-0.0125 0.0 -0.0275" rpy="0.0 0.0 0.0" />
+        <geometry>
+          <box size="0.04 0.03 0.01" />
         </geometry>
       </collision>
@@ -199,5 +211,11 @@
         <origin xyz="-0.09 0.0 0.0" rpy="0.0 0.0 0.0" />
         <geometry>
-          <box size="0.14 0.03 0.04" />
+          <box size="0.13 0.03 0.055" />
+        </geometry>
+      </collision>
+      <collision>
+        <origin xyz="-0.03 0.0 0.0" rpy="0.0 0.0 0.0" />
+        <geometry>
+          <box size="0.01 0.04 0.055" />
         </geometry>
       </collision>

Commit message: updated joint limits

File: hector_tracked_vehicles_description/urdf/jasmine_2018_ugv_arm.urdf.xacro (robot description, xacro)
@@ -181,5 +181,5 @@
       <origin xyz="0.031 0.2545 0.0" rpy="0.0 0.0 ${-pi}" />
       <axis xyz="0 0 1" />
-      <limit lower="${-pi/2}" upper="${pi/2}" effort="${XM430_W350_max_effort}" velocity="${XM430_W350_max_velocity}" />
+      <limit lower="${-86.368*pi/180}" upper="${114.8*pi/180}" effort="${XM430_W350_max_effort}" velocity="${XM430_W350_max_velocity}" />
       <parent link="arm_pitch_link_0" />
       <child link="arm_pitch_link_1" />
@@ -245,5 +245,5 @@
       <origin xyz="-0.2017 -0.002 0.0" rpy="0.0 0.0 0.0" />
       <axis xyz="0 0 1" />
-      <limit lower="${-pi / 2}" upper="${pi / 2}" effort="${XM430_W350_max_effort}" velocity="${XM430_W350_max_velocity}" />
+      <limit lower="${-109.6*pi/180}" upper="${114.8*pi/180}" effort="${XM430_W350_max_effort}" velocity="${XM430_W350_max_velocity}" />
       <parent link="arm_pitch_link_1" />
       <child link="arm_pitch_link_2" />
@@ -300,5 +300,5 @@
       <origin xyz="-0.073 0.0 -0.012" rpy="${pi/2} 0.0 ${-pi/2}" />
       <axis xyz="0 0 1" />
-      <limit lower="${-pi}" upper="${162.976*pi/180}" effort="${XM430_W350_max_effort}" velocity="${XM430_W350_max_velocity}" />
+      <limit lower="${-178.24*pi/180}" upper="${136.8*pi/180}" effort="${XM430_W350_max_effort}" velocity="${XM430_W350_max_velocity}" />
       <parent link="arm_pitch_link_2" />
       <child link="arm_roll_link" />

Commit message: updated the arm URDF to include the new cameras

File: hector_tracked_vehicles_description/urdf/jasmine_2018_ugv_arm.urdf.xacro (robot description, xacro)
@@ -351,5 +351,5 @@
     <link name="gripper_palm_link">
       <visual>
-        <origin xyz="0.0 0.0 0.0" rpy="0.0 0.0 0.0" />
+        <origin xyz="0.0 0.0 0.0" rpy="0.0 0.0 ${pi}" />
         <geometry>
           <mesh filename="package://hector_tracked_vehicles_description/meshes/jasmine_ugv/gripper/gripper_palm.stl" scale="0.001 0.001 0.001" />
@@ -399,4 +399,10 @@
         <geometry>
           <cylinder length="0.02" radius="0.028" />
+        </geometry>
+      </collision>
+      <collision>
+        <origin xyz="0.0615 0.0 0.048" rpy="0.0 0.0 0.0" />
+        <geometry>
+          <box size="0.043 0.07 0.035" />
         </geometry>
       </collision>
@@ -556,6 +562,12 @@
     </link>
     <xacro:generic_camera name="gripper_cam" parent="gripper_palm_link" ros_topic="/gripper_cam/image_raw" cam_info_topic="/gripper_cam/camera_info" update_rate="15" res_x="640" res_y="480" image_format="R8G8B8" hfov="60">
-      <origin xyz="0 0 ${0.034 + 0.02}" rpy="${pi} ${-pi/2} ${-pi/2}"/>
+      <origin xyz="0 0 0.038" rpy="${pi} ${-pi/2} 0"/>
     </xacro:generic_camera>
+    <xacro:generic_camera name="gripper_top_cam" parent="gripper_palm_link" ros_topic="/gripper_top_cam/image_raw" cam_info_topic="/gripper_top_cam/camera_info" update_rate="15" res_x="640" res_y="480" image_format="R8G8B8" hfov="60">
+      <origin xyz="0.067 0 0.048" rpy="${pi} ${-pi/2} 0"/>
+    </xacro:generic_camera>
+    <xacro:seek_thermal_compact_camera_no_geom name="gripper_thermal_cam" parent="gripper_palm_link">
+      <origin xyz="0.051 0.006 0.045" rpy="0 ${-0.5*M_PI} ${-0.5*M_PI}"/>
+    </xacro:seek_thermal_compact_camera_no_geom>
   </xacro:macro>
 </robot>

Commit message: update the gripper roll joint according to the real robot

File: hector_tracked_vehicles_description/urdf/jasmine_2018_ugv_arm.urdf.xacro (robot description, xacro)
@@ -298,7 +298,7 @@
     </link>
     <joint name="arm_roll_joint" type="revolute">
-      <origin xyz="-0.073 0.0 -0.012" rpy="${pi/2} 0.0 ${-pi/2}" />
-      <axis xyz="0 0 1" />
-      <limit lower="${-178.24*pi/180}" upper="${136.8*pi/180}" effort="${XM430_W350_max_effort}" velocity="${XM430_W350_max_velocity}" />
+      <origin xyz="-0.073 0.0 -0.012" rpy="${pi/2} ${-pi/2} ${-pi/2}" />
+      <axis xyz="0 0 1" />
+      <limit lower="${-178.464*pi/180}" upper="${178.376*pi/180}" effort="${XM430_W350_max_effort}" velocity="${XM430_W350_max_velocity}" />
       <parent link="arm_pitch_link_2" />
       <child link="arm_roll_link" />
