Commit message: jasmine vlp16 calibration

File: hector_tracked_vehicles_description/calibrations/jasmine_2018_vlp16_calibration.urdf.xacro (robot description, xacro)
@@ -1,5 +1,9 @@
 <?xml version="1.0"?>
-<!-- Manually copied from tracker setup -->
-<robot xmlns:xacro="http://ros.org/wiki/xacro" name="calibration">
-  <origin xyz="0.0 0.0 0.09446" rpy="${M_PI*0.250} 0.0 ${M_PI}"/>
+<!-- =================================================================================== -->
+<!-- |    This document was autogenerated by lidar_calibration on 25.04.2018, 20:07:57.| -->
+<!-- |    Insert this transformation between frames spin_lidar_lidar_mount_link and spin_lidar_pitch_hokuyo_laser_frame. | -->
+<!-- |    EDITING THIS FILE BY HAND IS NOT RECOMMENDED                                 | -->
+<!-- =================================================================================== -->
+<robot xmlns:xacro="http://www.ros.org/wiki/xacro" name="calibration">
+  <origin xyz="0.00121691 0.00757118 0" rpy="0.790913 -0.00506962 3.14157"/>
 </robot>

Commit message: Revert "jasmine vlp16 calibration"
This reverts commit 69ac55258e15744bf5847f4693cb53e17fee8d04.

File: hector_tracked_vehicles_description/calibrations/jasmine_2018_vlp16_calibration.urdf.xacro (robot description, xacro)
@@ -1,9 +1,5 @@
 <?xml version="1.0"?>
-<!-- =================================================================================== -->
-<!-- |    This document was autogenerated by lidar_calibration on 25.04.2018, 20:07:57.| -->
-<!-- |    Insert this transformation between frames spin_lidar_lidar_mount_link and spin_lidar_pitch_hokuyo_laser_frame. | -->
-<!-- |    EDITING THIS FILE BY HAND IS NOT RECOMMENDED                                 | -->
-<!-- =================================================================================== -->
-<robot xmlns:xacro="http://www.ros.org/wiki/xacro" name="calibration">
-  <origin xyz="0.00121691 0.00757118 0" rpy="0.790913 -0.00506962 3.14157"/>
+<!-- Manually copied from tracker setup -->
+<robot xmlns:xacro="http://ros.org/wiki/xacro" name="calibration">
+  <origin xyz="0.0 0.0 0.09446" rpy="${M_PI*0.250} 0.0 ${M_PI}"/>
 </robot>

Commit message: fixed jasmine vlp16 calibration

File: hector_tracked_vehicles_description/calibrations/jasmine_2018_vlp16_calibration.urdf.xacro (robot description, xacro)
@@ -1,5 +1,9 @@
 <?xml version="1.0"?>
-<!-- Manually copied from tracker setup -->
-<robot xmlns:xacro="http://ros.org/wiki/xacro" name="calibration">
-  <origin xyz="0.0 0.0 0.09446" rpy="${M_PI*0.250} 0.0 ${M_PI}"/>
+<!-- =================================================================================== -->
+<!-- |    This document was autogenerated by lidar_calibration on 25.04.2018, 21:46:45.| -->
+<!-- |    Insert this transformation between frames spin_lidar_lidar_mount_link and spin_lidar_pitch_hokuyo_laser_frame. | -->
+<!-- |    EDITING THIS FILE BY HAND IS NOT RECOMMENDED                                 | -->
+<!-- =================================================================================== -->
+<robot xmlns:xacro="http://www.ros.org/wiki/xacro" name="calibration">
+  <origin xyz="-0.00203613 0.00579971 0.0944673" rpy="0.789793 -0.00528362 3.14158"/>
 </robot>

Commit message: Update vlp16 setup to have fixed frame in correct location (i.e. spinning lidar center)

File: hector_tracked_vehicles_description/calibrations/jasmine_2018_vlp16_calibration.urdf.xacro (robot description, xacro)
@@ -6,4 +6,4 @@
 <!-- =================================================================================== -->
 <robot xmlns:xacro="http://www.ros.org/wiki/xacro" name="calibration">
-  <origin xyz="-0.00203613 0.00579971 0.0944673" rpy="0.789793 -0.00528362 3.14158"/>
+  <origin xyz="-0.00203613 0.00579971 0.0" rpy="0.789793 -0.00528362 3.14158"/>
 </robot>

File: hector_tracked_vehicles_description/urdf/jasmine_2018_ugv.urdf.xacro (robot description, xacro)
@@ -29,5 +29,5 @@
     <xacro:spinning_sensor_mount_macro parent="base_link"  name="spin_lidar" scaling="0.001">
       <!-- the angles are due to ground calibration with tud tracker vlp16 -->
-      <origin xyz="${+0.0 } 0.0 ${0.27}" rpy="0.0 0.0 0"/>
+      <origin xyz="${+0.0 } 0.0 ${0.27 + 0.0944673}" rpy="0.0 0.0 0"/>
     </xacro:spinning_sensor_mount_macro>
     <xacro:include filename="$(find hector_sensors_description)/urdf/ricoh_theta.urdf.xacro"/>

File: hector_tracked_vehicles_description/urdf/jasmine_ugv_base.urdf.xacro (robot description, xacro)
@@ -86,4 +86,10 @@
               <xacro:jasmine_ugv_tracks t_base_size_x="${base_size_x}"  t_base_size_y="${base_size_y}" t_base_size_z="${base_size_z}" t_flipper_offset_x="${flipper_offset_x}" t_wheel_offset_y="${wheel_offset_y}" t_wheel_radius_big="${wheel_radius_big*1.2}" t_track_width="${track_width}">
               </xacro:jasmine_ugv_tracks>
+              <collision>
+                <origin xyz="0.2 0.04 0.13" rpy="0 0 0" />
+                <geometry>
+                    <box size="${0.1} ${0.2} ${0.15}" />
+                </geometry>
+              </collision>
             </xacro:if>
         </link>

Commit message: reset vlp16 calibration

File: hector_tracked_vehicles_description/calibrations/jasmine_2018_vlp16_calibration.urdf.xacro (robot description, xacro)
@@ -5,5 +5,6 @@
 <!-- |    EDITING THIS FILE BY HAND IS NOT RECOMMENDED                                 | -->
 <!-- =================================================================================== -->
+<!-- Set to identity transform on 17.09.2018 by MO -->
 <robot xmlns:xacro="http://www.ros.org/wiki/xacro" name="calibration">
-  <origin xyz="-0.00203613 0.00579971 0.0" rpy="0.789793 -0.00528362 3.14158"/>
+  <origin xyz="0.0 0.0 0.0" rpy="0.7854 0.0 0.0"/>
 </robot>

Commit message: lidar calibration

File: hector_tracked_vehicles_description/calibrations/jasmine_2018_vlp16_calibration.urdf.xacro (robot description, xacro)
@@ -1,10 +1,9 @@
 <?xml version="1.0"?>
 <!-- =================================================================================== -->
-<!-- |    This document was autogenerated by lidar_calibration on 25.04.2018, 21:46:45.| -->
+<!-- |    This document was autogenerated by lidar_calibration on 6.10.2018, 14:38:10.| -->
 <!-- |    Insert this transformation between frames spin_lidar_lidar_mount_link and spin_lidar_pitch_hokuyo_laser_frame. | -->
 <!-- |    EDITING THIS FILE BY HAND IS NOT RECOMMENDED                                 | -->
 <!-- =================================================================================== -->
-<!-- Set to identity transform on 17.09.2018 by MO -->
 <robot xmlns:xacro="http://www.ros.org/wiki/xacro" name="calibration">
-  <origin xyz="0.0 0.0 0.0" rpy="0.7854 0.0 0.0"/>
+  <origin xyz="0 -0.00396994 0" rpy="-2.35147 -3.13295 3.14155"/>
 </robot>

Commit message: lidar calibration

File: hector_tracked_vehicles_description/calibrations/jasmine_2018_vlp16_calibration.urdf.xacro (robot description, xacro)
@@ -1,9 +1,9 @@
 <?xml version="1.0"?>
 <!-- =================================================================================== -->
-<!-- |    This document was autogenerated by lidar_calibration on 6.10.2018, 14:38:10.| -->
+<!-- |    This document was autogenerated by lidar_calibration on 2.05.2019, 08:52:49.| -->
 <!-- |    Insert this transformation between frames spin_lidar_lidar_mount_link and spin_lidar_pitch_hokuyo_laser_frame. | -->
 <!-- |    EDITING THIS FILE BY HAND IS NOT RECOMMENDED                                 | -->
 <!-- =================================================================================== -->
 <robot xmlns:xacro="http://www.ros.org/wiki/xacro" name="calibration">
-  <origin xyz="0 -0.00396994 0" rpy="-2.35147 -3.13295 3.14155"/>
+  <origin xyz="-0.00218016 -0.00376291 0" rpy="-2.35019 -3.1334 3.14154"/>
 </robot>

Commit message: use the default lidar transformation until Martin calibrates Jasmine again

File: hector_tracked_vehicles_description/calibrations/jasmine_2018_vlp16_calibration.urdf.xacro (robot description, xacro)
@@ -6,4 +6,4 @@
 <!-- =================================================================================== -->
 <robot xmlns:xacro="http://www.ros.org/wiki/xacro" name="calibration">
-  <origin xyz="-0.00218016 -0.00376291 0" rpy="-2.35019 -3.1334 3.14154"/>
+  <origin xyz="0 0 0" rpy="${M_PI/4} 0 0"/>
 </robot>

Commit message: lidar calibration

File: hector_tracked_vehicles_description/calibrations/jasmine_2018_vlp16_calibration.urdf.xacro (robot description, xacro)
@@ -1,9 +1,9 @@
 <?xml version="1.0"?>
 <!-- =================================================================================== -->
-<!-- |    This document was autogenerated by lidar_calibration on 2.05.2019, 08:52:49.| -->
-<!-- |    Insert this transformation between frames spin_lidar_lidar_mount_link and spin_lidar_pitch_hokuyo_laser_frame. | -->
+<!-- |    This document was autogenerated by lidar_calibration on 20.07.2020, 17:47:08.| -->
+<!-- |    Insert this transformation between frames spin_lidar_mount_link and spin_lidar_laser_frame. | -->
 <!-- |    EDITING THIS FILE BY HAND IS NOT RECOMMENDED                                 | -->
 <!-- =================================================================================== -->
 <robot xmlns:xacro="http://www.ros.org/wiki/xacro" name="calibration">
-  <origin xyz="0 0 0" rpy="${M_PI/4} 0 0"/>
+  <origin xyz="-0.00137209 -0.00430858 0" rpy="-2.35412 -3.13796 3.14158"/>
 </robot>
